Commit message: rename unused "name" param in kinova to avoid confusion with component names

File: urdf/kinova.urdf.xacro (robot description, xacro)
@@ -55,5 +55,5 @@
     <xacro:property name="prefix" value="${device_namespace + '_' if device_namespace != '' else ''}" />
     <!-- robot name parameter -->
-    <xacro:property name="name" value="kinova_arm" />
+    <xacro:property name="robot_name" value="kinova_arm" />
     <!-- Arguments -->
     <xacro:property name="robot_ip" value="192.168.11.11" />

Commit message: kinova urdf: remove robot_name

File: urdf/kinova.urdf.xacro (robot description, xacro)
@@ -58,6 +58,4 @@
       ns="kinova_manipulator"
     />
-    <!-- robot name parameter -->
-    <xacro:property name="robot_name" value="kinova_arm" />
     <!-- Arguments -->
     <xacro:property name="robot_ip" value="192.168.11.11" />
