Commit message: add simple visuals

File: urdf/intel_realsense_d435.urdf.xacro (robot description, xacro)
@@ -61,9 +61,19 @@
     </joint>
     <link name="${device_namespace}_link">
-      <visual>
+      <!-- <visual>
         <origin xyz="0.0 0.0 0.0" rpy="0.0 0.0 0.0" />
         <geometry>
           <mesh filename="package://husarion_components_description/meshes/intel_realsense_d435.dae" />
         </geometry>
+      </visual> -->
+      <!-- TODO Remove simple visuals when mesh is ready -->
+      <visual>
+        <origin xyz="0.0 0.0 0.0" rpy="0.0 0.0 0.0" />
+        <geometry>
+          <box size="${d435_cam_depth} ${d435_cam_width} ${d435_cam_height}" />
+        </geometry>
+        <material name="LightGrey">
+          <color rgba="0.6 0.6 0.6 1.0" />
+        </material>
       </visual>
       <collision>

File: urdf/orbbec_astra.urdf.xacro (robot description, xacro)
@@ -32,9 +32,28 @@
     </joint>
     <link name="${device_namespace}_orbbec_astra_link">
-      <visual>
+      <!-- <visual>
         <origin xyz="0.0 0.0 0.0" rpy="0.0 0.0 0.0" />
         <geometry>
           <mesh filename="package://husarion_components_description/meshes/orbbec_astra.dae" />
         </geometry>
+      </visual> -->
+      <!-- TODO Remove simple visuals when mesh is ready -->
+      <visual>
+        <origin xyz="${0.0225-0.04/2.0} 0.0 ${0.019+0.03/2.0}" rpy="0.0 0.0 0.0" />
+        <geometry>
+          <box size="0.04 0.165 0.03" />
+        </geometry>
+        <material name="LightGrey">
+          <color rgba="0.6 0.6 0.6 1.0" />
+        </material>
+      </visual>
+      <visual>
+        <origin xyz="${0.0235-0.06/2.0} 0.0 ${0.019/2.0}" rpy="0.0 0.0 0.0" />
+        <geometry>
+          <box size="0.06 0.06 0.019" />
+        </geometry>
+        <material name="LightGrey">
+          <color rgba="0.6 0.6 0.6 1.0" />
+        </material>
       </visual>
       <!-- camera module collision -->

File: urdf/ouster.urdf.xacro (robot description, xacro)
@@ -65,9 +65,19 @@
     </joint>
     <link name="${prefix}ouster_${model}_link">
-      <visual>
+      <!-- <visual>
         <origin xyz="0.0 0.0 0.0" rpy="0.0 0.0 0.0" />
         <geometry>
           <mesh filename="package://husarion_components_description/meshes/${mesh}.dae" />
         </geometry>
+      </visual> -->
+      <!-- TODO Remove simple visuals when mesh is ready -->
+      <visual>
+        <origin xyz="0.0 0.0 0.0" rpy="0.0 0.0 0.0" />
+        <geometry>
+          <cylinder radius="${0.085/2.0}" length="0.073" />
+        </geometry>
+        <material name="LightGrey">
+          <color rgba="0.6 0.6 0.6 1.0" />
+        </material>
       </visual>
       <collision>

File: urdf/slamtec_rplidar.urdf.xacro (robot description, xacro)
@@ -84,6 +84,5 @@
         <origin xyz="0.0 0.0 0.025" rpy="0.0 0.0 0.0" />
         <geometry>
-          <cylinder radius="0.022" length="0.05" />
-          <box size="0.0555 0.0555 0.0195" />
+          <cylinder radius="0.025" length="0.05" />
         </geometry>
       </xacro:property>
@@ -203,9 +202,17 @@
     </joint>
     <link name="${prefix}slamtec_rplidar_link">
+      <!-- <visual>
+        <origin xyz="0.0 0.0 0.0" rpy="0.0 0.0 0.0" />
+        <geometry>
+          <mesh filename="package://husarion_components_description/meshes/rplidar/${mesh}" />
+        </geometry>
+      </visual> -->
+      <!-- TODO Remove simple visuals when mesh is ready -->
       <visual>
         <origin xyz="0.0 0.0 0.0" rpy="0.0 0.0 0.0" />
-        <geometry>
-          <mesh filename="package://husarion_components_description/meshes/rplidar/${mesh}" />
-        </geometry>
+        <xacro:insert_block name="collision" />
+        <material name="LightGrey">
+          <color rgba="0.6 0.6 0.6 1.0" />
+        </material>
       </visual>
       <collision>

File: urdf/stereolabs_zed.urdf.xacro (robot description, xacro)
@@ -30,4 +30,10 @@
       <xacro:property name="screw_offset_z" value="0.0" />
       <xacro:property name="optical_offset_x" value="-0.01" />
+      <xacro:property name="collision">
+        <origin xyz="${screw_offset_x-0.02} 0 ${screw_offset_z}" rpy="0.0 0.0 0.0" />
+        <geometry>
+          <box size="0.033 0.175 0.03" />
+        </geometry>
+      </xacro:property>
     </xacro:if>
     <xacro:if value="${model == 'zedm'}">
@@ -38,4 +44,10 @@
       <xacro:property name="screw_offset_z" value="0.0" />
       <xacro:property name="optical_offset_x" value="0.0" />
+      <xacro:property name="collision">
+        <origin xyz="${screw_offset_x-0.015} 0.008 ${screw_offset_z}" rpy="0.0 0.0 0.0" />
+        <geometry>
+          <box size="0.026 0.124 0.03" />
+        </geometry>
+      </xacro:property>
     </xacro:if>
     <xacro:if value="${model == 'zed2'}">
@@ -46,4 +58,10 @@
       <xacro:property name="screw_offset_z" value="0.0" />
       <xacro:property name="optical_offset_x" value="-0.01" />
+      <xacro:property name="collision">
+        <origin xyz="${screw_offset_x-0.02} 0 ${screw_offset_z}" rpy="0.0 0.0 0.0" />
+        <geometry>
+          <box size="0.033 0.175 0.03" />
+        </geometry>
+      </xacro:property>
     </xacro:if>
     <xacro:if value="${model == 'zed2i'}">
@@ -54,4 +72,10 @@
       <xacro:property name="screw_offset_z" value="0.0" />
       <xacro:property name="optical_offset_x" value="-0.01" />
+      <xacro:property name="collision">
+        <origin xyz="${screw_offset_x-0.015} 0 ${screw_offset_z}" rpy="0.0 0.0 0.0" />
+        <geometry>
+          <box size="0.043 0.175 0.03" />
+        </geometry>
+      </xacro:property>
     </xacro:if>
     <xacro:if value="${model == 'zedx'}">
@@ -62,4 +86,10 @@
       <xacro:property name="screw_offset_z" value="-0.016" />
       <xacro:property name="optical_offset_x" value="-0.01" />
+      <xacro:property name="collision">
+        <origin xyz="${screw_offset_z-0.01} 0 0" rpy="0.0 0.0 0.0" />
+        <geometry>
+          <box size="0.037 0.163 0.032" />
+        </geometry>
+      </xacro:property>
     </xacro:if>
     <xacro:if value="${model == 'zedxm'}">
@@ -70,4 +100,10 @@
       <xacro:property name="screw_offset_z" value="-0.016" />
       <xacro:property name="optical_offset_x" value="-0.01" />
+      <xacro:property name="collision">
+        <origin xyz="${screw_offset_z-0.01} 0 0" rpy="0.0 0.0 0.0" />
+        <geometry>
+          <box size="0.037 0.094 0.032" />
+        </geometry>
+      </xacro:property>
     </xacro:if>
     <!-- Camera mounting point (the threaded screw hole in the bottom) -->
@@ -84,5 +120,5 @@
         <origin xyz="${screw_offset_x-0.02} 0 ${screw_offset_z}" rpy="0 0 0" />
         <geometry>
-          <mesh filename="package://husarion_components_description/meshes/stereolabs/${model}.stl" />
+          <mesh filename="package://zed_msgs/meshes/${model}.stl" />
         </geometry>
         <material name="mat">
@@ -91,7 +127,5 @@
       </visual>
       <collision>
-        <geometry>
-          <mesh filename="package://husarion_components_description/meshes/stereolabs/${model}.stl" />
-        </geometry>
+        <xacro:insert_block name="collision" />
       </collision>
     </link>

File: urdf/velodyne_puck.urdf.xacro (robot description, xacro)
@@ -28,9 +28,19 @@
     </joint>
     <link name="${prefix}velodyne_puck_link">
-      <visual>
+      <!-- <visual>
         <origin xyz="0.0 0.0 0.0" rpy="0.0 0.0 0.0" />
         <geometry>
           <mesh filename="package://husarion_components_description/meshes/velodyne_puck.dae" />
         </geometry>
+      </visual> -->
+      <!-- TODO Remove simple visuals when mesh is ready -->
+      <visual>
+        <origin xyz="0.0 0.0 ${0.072/2.0}" rpy="0.0 0.0 0.0" />
+        <geometry>
+          <cylinder radius="${0.103/2.0}" length="0.072" />
+        </geometry>
+        <material name="LightGrey">
+          <color rgba="0.6 0.6 0.6 1.0" />
+        </material>
       </visual>
       <collision>

File: urdf/wibotic_receiver.urdf.xacro (robot description, xacro)
@@ -27,5 +27,5 @@
     </joint>
     <link name="${prefix}wibotic_receiver_link">
-      <visual>
+      <!-- <visual>
         <origin xyz="0.0 0.0 0.0" rpy="0.0 0.0 ${pi/2.0}" />
         <geometry>
@@ -35,9 +35,34 @@
           <color rgba="0.15 0.15 0.15 1.0" />
         </material>
+      </visual> -->
+      <!-- TODO Remove simple visuals when mesh is ready -->
+      <visual>
+        <origin xyz="-0.008 0.0 0.085" rpy="0.0 0.0 0.0" />
+        <geometry>
+          <box size="0.015 0.135 0.19" />
+        </geometry>
+        <material name="DarkGrey">
+          <color rgba="0.2 0.2 0.2 1.0" />
+        </material>
+      </visual>
+      <visual>
+        <origin xyz="0.014 0.0 0.115" rpy="0.0 ${pi/2.0} 0.0" />
+        <geometry>
+          <cylinder length="0.03" radius="0.07" />
+        </geometry>
+        <material name="DarkGrey">
+          <color rgba="0.2 0.2 0.2 1.0" />
+        </material>
       </visual>
       <collision>
-        <origin xyz="0.0 0.0 0.0" rpy="0.0 0.0 ${pi/2.0}" />
+        <origin xyz="-0.008 0.0 0.085" rpy="0.0 0.0 0.0" />
         <geometry>
-          <mesh filename="package://husarion_components_description/meshes/wibotic_receiver.stl" />
+          <box size="0.015 0.135 0.19" />
+        </geometry>
+      </collision>
+      <collision>
+        <origin xyz="0.014 0.0 0.115" rpy="0.0 ${pi/2.0} 0.0" />
+        <geometry>
+          <cylinder length="0.03" radius="0.07" />
         </geometry>
       </collision>

File: urdf/wibotic_station.urdf.xacro (robot description, xacro)
@@ -19,5 +19,6 @@
                params="parent_link
                        xyz:='0.0 0.0 0.0'
-                       rpy:='0.0 0.0 0.0'">
+                       rpy:='0.0 0.0 0.0'
+                       device_namespace:='station'">
     <xacro:property name="prefix" value="${device_namespace + '_' if device_namespace != '' else ''}" />
     <joint name="${parent_link.rstrip('_link')}_to_${prefix}wibotic_station_joint" type="fixed">
@@ -27,8 +28,15 @@
     </joint>
     <link name="${prefix}wibotic_station_link">
-      <visual>
+      <!-- <visual>
         <origin xyz="0.0 0.0 0.0" rpy="0.0 0.0 ${pi/2.0}" />
         <geometry>
           <mesh filename="package://husarion_components_description/meshes/wibotic_station.stl" />
+        </geometry>
+      </visual> -->
+      <!-- TODO Remove simple visuals when mesh is ready -->
+      <visual>
+        <origin xyz="-0.2 0.0  0.4" rpy="0.0 0.0 0.0" />
+        <geometry>
+          <box size="0.4 0.5 0.8" />
         </geometry>
         <material name="LightGrey">
@@ -47,7 +55,7 @@
         <origin xyz="-0.2 0.0 0.0" rpy="0.0 0.0 0.0" />
         <mass value="15.0" />
-        <inertia ixx="0.001111" ixy="0.0" ixz="0.0"
-          iyy="0.001111" iyz="0.0"
-          izz="0.001111" />
+        <inertia ixx="0.001111" ixy="0.0"      ixz="0.0"
+                                iyy="0.001111" iyz="0.0"
+                                               izz="0.001111" />
       </inertial>
     </link>

Commit message: use realsense2_description meshes

File: urdf/intel_realsense_d435.urdf.xacro (robot description, xacro)
@@ -34,11 +34,4 @@
     <xacro:property name="d435_cam_depth" value="0.02505" />
     <xacro:property name="d435_cam_mount_from_center_offset" value="0.0149" />
-    <!-- glass cover is 0.1 mm inwards from front aluminium plate -->
-    <xacro:property name="d435_glass_to_front" value="0.0001" />
-    <!-- see datasheet Revision 007, Fig. 4-4 page 65 -->
-    <xacro:property name="d435_zero_depth_to_glass" value="0.0042" />
-    <!-- convenience precomputation to avoid clutter-->
-    <xacro:property name="d435_mesh_x_offset"
-      value="${d435_cam_mount_from_center_offset-d435_glass_to_front-d435_zero_depth_to_glass}" />
     <!-- The following offset is relative the the physical D435 camera peripheral
       camera tripod mount -->
@@ -55,5 +48,5 @@
     <link name="${device_namespace}_bottom_screw_frame" />
     <joint name="${device_namespace}_bottom_screw_to_${device_namespace}_joint" type="fixed">
-      <origin xyz="${d435_mesh_x_offset} ${d435_cam_depth_py} ${d435_cam_depth_pz}"
+      <origin xyz="0.0 ${d435_cam_depth_py} ${d435_cam_depth_pz}"
         rpy="0.0 0.0 0.0" />
       <parent link="${device_namespace}_bottom_screw_frame" />
@@ -61,19 +54,9 @@
     </joint>
     <link name="${device_namespace}_link">
-      <!-- <visual>
-        <origin xyz="0.0 0.0 0.0" rpy="0.0 0.0 0.0" />
+      <visual>
+        <origin xyz="${d435_cam_mount_from_center_offset} ${-d435_cam_depth_py} 0.0" rpy="${pi/2.0} 0.0 ${pi/2.0}" />
         <geometry>
-          <mesh filename="package://husarion_components_description/meshes/intel_realsense_d435.dae" />
+          <mesh filename="package://realsense2_description/meshes/d435.dae" />
         </geometry>
-      </visual> -->
-      <!-- TODO Remove simple visuals when mesh is ready -->
-      <visual>
-        <origin xyz="0.0 0.0 0.0" rpy="0.0 0.0 0.0" />
-        <geometry>
-          <box size="${d435_cam_depth} ${d435_cam_width} ${d435_cam_height}" />
-        </geometry>
-        <material name="LightGrey">
-          <color rgba="0.6 0.6 0.6 1.0" />
-        </material>
       </visual>
       <collision>

Commit message: Add visuals (#2)
* add NOTICE.md file

* add simple visuals

* add backport action

* unify files

* use realsense2_description meshes

File: urdf/intel_realsense_d435.urdf.xacro (robot description, xacro)
@@ -34,11 +34,4 @@
     <xacro:property name="d435_cam_depth" value="0.02505" />
     <xacro:property name="d435_cam_mount_from_center_offset" value="0.0149" />
-    <!-- glass cover is 0.1 mm inwards from front aluminium plate -->
-    <xacro:property name="d435_glass_to_front" value="0.0001" />
-    <!-- see datasheet Revision 007, Fig. 4-4 page 65 -->
-    <xacro:property name="d435_zero_depth_to_glass" value="0.0042" />
-    <!-- convenience precomputation to avoid clutter-->
-    <xacro:property name="d435_mesh_x_offset"
-      value="${d435_cam_mount_from_center_offset-d435_glass_to_front-d435_zero_depth_to_glass}" />
     <!-- The following offset is relative the the physical D435 camera peripheral
       camera tripod mount -->
@@ -55,5 +48,5 @@
     <link name="${device_namespace}_bottom_screw_frame" />
     <joint name="${device_namespace}_bottom_screw_to_${device_namespace}_joint" type="fixed">
-      <origin xyz="${d435_mesh_x_offset} ${d435_cam_depth_py} ${d435_cam_depth_pz}"
+      <origin xyz="0.0 ${d435_cam_depth_py} ${d435_cam_depth_pz}"
         rpy="0.0 0.0 0.0" />
       <parent link="${device_namespace}_bottom_screw_frame" />
@@ -62,7 +55,7 @@
     <link name="${device_namespace}_link">
       <visual>
-        <origin xyz="0.0 0.0 0.0" rpy="0.0 0.0 0.0" />
+        <origin xyz="${d435_cam_mount_from_center_offset} ${-d435_cam_depth_py} 0.0" rpy="${pi/2.0} 0.0 ${pi/2.0}" />
         <geometry>
-          <mesh filename="package://husarion_components_description/meshes/intel_realsense_d435.dae" />
+          <mesh filename="package://realsense2_description/meshes/d435.dae" />
         </geometry>
       </visual>

File: urdf/stereolabs_zed.urdf.xacro (robot description, xacro)
@@ -30,4 +30,10 @@
       <xacro:property name="screw_offset_z" value="0.0" />
       <xacro:property name="optical_offset_x" value="-0.01" />
+      <xacro:property name="collision">
+        <origin xyz="${screw_offset_x-0.02} 0 ${screw_offset_z}" rpy="0.0 0.0 0.0" />
+        <geometry>
+          <box size="0.033 0.175 0.03" />
+        </geometry>
+      </xacro:property>
     </xacro:if>
     <xacro:if value="${model == 'zedm'}">
@@ -38,4 +44,10 @@
       <xacro:property name="screw_offset_z" value="0.0" />
       <xacro:property name="optical_offset_x" value="0.0" />
+      <xacro:property name="collision">
+        <origin xyz="${screw_offset_x-0.015} 0.008 ${screw_offset_z}" rpy="0.0 0.0 0.0" />
+        <geometry>
+          <box size="0.026 0.124 0.03" />
+        </geometry>
+      </xacro:property>
     </xacro:if>
     <xacro:if value="${model == 'zed2'}">
@@ -46,4 +58,10 @@
       <xacro:property name="screw_offset_z" value="0.0" />
       <xacro:property name="optical_offset_x" value="-0.01" />
+      <xacro:property name="collision">
+        <origin xyz="${screw_offset_x-0.02} 0 ${screw_offset_z}" rpy="0.0 0.0 0.0" />
+        <geometry>
+          <box size="0.033 0.175 0.03" />
+        </geometry>
+      </xacro:property>
     </xacro:if>
     <xacro:if value="${model == 'zed2i'}">
@@ -54,4 +72,10 @@
       <xacro:property name="screw_offset_z" value="0.0" />
       <xacro:property name="optical_offset_x" value="-0.01" />
+      <xacro:property name="collision">
+        <origin xyz="${screw_offset_x-0.015} 0 ${screw_offset_z}" rpy="0.0 0.0 0.0" />
+        <geometry>
+          <box size="0.043 0.175 0.03" />
+        </geometry>
+      </xacro:property>
     </xacro:if>
     <xacro:if value="${model == 'zedx'}">
@@ -62,4 +86,10 @@
       <xacro:property name="screw_offset_z" value="-0.016" />
       <xacro:property name="optical_offset_x" value="-0.01" />
+      <xacro:property name="collision">
+        <origin xyz="${screw_offset_z-0.01} 0 0" rpy="0.0 0.0 0.0" />
+        <geometry>
+          <box size="0.037 0.163 0.032" />
+        </geometry>
+      </xacro:property>
     </xacro:if>
     <xacro:if value="${model == 'zedxm'}">
@@ -70,4 +100,10 @@
       <xacro:property name="screw_offset_z" value="-0.016" />
       <xacro:property name="optical_offset_x" value="-0.01" />
+      <xacro:property name="collision">
+        <origin xyz="${screw_offset_z-0.01} 0 0" rpy="0.0 0.0 0.0" />
+        <geometry>
+          <box size="0.037 0.094 0.032" />
+        </geometry>
+      </xacro:property>
     </xacro:if>
     <!-- Camera mounting point (the threaded screw hole in the bottom) -->
@@ -84,5 +120,5 @@
         <origin xyz="${screw_offset_x-0.02} 0 ${screw_offset_z}" rpy="0 0 0" />
         <geometry>
-          <mesh filename="package://husarion_components_description/meshes/stereolabs/${model}.stl" />
+          <mesh filename="package://zed_msgs/meshes/${model}.stl" />
         </geometry>
         <material name="mat">
@@ -91,7 +127,5 @@
       </visual>
       <collision>
-        <geometry>
-          <mesh filename="package://husarion_components_description/meshes/stereolabs/${model}.stl" />
-        </geometry>
+        <xacro:insert_block name="collision" />
       </collision>
     </link>
@@ -156,53 +190,27 @@
       </joint>
     </xacro:if>
-    <!-- It is also possible to use single rgbd_camera sensor, but using separate rgb and depth
-    camera
-      should be more accurate different frames and fovs can be set -->
-    <gazebo reference="${device_namespace}_center">
-      <sensor type="camera" name="${ns}${device_namespace}_stereolabs_zed_color">
-        <always_on>true</always_on>
-        <update_rate>30.0</update_rate>
-        <topic>${ns}${device_namespace}/zed_node/rgb/image_rect_color</topic>
-        <visualize>false</visualize>
-        <gz_frame_id>${ns}${device_namespace}_center_optical_frame</gz_frame_id>
-        <camera>
-          <horizontal_fov>${110.0/180.0*pi}</horizontal_fov>
-          <image>
-            <width>1920</width>
-            <height>1080</height>
-            <format>R8G8B8</format>
-          </image>
-          <clip>
-            <near>0.02</near>
-            <far>300.0</far>
-          </clip>
-        </camera>
-      </sensor>
-    </gazebo>
-    <gazebo reference="${device_namespace}_center">
-      <sensor type="depth_camera" name="${ns}${device_namespace}_stereolabs_zed_depth">
-        <always_on>true</always_on>
-        <update_rate>30.0</update_rate>
-        <topic>${ns}${device_namespace}/zed_node/depth</topic>
-        <visualize>false</visualize>
-        <gz_frame_id>${ns}${device_namespace}_center_optical_frame</gz_frame_id>
-        <camera>
-          <horizontal_fov>${110.0/180.0*pi}</horizontal_fov>
-          <image>
-            <width>1920</width>
-            <height>1080</height>
-            <format>R_FLOAT32</format>
-          </image>
-          <clip>
-            <near>0.3</near>
-            <far>20.0</far>
-          </clip>
-          <noise type="gaussian">
-            <mean>0.0</mean>
-            <stddev>0.03</stddev>
-          </noise>
-        </camera>
-      </sensor>
-    </gazebo>
+    <!-- GAZEBO -->
+    <xacro:include filename="$(find husarion_components_description)/urdf/gz_sensor.urdf.xacro" ns="gz_sensor" />
+    <xacro:gz_sensor.camera
+      reference="${device_namespace}_center"
+      name="${ns}${device_namespace}_stereolabs_zed_color"
+      topic="${ns}${device_namespace}/zed_node/rgb/image_rect_color"
+      frame_id="${ns}${device_namespace}_center_optical_frame"
+      frequency="30"
+      width="1920"
+      height="1080"
+      fov="${110.0/180.0*pi}" />
+    <xacro:gz_sensor.depth_camera
+      reference="${device_namespace}_center"
+      name="${ns}${device_namespace}_stereolabs_zed_depth"
+      topic="${ns}${device_namespace}/zed_node/depth"
+      frame_id="${ns}${device_namespace}_center_optical_frame"
+      frequency="30"
+      width="1920"
+      height="1080"
+      fov="${110.0/180.0*pi}"
+      min_dist="0.3"
+      max_dist="20.0"
+      stddev_error="0.03" />
   </xacro:macro>
 </robot>
