Commit message: macros: rename prefixes: ns -> robot_namespace_slash prefix -> component_name_underscore device_ns -> component_name_slash

File: urdf/intel_realsense_d435.urdf.xacro (robot description, xacro)
@@ -21,5 +21,5 @@
                        robot_namespace:=''
                        component_name:=''">
-    <xacro:property name="ns" value="${robot_namespace + '/' if robot_namespace != '' else ''}" />
+    <xacro:property name="robot_namespace_slash" value="${robot_namespace + '/' if robot_namespace != '' else ''}" />
     <!-- The following values are approximate, and the camera node
       publishing TF values with actual calibrated camera extrinsic values -->
@@ -137,7 +137,7 @@
     <xacro:gz_sensor.camera
       reference="${component_name}_link"
-      name="${ns}${component_name}_intel_realsense_d435_color"
-      topic="${ns}${component_name}/color/image_raw"
-      frame_id="${ns}${component_name}_color_optical_frame"
+      name="${robot_namespace_slash}${component_name}_intel_realsense_d435_color"
+      topic="${robot_namespace_slash}${component_name}/color/image_raw"
+      frame_id="${robot_namespace_slash}${component_name}_color_optical_frame"
       frequency="30"
       width="1280"
@@ -146,7 +146,7 @@
     <xacro:gz_sensor.depth_camera
       reference="${component_name}_link"
-      name="${ns}${component_name}_intel_realsense_d435_depth"
-      topic="${ns}${component_name}/depth/image_rect_raw"
-      frame_id="${ns}${component_name}_depth_optical_frame"
+      name="${robot_namespace_slash}${component_name}_intel_realsense_d435_depth"
+      topic="${robot_namespace_slash}${component_name}/depth/image_rect_raw"
+      frame_id="${robot_namespace_slash}${component_name}_depth_optical_frame"
       frequency="30"
       width="1280"

File: urdf/kinova.urdf.xacro (robot description, xacro)
@@ -52,6 +52,6 @@
       ns="kinova_manipulator"
     />
-    <xacro:property name="ns" value="${robot_namespace + '/' if robot_namespace != '' else ''}" />
-    <xacro:property name="prefix" value="${component_name + '_' if component_name != '' else ''}" />
+    <xacro:property name="robot_namespace_slash" value="${robot_namespace + '/' if robot_namespace != '' else ''}" />
+    <xacro:property name="component_name_underscore" value="${component_name + '_' if component_name != '' else ''}" />
     <!-- robot name parameter -->
     <xacro:property name="robot_name" value="kinova_arm" />
@@ -96,5 +96,5 @@
       connection_inactivity_timeout_ms="${connection_inactivity_timeout_ms}"
       use_internal_bus_gripper_comm="${use_internal_bus_gripper_comm}"
-      prefix="${prefix}"
+      prefix="${component_name_underscore}"
       sim_ignition="true"
       use_fake_hardware="${use_fake_hardware}"
@@ -117,6 +117,6 @@
       <xacro:arg name="sim_isaac" default="false" />
       <xacro:kinova_manipulator.load_gripper
-        parent="${prefix}${last_arm_link}"
-        prefix="${prefix}"
+        parent="${component_name_underscore}${last_arm_link}"
+        prefix="${component_name_underscore}"
         use_fake_hardware="${use_fake_hardware}"
         fake_sensor_commands="${fake_sensor_commands}"
@@ -127,5 +127,5 @@
     <xacro:if value="${vision}">
       <gazebo reference="${component_name}_camera_color_frame">
-        <sensor name="${ns}${component_name}_camera_sensor" type="rgbd_camera">
+        <sensor name="${robot_namespace_slash}${component_name}_camera_sensor" type="rgbd_camera">
           <camera>
             <horizontal_fov>1.047</horizontal_fov>
@@ -183,5 +183,5 @@
           <update_rate>${camera_fps}</update_rate>
           <visualize>true</visualize>
-          <topic>${ns}${component_name}/wrist_mounted_camera</topic>
+          <topic>${robot_namespace_slash}${component_name}/wrist_mounted_camera</topic>
           <enable_metrics>false</enable_metrics>
         </sensor>

File: urdf/luxonis_depthai.urdf.xacro (robot description, xacro)
@@ -22,7 +22,7 @@
                        use_sim:=False">
     <xacro:include filename="$(find depthai_descriptions)/urdf/include/depthai_macro.urdf.xacro" />
-    <xacro:property name="ns" value="${robot_namespace + '/' if robot_namespace != '' else ''}" />
+    <xacro:property name="robot_namespace_slash" value="${robot_namespace + '/' if robot_namespace != '' else ''}" />
     <xacro:depthai_camera camera_name="${component_name}" parent="${parent_link}"
-      base_frame="${ns}${component_name}" camera_model="${model}"
+      base_frame="${robot_namespace_slash}${component_name}" camera_model="${model}"
       cam_pos_x="${xyz.split()[0]}" cam_pos_y="${xyz.split()[1]}" cam_pos_z="${xyz.split()[2]}"
       cam_roll="${rpy.split()[0]}" cam_pitch="${rpy.split()[1]}" cam_yaw="${rpy.split()[2]}"
@@ -31,8 +31,8 @@
       ns="gz_sensor" />
     <xacro:gz_sensor.camera
-      reference="${ns}${component_name}"
-      name="${ns}${component_name}_color"
-      topic="${ns}${component_name}/rgb/color"
-      frame_id="${ns}${component_name}_rgb_camera_frame"
+      reference="${robot_namespace_slash}${component_name}"
+      name="${robot_namespace_slash}${component_name}_color"
+      topic="${robot_namespace_slash}${component_name}/rgb/color"
+      frame_id="${robot_namespace_slash}${component_name}_rgb_camera_frame"
       frequency="30"
       width="1280"
@@ -40,8 +40,8 @@
       fov="${60.0/180.0*pi}" />
     <xacro:gz_sensor.depth_camera
-      reference="${ns}${component_name}"
-      name="${ns}${component_name}_depth"
-      topic="${ns}${component_name}/stereo/depth"
-      frame_id="${ns}${component_name}_rgb_camera_frame"
+      reference="${robot_namespace_slash}${component_name}"
+      name="${robot_namespace_slash}${component_name}_depth"
+      topic="${robot_namespace_slash}${component_name}/stereo/depth"
+      frame_id="${robot_namespace_slash}${component_name}_rgb_camera_frame"
       frequency="30"
       width="1280"

File: urdf/orbbec_astra.urdf.xacro (robot description, xacro)
@@ -19,5 +19,5 @@
                        robot_namespace:=''
                        component_name:=''">
-    <xacro:property name="ns" value="${robot_namespace + '/' if robot_namespace != '' else ''}" />
+    <xacro:property name="robot_namespace_slash" value="${robot_namespace + '/' if robot_namespace != '' else ''}" />
     <joint name="${parent_link.rstrip('_link')}_to_${component_name}_joint" type="fixed">
       <origin xyz="${xyz}" rpy="${rpy}" />
@@ -108,7 +108,7 @@
     <xacro:gz_sensor.camera
       reference="${component_name}_link"
-      name="${ns}${component_name}_orbbec_astra_color"
-      topic="${ns}${component_name}/color/image_raw"
-      frame_id="${ns}${component_name}_color_optical_frame"
+      name="${robot_namespace_slash}${component_name}_orbbec_astra_color"
+      topic="${robot_namespace_slash}${component_name}/color/image_raw"
+      frame_id="${robot_namespace_slash}${component_name}_color_optical_frame"
       frequency="30"
       width="640"
@@ -117,7 +117,7 @@
     <xacro:gz_sensor.depth_camera
       reference="${component_name}_link"
-      name="${ns}${component_name}_orbbec_astra_depth"
-      topic="${ns}${component_name}/depth/image_raw"
-      frame_id="${ns}${component_name}_depth_optical_frame"
+      name="${robot_namespace_slash}${component_name}_orbbec_astra_depth"
+      topic="${robot_namespace_slash}${component_name}/depth/image_raw"
+      frame_id="${robot_namespace_slash}${component_name}_depth_optical_frame"
       frequency="30"
       width="640"

File: urdf/ouster.urdf.xacro (robot description, xacro)
@@ -56,13 +56,13 @@
       <xacro:property name="mesh" value="ouster_os01" scope="parent"/>
     </xacro:if>
-    <xacro:property name="ns" value="${robot_namespace + '/' if robot_namespace != '' else ''}" />
-    <xacro:property name="prefix" value="${component_name + '_' if component_name != '' else ''}" />
-    <xacro:property name="device_ns" value="${component_name + '/' if component_name != '' else ''}" />
-    <joint name="${parent_link.rstrip('_link')}_to_${prefix}ouster_${model}_joint" type="fixed">
+    <xacro:property name="robot_namespace_slash" value="${robot_namespace + '/' if robot_namespace != '' else ''}" />
+    <xacro:property name="component_name_underscore" value="${component_name + '_' if component_name != '' else ''}" />
+    <xacro:property name="component_name_slash" value="${component_name + '/' if component_name != '' else ''}" />
+    <joint name="${parent_link.rstrip('_link')}_to_${component_name_underscore}ouster_${model}_joint" type="fixed">
       <origin xyz="${xyz}" rpy="${rpy}" />
       <parent link="${parent_link}" />
-      <child link="${prefix}ouster_${model}_link" />
+      <child link="${component_name_underscore}ouster_${model}_link" />
     </joint>
-    <link name="${prefix}ouster_${model}_link">
+    <link name="${component_name_underscore}ouster_${model}_link">
       <!-- <visual>
         <origin xyz="0.0 0.0 0.0" rpy="0.0 0.0 0.0" />
@@ -95,14 +95,14 @@
       </inertial>
     </link>
-    <joint name="${prefix}ouster_${model}_to_${prefix}os_lidar_joint" type="fixed">
+    <joint name="${component_name_underscore}ouster_${model}_to_${component_name_underscore}os_lidar_joint" type="fixed">
       <origin xyz="0.0 0.0 0.03618" rpy="0.0 0.0 0.0" />
-      <parent link="${prefix}ouster_${model}_link" />
-      <child link="${prefix}os_lidar" />
+      <parent link="${component_name_underscore}ouster_${model}_link" />
+      <child link="${component_name_underscore}os_lidar" />
     </joint>
-    <link name="${prefix}os_lidar" />
-    <gazebo reference="${prefix}os_lidar">
+    <link name="${component_name_underscore}os_lidar" />
+    <gazebo reference="${component_name_underscore}os_lidar">
       <!-- gpu_lidar has to be set, CPU lidar doesn't work in ignition -
       https://github.com/gazebosim/gz-sensors/issues/26 -->
-      <sensor type="gpu_lidar" name="${ns}${prefix}ouster_${model}_sensor">
+      <sensor type="gpu_lidar" name="${robot_namespace_slash}${component_name_underscore}ouster_${model}_sensor">
         <visualize>false</visualize>
         <ray>
@@ -133,6 +133,6 @@
         </ray>
         <update_rate>20.0</update_rate>
-        <topic>${ns}${device_ns}ouster/points</topic>
-        <gz_frame_id>${ns}${prefix}os_lidar</gz_frame_id>
+        <topic>${robot_namespace_slash}${component_name_slash}ouster/points</topic>
+        <gz_frame_id>${robot_namespace_slash}${component_name_underscore}os_lidar</gz_frame_id>
         <always_on>true</always_on>
       </sensor>

File: urdf/robotiq.urdf.xacro (robot description, xacro)
@@ -22,7 +22,7 @@
       filename="$(find robotiq_description)/urdf/robotiq_${robotiq_type}_macro.urdf.xacro"
       ns="gripper" />
-    <xacro:property name="prefix" value="${component_name + '_' if component_name != '' else ''}" />
+    <xacro:property name="component_name_underscore" value="${component_name + '_' if component_name != '' else ''}" />
     <xacro:gripper.robotiq_gripper name="${component_name}robotiq_${robotiq_type}"
-      prefix="${prefix}"
+      prefix="${component_name_underscore}"
       parent="${parent_link}"
       use_fake_hardware="false"

File: urdf/slamtec_rplidar.urdf.xacro (robot description, xacro)
@@ -20,7 +20,7 @@
                        component_name:=''
                        model:=s3">
-    <xacro:property name="ns" value="${robot_namespace + '/' if robot_namespace != '' else ''}" />
-    <xacro:property name="prefix" value="${component_name + '_' if component_name != '' else ''}" />
-    <xacro:property name="device_ns" value="${component_name + '/' if component_name != '' else ''}" />
+    <xacro:property name="robot_namespace_slash" value="${robot_namespace + '/' if robot_namespace != '' else ''}" />
+    <xacro:property name="component_name_underscore" value="${component_name + '_' if component_name != '' else ''}" />
+    <xacro:property name="component_name_slash" value="${component_name + '/' if component_name != '' else ''}" />
     <xacro:if value="${model == 's3'}">
       <!-- Spec: https://www.slamtec.ai/wp-content/uploads/2023/11/SLAMTEC_rplidar_datasheet_S3_v1.0_en.pdf -->
@@ -196,10 +196,10 @@
       </xacro:property>
     </xacro:if>
-    <joint name="${parent_link.rstrip('_link')}_to_${prefix}slamtec_rplidar_joint" type="fixed">
+    <joint name="${parent_link.rstrip('_link')}_to_${component_name_underscore}slamtec_rplidar_joint" type="fixed">
       <origin xyz="${xyz}" rpy="${rpy}" />
       <parent link="${parent_link}" />
-      <child link="${prefix}slamtec_rplidar_link" />
+      <child link="${component_name_underscore}slamtec_rplidar_link" />
     </joint>
-    <link name="${prefix}slamtec_rplidar_link">
+    <link name="${component_name_underscore}slamtec_rplidar_link">
       <!-- <visual>
         <origin xyz="0.0 0.0 0.0" rpy="0.0 0.0 0.0" />
@@ -222,17 +222,17 @@
       </inertial>
     </link>
-    <joint name="${prefix}slamtec_rplidar_to_${prefix}laser_joint" type="fixed">
+    <joint name="${component_name_underscore}slamtec_rplidar_to_${component_name_underscore}laser_joint" type="fixed">
       <xacro:insert_block name="joint" />
-      <parent link="${prefix}slamtec_rplidar_link" />
-      <child link="${prefix}laser" />
+      <parent link="${component_name_underscore}slamtec_rplidar_link" />
+      <child link="${component_name_underscore}laser" />
     </joint>
-    <link name="${prefix}laser" />
-    <gazebo reference="${prefix}laser">
-      <sensor type="gpu_lidar" name="${ns}${prefix}slamtec_rplidar_sensor">
+    <link name="${component_name_underscore}laser" />
+    <gazebo reference="${component_name_underscore}laser">
+      <sensor type="gpu_lidar" name="${robot_namespace_slash}${component_name_underscore}slamtec_rplidar_sensor">
         <always_on>false</always_on>
         <update_rate>10</update_rate>
         <visualize>false</visualize>
-        <topic>${ns}${device_ns}scan</topic>
-        <gz_frame_id>${ns}${prefix}laser</gz_frame_id>
+        <topic>${robot_namespace_slash}${component_name_slash}scan</topic>
+        <gz_frame_id>${robot_namespace_slash}${component_name_underscore}laser</gz_frame_id>
         <ray>
           <scan>

File: urdf/stereolabs_zed.urdf.xacro (robot description, xacro)
@@ -23,5 +23,5 @@
                        robot_namespace:=''
                        component_name:=''">
-    <xacro:property name="ns" value="${robot_namespace + '/' if robot_namespace != '' else ''}" />
+    <xacro:property name="robot_namespace_slash" value="${robot_namespace + '/' if robot_namespace != '' else ''}" />
     <xacro:if value="${model == 'zed'}">
       <xacro:property name="baseline" value="0.12" />
@@ -303,7 +303,7 @@
     <xacro:gz_sensor.camera
       reference="${component_name}_camera_center"
-      name="${ns}${component_name}_stereolabs_zed_color"
-      topic="${ns}${component_name}/zed_node/rgb/image_rect_color"
-      frame_id="${ns}${component_name}_camera_center"
+      name="${robot_namespace_slash}${component_name}_stereolabs_zed_color"
+      topic="${robot_namespace_slash}${component_name}/zed_node/rgb/image_rect_color"
+      frame_id="${robot_namespace_slash}${component_name}_camera_center"
       frequency="30"
       width="1280"
@@ -312,7 +312,7 @@
     <xacro:gz_sensor.depth_camera
       reference="${component_name}_camera_center"
-      name="${ns}${component_name}_stereolabs_zed_depth"
-      topic="${ns}${component_name}/zed_node/depth"
-      frame_id="${ns}${component_name}_camera_center"
+      name="${robot_namespace_slash}${component_name}_stereolabs_zed_depth"
+      topic="${robot_namespace_slash}${component_name}/zed_node/depth"
+      frame_id="${robot_namespace_slash}${component_name}_camera_center"
       frequency="30"
       width="1280"

File: urdf/teltonika_003R-00253.urdf.xacro (robot description, xacro)
@@ -19,14 +19,14 @@
                        robot_namespace:=''
                        component_name:=''">
-    <xacro:property name="ns" value="${robot_namespace + '/' if robot_namespace != '' else ''}" />
-    <xacro:property name="prefix" value="${component_name + '_' if component_name != '' else ''}" />
-    <xacro:property name="device_ns" value="${component_name + '/' if component_name != '' else ''}" />
-    <joint name="${parent_link.rstrip('_link')}_to_${prefix}teltonika_mounting_joint"
+    <xacro:property name="robot_namespace_slash" value="${robot_namespace + '/' if robot_namespace != '' else ''}" />
+    <xacro:property name="component_name_underscore" value="${component_name + '_' if component_name != '' else ''}" />
+    <xacro:property name="component_name_slash" value="${component_name + '/' if component_name != '' else ''}" />
+    <joint name="${parent_link.rstrip('_link')}_to_${component_name_underscore}teltonika_mounting_joint"
       type="fixed">
       <origin xyz="${xyz}" rpy="${rpy}" />
       <parent link="${parent_link}" />
-      <child link="${prefix}teltonika_mounting_link" />
+      <child link="${component_name_underscore}teltonika_mounting_link" />
     </joint>
-    <link name="${prefix}teltonika_mounting_link">
+    <link name="${component_name_underscore}teltonika_mounting_link">
       <visual>
         <origin xyz="0.0 0.0 0.0" rpy="0.0 0.0 0.0" />
@@ -51,18 +51,18 @@
     </link>
     <joint
-      name="${prefix}teltonika_mounting_link_to_${prefix}teltonika_joint"
+      name="${component_name_underscore}teltonika_mounting_link_to_${component_name_underscore}teltonika_joint"
       type="fixed">
       <origin xyz="0.045 0.0 0.0058" rpy="0.0 0.0 0.0" />
-      <parent link="${prefix}teltonika_mounting_link" />
-      <child link="${prefix}teltonika" />
+      <parent link="${component_name_underscore}teltonika_mounting_link" />
+      <child link="${component_name_underscore}teltonika" />
     </joint>
-    <link name="${prefix}teltonika" />
-    <gazebo reference="${prefix}teltonika">
+    <link name="${component_name_underscore}teltonika" />
+    <gazebo reference="${component_name_underscore}teltonika">
       <sensor name="navsat" type="navsat">
         <plugin filename="ignition-gazebo-navsat-system" name="ignition::gazebo::systems::NavSat" />
         <always_on>1</always_on>
         <update_rate>1</update_rate>
-        <topic>${ns}${device_ns}fix</topic>
-        <gz_frame_id>${ns}${device_ns}teltonika</gz_frame_id>
+        <topic>${robot_namespace_slash}${component_name_slash}fix</topic>
+        <gz_frame_id>${robot_namespace_slash}${component_name_slash}teltonika</gz_frame_id>
       </sensor>
     </gazebo>

File: urdf/ur.urdf.xacro (robot description, xacro)
@@ -45,5 +45,5 @@
                        ur_type:=ur3e">
     <xacro:include filename="$(find ur_description)/urdf/ur_macro.xacro" ns="ur_manipulator" />
-    <xacro:property name="prefix" value="${component_name + '_' if component_name != '' else ''}" />
+    <xacro:property name="component_name_underscore" value="${component_name + '_' if component_name != '' else ''}" />
     <xacro:property name="joint_limit_params"
       value="$(find ur_description)/config/${ur_type}/joint_limits.yaml" scope="parent" />
@@ -61,5 +61,5 @@
     <xacro:ur_manipulator.ur_robot
       name="${ur_type}"
-      tf_prefix="${prefix}"
+      tf_prefix="${component_name_underscore}"
       parent="${parent_link}"
       joint_limits_parameters_file="${joint_limit_params}"
@@ -70,9 +70,9 @@
       <origin xyz="${xyz}" rpy="${rpy}" />
     </xacro:ur_manipulator.ur_robot>
-    <ros2_control name="${prefix + ur_type}" type="system">
+    <ros2_control name="${component_name_underscore}${ur_type}" type="system">
       <hardware>
         <plugin>gz_ros2_control/GazeboSimSystem</plugin>
       </hardware>
-      <joint name="${prefix}shoulder_pan_joint">
+      <joint name="${component_name_underscore}shoulder_pan_joint">
         <command_interface name="position">
           <param name="min">{-2*pi}</param>
@@ -90,5 +90,5 @@
         <state_interface name="effort" />
       </joint>
-      <joint name="${prefix}shoulder_lift_joint">
+      <joint name="${component_name_underscore}shoulder_lift_joint">
         <command_interface name="position">
           <param name="min">{-2*pi}</param>
@@ -106,5 +106,5 @@
         <state_interface name="effort" />
       </joint>
-      <joint name="${prefix}elbow_joint">
+      <joint name="${component_name_underscore}elbow_joint">
         <command_interface name="position">
           <param name="min">{-pi}</param>
@@ -122,5 +122,5 @@
         <state_interface name="effort" />
       </joint>
-      <joint name="${prefix}wrist_1_joint">
+      <joint name="${component_name_underscore}wrist_1_joint">
         <command_interface name="position">
           <param name="min">{-2*pi}</param>
@@ -138,5 +138,5 @@
         <state_interface name="effort" />
       </joint>
-      <joint name="${prefix}wrist_2_joint">
+      <joint name="${component_name_underscore}wrist_2_joint">
         <command_interface name="position">
           <param name="min">{-2*pi}</param>
@@ -154,5 +154,5 @@
         <state_interface name="effort" />
       </joint>
-      <joint name="${prefix}wrist_3_joint">
+      <joint name="${component_name_underscore}wrist_3_joint">
         <command_interface name="position">
           <param name="min">{-2*pi}</param>
