Commit message: macros: rename prefixes: ns -> robot_namespace_slash prefix -> component_name_underscore device_ns -> component_name_slash

File: urdf/velodyne_puck.urdf.xacro (robot description, xacro)
@@ -19,13 +19,13 @@
                        robot_namespace:=''
                        component_name:=''">
-    <xacro:property name="ns" value="${robot_namespace + '/' if robot_namespace != '' else ''}" />
-    <xacro:property name="prefix" value="${component_name + '_' if component_name != '' else ''}" />
-    <xacro:property name="device_ns" value="${component_name + '/' if component_name != '' else ''}" />
-    <joint name="${parent_link.rstrip('_link')}_to_${prefix}velodyne_puck_joint" type="fixed">
+    <xacro:property name="robot_namespace_slash" value="${robot_namespace + '/' if robot_namespace != '' else ''}" />
+    <xacro:property name="component_name_underscore" value="${component_name + '_' if component_name != '' else ''}" />
+    <xacro:property name="component_name_slash" value="${component_name + '/' if component_name != '' else ''}" />
+    <joint name="${parent_link.rstrip('_link')}_to_${component_name_underscore}velodyne_puck_joint" type="fixed">
       <origin xyz="${xyz}" rpy="${rpy}" />
       <parent link="${parent_link}" />
-      <child link="${prefix}velodyne_puck_link" />
+      <child link="${component_name_underscore}velodyne_puck_link" />
     </joint>
-    <link name="${prefix}velodyne_puck_link">
+    <link name="${component_name_underscore}velodyne_puck_link">
       <!-- <visual>
         <origin xyz="0.0 0.0 0.0" rpy="0.0 0.0 0.0" />
@@ -58,15 +58,15 @@
       </inertial>
     </link>
-    <joint name="${prefix}velodyne_puck_to_${prefix}velodyne_joint"
+    <joint name="${component_name_underscore}velodyne_puck_to_${component_name_underscore}velodyne_joint"
       type="fixed">
       <origin xyz="0.0 0.0 0.0378" rpy="0.0 0.0 0.0" />
-      <parent link="${prefix}velodyne_puck_link" />
-      <child link="${prefix}velodyne" />
+      <parent link="${component_name_underscore}velodyne_puck_link" />
+      <child link="${component_name_underscore}velodyne" />
     </joint>
-    <link name="${prefix}velodyne" />
-    <gazebo reference="${prefix}velodyne">
+    <link name="${component_name_underscore}velodyne" />
+    <gazebo reference="${component_name_underscore}velodyne">
       <!-- gpu_lidar has to be set, CPU lidar doesn't work in ignition -
       https://github.com/gazebosim/gz-sensors/issues/26 -->
-      <sensor type="gpu_lidar" name="${ns}${prefix}velodyne_puck_sensor">
+      <sensor type="gpu_lidar" name="${robot_namespace_slash}${component_name_underscore}velodyne_puck_sensor">
         <visualize>false</visualize>
         <update_rate>10.0</update_rate>
@@ -97,6 +97,6 @@
           </noise>
         </ray>
-        <topic>${ns}${device_ns}velodyne_points</topic>
-        <gz_frame_id>${ns}${prefix}velodyne</gz_frame_id>
+        <topic>${robot_namespace_slash}${component_name_slash}velodyne_points</topic>
+        <gz_frame_id>${robot_namespace_slash}${component_name_underscore}velodyne</gz_frame_id>
         <always_on>true</always_on>
       </sensor>

File: urdf/wibotic_receiver.urdf.xacro (robot description, xacro)
@@ -19,12 +19,12 @@
                        robot_namespace:=''
                        component_name:=''">
-    <xacro:property name="ns" value="${robot_namespace + '/' if robot_namespace != '' else ''}" />
-    <xacro:property name="prefix" value="${component_name + '_' if component_name != '' else ''}" />
-    <joint name="${parent_link.rstrip('_link')}_to_${prefix}wibotic_receiver_joint" type="fixed">
+    <xacro:property name="robot_namespace_slash" value="${robot_namespace + '/' if robot_namespace != '' else ''}" />
+    <xacro:property name="component_name_underscore" value="${component_name + '_' if component_name != '' else ''}" />
+    <joint name="${parent_link.rstrip('_link')}_to_${component_name_underscore}wibotic_receiver_joint" type="fixed">
       <origin xyz="${xyz}" rpy="${rpy}" />
       <parent link="${parent_link}" />
-      <child link="${prefix}wibotic_receiver_link" />
+      <child link="${component_name_underscore}wibotic_receiver_link" />
     </joint>
-    <link name="${prefix}wibotic_receiver_link">
+    <link name="${component_name_underscore}wibotic_receiver_link">
       <!-- <visual>
         <origin xyz="0.0 0.0 0.0" rpy="0.0 0.0 ${pi/2.0}" />

File: urdf/wibotic_station.urdf.xacro (robot description, xacro)
@@ -21,11 +21,11 @@
                        rpy:='0.0 0.0 0.0'
                        component_name:=''">
-    <xacro:property name="prefix" value="${component_name + '_' if component_name != '' else ''}" />
-    <joint name="${parent_link.rstrip('_link')}_to_${prefix}wibotic_station_joint" type="fixed">
+    <xacro:property name="component_name_underscore" value="${component_name + '_' if component_name != '' else ''}" />
+    <joint name="${parent_link.rstrip('_link')}_to_${component_name_underscore}wibotic_station_joint" type="fixed">
       <origin xyz="${xyz}" rpy="${rpy}" />
       <parent link="${parent_link}" />
-      <child link="${prefix}wibotic_station_link" />
+      <child link="${component_name_underscore}wibotic_station_link" />
     </joint>
-    <link name="${prefix}wibotic_station_link">
+    <link name="${component_name_underscore}wibotic_station_link">
       <!-- <visual>
         <origin xyz="0.0 0.0 0.0" rpy="0.0 0.0 ${pi/2.0}" />
@@ -60,17 +60,17 @@
       </inertial>
     </link>
-    <joint name="${prefix}wibotic_station_to_${prefix}wibotic_transmitter_joint" type="fixed">
+    <joint name="${component_name_underscore}wibotic_station_to_${component_name_underscore}wibotic_transmitter_joint" type="fixed">
       <!-- This should be when docking is released for panther-docker
       <origin xyz="0.05 0.0 0.295" rpy="0.0 0.0 ${pi}" /> -->
       <origin xyz="0.05 0.0 0.5" rpy="0.0 0.0 ${pi}" />
-      <parent link="${prefix}wibotic_station_link" />
-      <child link="${prefix}wibotic_transmitter_link" />
+      <parent link="${component_name_underscore}wibotic_station_link" />
+      <child link="${component_name_underscore}wibotic_transmitter_link" />
     </joint>
-    <link name="${prefix}wibotic_transmitter_link" />
+    <link name="${component_name_underscore}wibotic_transmitter_link" />
   </xacro:macro>
   <xacro:macro name="create_apriltag"
     params="name size:=$(arg apriltag_size) component_name:=''">
-    <xacro:property name="prefix" value="${component_name + '_' if component_name != '' else ''}" />
-    <link name="${prefix}${name}_link">
+    <xacro:property name="component_name_underscore" value="${component_name + '_' if component_name != '' else ''}" />
+    <link name="${component_name_underscore}${name}_link">
       <visual>
         <origin xyz="0 0 0" rpy="0 0 0" />
@@ -83,10 +83,10 @@
       </visual>
       </link>
-    <joint name="${name}_to_${name}_${prefix}image_link_joint" type="fixed">
+    <joint name="${name}_to_${name}_${component_name_underscore}image_link_joint" type="fixed">
       <origin xyz="0 0 0" rpy="0 -${pi/2.0} ${pi/2.0}" />
-      <parent link="${prefix}${name}_link" />
-      <child link="${prefix}${name}_image_link" />
+      <parent link="${component_name_underscore}${name}_link" />
+      <child link="${component_name_underscore}${name}_image_link" />
     </joint>
-    <link name="${prefix}${name}_image_link">
+    <link name="${component_name_underscore}${name}_image_link">
       <collision>
         <origin xyz="0 0 0" rpy="0 ${pi/2.0} 0" />
@@ -110,5 +110,5 @@
       </inertial>
     </link>
-    <gazebo reference="${prefix}${name}_image_link">
+    <gazebo reference="${component_name_underscore}${name}_image_link">
       <visual>
         <material>
@@ -128,5 +128,5 @@
     <xacro:property name="apriltag_size_prop" value="$(arg apriltag_size)" />
     <xacro:wibotic_station
-      component_name="$(arg component_name)" parent_link="${prefix}${name}_image_link"  xyz="0.0 0.0 0.5"
+      component_name="$(arg component_name)" parent_link="${component_name_underscore}${name}_image_link"  xyz="0.0 0.0 0.5"
       rpy="${pi} 0 0 " />
   </xacro:macro>
