Commit message: macros: replace the uses of ${robot_namespace}/ and ${component_name}_ or with / at the end

File: urdf/intel_realsense_d435.urdf.xacro (robot description, xacro)
@@ -22,4 +22,6 @@
                        component_name:=''">
     <xacro:property name="robot_namespace_slash" value="${robot_namespace + '/' if robot_namespace != '' else ''}" />
+    <xacro:property name="component_name_underscore" value="${component_name + '_' if component_name != '' else ''}" />
+    <xacro:property name="component_name_slash" value="${component_name + '/' if component_name != '' else ''}" />
     <!-- The following values are approximate, and the camera node
       publishing TF values with actual calibrated camera extrinsic values -->
@@ -41,17 +43,17 @@
     <xacro:property name="d435_cam_depth_pz" value="${d435_cam_height/2}" />
     <!-- camera body, with origin at bottom screw mount -->
-    <joint name="${parent_link.rstrip('_link')}_to_${component_name}_bottom_screw_joint" type="fixed">
+    <joint name="${parent_link.rstrip('_link')}_to_${component_name_underscore}bottom_screw_joint" type="fixed">
       <origin xyz="${xyz}" rpy="${rpy}" />
       <parent link="${parent_link}" />
-      <child link="${component_name}_bottom_screw_frame" />
+      <child link="${component_name_underscore}bottom_screw_frame" />
     </joint>
-    <link name="${component_name}_bottom_screw_frame" />
-    <joint name="${component_name}_bottom_screw_to_${component_name}_joint" type="fixed">
+    <link name="${component_name_underscore}bottom_screw_frame" />
+    <joint name="${component_name_underscore}bottom_screw_to_${component_name_underscore}joint" type="fixed">
       <origin xyz="0.0 ${d435_cam_depth_py} ${d435_cam_depth_pz}"
         rpy="0.0 0.0 0.0" />
-      <parent link="${component_name}_bottom_screw_frame" />
-      <child link="${component_name}_link" />
+      <parent link="${component_name_underscore}bottom_screw_frame" />
+      <child link="${component_name_underscore}link" />
     </joint>
-    <link name="${component_name}_link">
+    <link name="${component_name_underscore}link">
       <visual>
         <origin xyz="${d435_cam_mount_from_center_offset} ${-d435_cam_depth_py} 0.0" rpy="${pi/2.0} 0.0 ${pi/2.0}" />
@@ -79,55 +81,55 @@
     <xacro:if value="${use_nominal_extrinsics}">
       <!-- camera depth joints and links -->
-      <joint name="${component_name}_to_${component_name}_depth_joint" type="fixed">
+      <joint name="${component_name_underscore}to_${component_name_underscore}depth_joint" type="fixed">
         <origin xyz="0.0 0.0 0.0" rpy="0.0 0.0 0.0" />
-        <parent link="${component_name}_link" />
-        <child link="${component_name}_depth_frame" />
+        <parent link="${component_name_underscore}link" />
+        <child link="${component_name_underscore}depth_frame" />
       </joint>
-      <link name="${component_name}_depth_frame" />
-      <joint name="${component_name}_depth_to_${component_name}_depth_optical_joint" type="fixed">
+      <link name="${component_name_underscore}depth_frame" />
+      <joint name="${component_name_underscore}depth_to_${component_name_underscore}depth_optical_joint" type="fixed">
         <origin xyz="0.0 0.0 0.0" rpy="${-pi/2.0} 0.0 ${-pi/2.0}" />
-        <parent link="${component_name}_depth_frame" />
-        <child link="${component_name}_depth_optical_frame" />
+        <parent link="${component_name_underscore}depth_frame" />
+        <child link="${component_name_underscore}depth_optical_frame" />
       </joint>
-      <link name="${component_name}_depth_optical_frame" />
+      <link name="${component_name_underscore}depth_optical_frame" />
       <!-- camera left IR joints and links -->
-      <joint name="${component_name}_to_${component_name}_infra1_joint" type="fixed">
+      <joint name="${component_name_underscore}to_${component_name_underscore}infra1_joint" type="fixed">
         <origin xyz="0.0 ${d435_cam_depth_to_infra1_offset} 0.0" rpy="0.0 0.0 0.0" />
-        <parent link="${component_name}_link" />
-        <child link="${component_name}_infra1_frame" />
+        <parent link="${component_name_underscore}link" />
+        <child link="${component_name_underscore}infra1_frame" />
       </joint>
-      <link name="${component_name}_infra1_frame" />
-      <joint name="${component_name}_infra1_to_${component_name}_infra1_optical_joint" type="fixed">
+      <link name="${component_name_underscore}infra1_frame" />
+      <joint name="${component_name_underscore}infra1_to_${component_name_underscore}infra1_optical_joint" type="fixed">
         <origin xyz="0.0 0.0 0.0" rpy="${-pi/2.0} 0.0 ${-pi/2.0}" />
-        <parent link="${component_name}_infra1_frame" />
-        <child link="${component_name}_infra1_optical_frame" />
+        <parent link="${component_name_underscore}infra1_frame" />
+        <child link="${component_name_underscore}infra1_optical_frame" />
       </joint>
-      <link name="${component_name}_infra1_optical_frame" />
+      <link name="${component_name_underscore}infra1_optical_frame" />
       <!-- camera right IR joints and links -->
-      <joint name="${component_name}_to_${component_name}_infra2_joint" type="fixed">
+      <joint name="${component_name_underscore}to_${component_name_underscore}infra2_joint" type="fixed">
         <origin xyz="0.0 ${d435_cam_depth_to_infra2_offset} 0.0" rpy="0.0 0.0 0.0" />
-        <parent link="${component_name}_link" />
-        <child link="${component_name}_infra2_frame" />
+        <parent link="${component_name_underscore}link" />
+        <child link="${component_name_underscore}infra2_frame" />
       </joint>
-      <link name="${component_name}_infra2_frame" />
-      <joint name="${component_name}_infra2_to_${component_name}_infra2_optical_joint" type="fixed">
+      <link name="${component_name_underscore}infra2_frame" />
+      <joint name="${component_name_underscore}infra2_to_${component_name_underscore}infra2_optical_joint" type="fixed">
         <origin xyz="0.0 0.0 0.0" rpy="${-pi/2.0} 0.0 ${-pi/2.0}" />
-        <parent link="${component_name}_infra2_frame" />
-        <child link="${component_name}_infra2_optical_frame" />
+        <parent link="${component_name_underscore}infra2_frame" />
+        <child link="${component_name_underscore}infra2_optical_frame" />
       </joint>
-      <link name="${component_name}_infra2_optical_frame" />
+      <link name="${component_name_underscore}infra2_optical_frame" />
       <!-- camera color joints and links -->
-      <joint name="${component_name}_to_${component_name}_color_joint" type="fixed">
+      <joint name="${component_name_underscore}to_${component_name_underscore}color_joint" type="fixed">
         <origin xyz="0.0 ${d435_cam_depth_to_color_offset} 0.0" rpy="0.0 0.0 0.0" />
-        <parent link="${component_name}_link" />
-        <child link="${component_name}_color_frame" />
+        <parent link="${component_name_underscore}link" />
+        <child link="${component_name_underscore}color_frame" />
       </joint>
-      <link name="${component_name}_color_frame" />
-      <joint name="${component_name}_color_to_${component_name}_color_optical_joint" type="fixed">
+      <link name="${component_name_underscore}color_frame" />
+      <joint name="${component_name_underscore}color_to_${component_name_underscore}color_optical_joint" type="fixed">
         <origin xyz="0.0 0.0 0.0" rpy="${-pi/2.0} 0.0 ${-pi/2.0}" />
-        <parent link="${component_name}_color_frame" />
-        <child link="${component_name}_color_optical_frame" />
+        <parent link="${component_name_underscore}color_frame" />
+        <child link="${component_name_underscore}color_optical_frame" />
       </joint>
-      <link name="${component_name}_color_optical_frame" />
+      <link name="${component_name_underscore}color_optical_frame" />
     </xacro:if>
     <xacro:include filename="$(find husarion_components_description)/urdf/gz_sensor.urdf.xacro" ns="gz_sensor" />
@@ -136,8 +138,8 @@
     <!-- https://github.com/IntelRealSense/realsense-ros#published-topics -->
     <xacro:gz_sensor.camera
-      reference="${component_name}_link"
-      name="${robot_namespace_slash}${component_name}_intel_realsense_d435_color"
-      topic="${robot_namespace_slash}${component_name}/color/image_raw"
-      frame_id="${robot_namespace_slash}${component_name}_color_optical_frame"
+      reference="${component_name_underscore}link"
+      name="${robot_namespace_slash}${component_name_underscore}intel_realsense_d435_color"
+      topic="${robot_namespace_slash}${component_name_slash}color/image_raw"
+      frame_id="${robot_namespace_slash}${component_name_underscore}color_optical_frame"
       frequency="30"
       width="1280"
@@ -145,8 +147,8 @@
       fov="${69.0/180.0*pi}" />
     <xacro:gz_sensor.depth_camera
-      reference="${component_name}_link"
-      name="${robot_namespace_slash}${component_name}_intel_realsense_d435_depth"
-      topic="${robot_namespace_slash}${component_name}/depth/image_rect_raw"
-      frame_id="${robot_namespace_slash}${component_name}_depth_optical_frame"
+      reference="${component_name_underscore}link"
+      name="${robot_namespace_slash}${component_name_underscore}intel_realsense_d435_depth"
+      topic="${robot_namespace_slash}${component_name_slash}depth/image_rect_raw"
+      frame_id="${robot_namespace_slash}${component_name_underscore}depth_optical_frame"
       frequency="30"
       width="1280"

File: urdf/kinova.urdf.xacro (robot description, xacro)
@@ -54,4 +54,5 @@
     <xacro:property name="robot_namespace_slash" value="${robot_namespace + '/' if robot_namespace != '' else ''}" />
     <xacro:property name="component_name_underscore" value="${component_name + '_' if component_name != '' else ''}" />
+    <xacro:property name="component_name_slash" value="${component_name + '/' if component_name != '' else ''}" />
     <!-- robot name parameter -->
     <xacro:property name="robot_name" value="kinova_arm" />
@@ -126,6 +127,6 @@
     </xacro:unless>
     <xacro:if value="${vision}">
-      <gazebo reference="${component_name}_camera_color_frame">
-        <sensor name="${robot_namespace_slash}${component_name}_camera_sensor" type="rgbd_camera">
+      <gazebo reference="${component_name_underscore}camera_color_frame">
+        <sensor name="${robot_namespace_slash}${component_name_underscore}camera_sensor" type="rgbd_camera">
           <camera>
             <horizontal_fov>1.047</horizontal_fov>
@@ -177,11 +178,11 @@
               </clip>
             </depth_camera>
-            <optical_frame_id>${component_name}_color_optical_frame</optical_frame_id>
+            <optical_frame_id>${component_name_underscore}color_optical_frame</optical_frame_id>
           </camera>
-          <gz_frame_id>${component_name}_camera_color_frame</gz_frame_id>
+          <gz_frame_id>${component_name_underscore}camera_color_frame</gz_frame_id>
           <always_on>1</always_on>
           <update_rate>${camera_fps}</update_rate>
           <visualize>true</visualize>
-          <topic>${robot_namespace_slash}${component_name}/wrist_mounted_camera</topic>
+          <topic>${robot_namespace_slash}${component_name_slash}wrist_mounted_camera</topic>
           <enable_metrics>false</enable_metrics>
         </sensor>

File: urdf/luxonis_depthai.urdf.xacro (robot description, xacro)
@@ -23,4 +23,6 @@
     <xacro:include filename="$(find depthai_descriptions)/urdf/include/depthai_macro.urdf.xacro" />
     <xacro:property name="robot_namespace_slash" value="${robot_namespace + '/' if robot_namespace != '' else ''}" />
+    <xacro:property name="component_name_underscore" value="${component_name + '_' if component_name != '' else ''}" />
+    <xacro:property name="component_name_slash" value="${component_name + '/' if component_name != '' else ''}" />
     <xacro:depthai_camera camera_name="${component_name}" parent="${parent_link}"
       base_frame="${robot_namespace_slash}${component_name}" camera_model="${model}"
@@ -32,7 +34,7 @@
     <xacro:gz_sensor.camera
       reference="${robot_namespace_slash}${component_name}"
-      name="${robot_namespace_slash}${component_name}_color"
-      topic="${robot_namespace_slash}${component_name}/rgb/color"
-      frame_id="${robot_namespace_slash}${component_name}_rgb_camera_frame"
+      name="${robot_namespace_slash}${component_name_underscore}color"
+      topic="${robot_namespace_slash}${component_name_slash}rgb/color"
+      frame_id="${robot_namespace_slash}${component_name_underscore}rgb_camera_frame"
       frequency="30"
       width="1280"
@@ -41,7 +43,7 @@
     <xacro:gz_sensor.depth_camera
       reference="${robot_namespace_slash}${component_name}"
-      name="${robot_namespace_slash}${component_name}_depth"
-      topic="${robot_namespace_slash}${component_name}/stereo/depth"
-      frame_id="${robot_namespace_slash}${component_name}_rgb_camera_frame"
+      name="${robot_namespace_slash}${component_name_underscore}depth"
+      topic="${robot_namespace_slash}${component_name_slash}stereo/depth"
+      frame_id="${robot_namespace_slash}${component_name_underscore}rgb_camera_frame"
       frequency="30"
       width="1280"

File: urdf/orbbec_astra.urdf.xacro (robot description, xacro)
@@ -20,16 +20,18 @@
                        component_name:=''">
     <xacro:property name="robot_namespace_slash" value="${robot_namespace + '/' if robot_namespace != '' else ''}" />
-    <joint name="${parent_link.rstrip('_link')}_to_${component_name}_joint" type="fixed">
+    <xacro:property name="component_name_underscore" value="${component_name + '_' if component_name != '' else ''}" />
+    <xacro:property name="component_name_slash" value="${component_name + '/' if component_name != '' else ''}" />
+    <joint name="${parent_link.rstrip('_link')}_to_${component_name_underscore}joint" type="fixed">
       <origin xyz="${xyz}" rpy="${rpy}" />
       <parent link="${parent_link}" />
-      <child link="${component_name}_link" />
+      <child link="${component_name_underscore}link" />
     </joint>
-    <link name="${component_name}_link" />
-    <joint name="${parent_link.rstrip('_link')}_to_${component_name}_orbbec_astra_joint" type="fixed">
+    <link name="${component_name_underscore}link" />
+    <joint name="${parent_link.rstrip('_link')}_to_${component_name_underscore}orbbec_astra_joint" type="fixed">
       <origin xyz="${xyz}" rpy="${rpy}" />
       <parent link="${parent_link}" />
-      <child link="${component_name}_orbbec_astra_link" />
+      <child link="${component_name_underscore}orbbec_astra_link" />
     </joint>
-    <link name="${component_name}_orbbec_astra_link">
+    <link name="${component_name_underscore}orbbec_astra_link">
       <!-- <visual>
         <origin xyz="0.0 0.0 0.0" rpy="0.0 0.0 0.0" />
@@ -79,36 +81,36 @@
       </inertial>
     </link>
-    <joint name="${parent_link.rstrip('_link')}_to_${component_name}_color_joint" type="fixed">
+    <joint name="${parent_link.rstrip('_link')}_to_${component_name_underscore}color_joint" type="fixed">
       <origin xyz="-0.002 0.0125 0.03325" rpy="-0.003 0.0 -0.003" />
-      <parent link="${component_name}_link" />
-      <child link="${component_name}_color_frame" />
+      <parent link="${component_name_underscore}link" />
+      <child link="${component_name_underscore}color_frame" />
     </joint>
-    <link name="${component_name}_depth_frame" />
-    <joint name="${parent_link.rstrip('_link')}_to_${component_name}_depth_joint" type="fixed">
+    <link name="${component_name_underscore}depth_frame" />
+    <joint name="${parent_link.rstrip('_link')}_to_${component_name_underscore}depth_joint" type="fixed">
       <origin xyz="0.0 0.0 0.03325" rpy="0.0 0.0 0.0" />
-      <parent link="${component_name}_link" />
-      <child link="${component_name}_depth_frame" />
+      <parent link="${component_name_underscore}link" />
+      <child link="${component_name_underscore}depth_frame" />
     </joint>
-    <link name="${component_name}_color_frame" />
-    <joint name="${component_name}_color_to_${component_name}_color_optical_joint" type="fixed">
+    <link name="${component_name_underscore}color_frame" />
+    <joint name="${component_name_underscore}color_to_${component_name_underscore}color_optical_joint" type="fixed">
       <origin xyz="0.0 0.0 0.0" rpy="${-pi/2} 0.0 ${-pi/2}" />
-      <parent link="${component_name}_color_frame" />
-      <child link="${component_name}_color_optical_frame" />
+      <parent link="${component_name_underscore}color_frame" />
+      <child link="${component_name_underscore}color_optical_frame" />
     </joint>
-    <link name="${component_name}_depth_optical_frame" />
-    <joint name="${component_name}_depth_to_${component_name}_depth_optical_joint" type="fixed">
+    <link name="${component_name_underscore}depth_optical_frame" />
+    <joint name="${component_name_underscore}depth_to_${component_name_underscore}depth_optical_joint" type="fixed">
       <origin xyz="0.0 0.0 0.0" rpy="${-pi/2} 0.0 ${-pi/2}" />
-      <parent link="${component_name}_depth_frame" />
-      <child link="${component_name}_depth_optical_frame" />
+      <parent link="${component_name_underscore}depth_frame" />
+      <child link="${component_name_underscore}depth_optical_frame" />
     </joint>
-    <link name="${component_name}_color_optical_frame" />
+    <link name="${component_name_underscore}color_optical_frame" />
     <!-- GAZEBO -->
     <!-- https://github.com/orbbec/OrbbecSDK_ROS2#all-available-topics -->
     <xacro:include filename="$(find husarion_components_description)/urdf/gz_sensor.urdf.xacro" ns="gz_sensor" />
     <xacro:gz_sensor.camera
-      reference="${component_name}_link"
-      name="${robot_namespace_slash}${component_name}_orbbec_astra_color"
-      topic="${robot_namespace_slash}${component_name}/color/image_raw"
-      frame_id="${robot_namespace_slash}${component_name}_color_optical_frame"
+      reference="${component_name_underscore}link"
+      name="${robot_namespace_slash}${component_name_underscore}orbbec_astra_color"
+      topic="${robot_namespace_slash}${component_name_slash}color/image_raw"
+      frame_id="${robot_namespace_slash}${component_name_underscore}color_optical_frame"
       frequency="30"
       width="640"
@@ -116,8 +118,8 @@
       fov="${60.0/180.0*pi}" />
     <xacro:gz_sensor.depth_camera
-      reference="${component_name}_link"
-      name="${robot_namespace_slash}${component_name}_orbbec_astra_depth"
-      topic="${robot_namespace_slash}${component_name}/depth/image_raw"
-      frame_id="${robot_namespace_slash}${component_name}_depth_optical_frame"
+      reference="${component_name_underscore}link"
+      name="${robot_namespace_slash}${component_name_underscore}orbbec_astra_depth"
+      topic="${robot_namespace_slash}${component_name_slash}depth/image_raw"
+      frame_id="${robot_namespace_slash}${component_name_underscore}depth_optical_frame"
       frequency="30"
       width="640"
