Commit message: macros: replace the uses of ${robot_namespace}/ and ${component_name}_ or with / at the end

File: urdf/stereolabs_zed.urdf.xacro (robot description, xacro)
@@ -24,4 +24,6 @@
                        component_name:=''">
     <xacro:property name="robot_namespace_slash" value="${robot_namespace + '/' if robot_namespace != '' else ''}" />
+    <xacro:property name="component_name_underscore" value="${component_name + '_' if component_name != '' else ''}" />
+    <xacro:property name="component_name_slash" value="${component_name + '/' if component_name != '' else ''}" />
     <xacro:if value="${model == 'zed'}">
       <xacro:property name="baseline" value="0.12" />
@@ -160,12 +162,12 @@
     </xacro:if>
     <!-- Camera mounting point (the threaded screw hole in the bottom) -->
-    <link name="${component_name}_camera_link" />
-    <joint name="${component_name}_base_joint" type="fixed">
+    <link name="${component_name_underscore}camera_link" />
+    <joint name="${component_name_underscore}base_joint" type="fixed">
       <parent link="${parent_link}" />
-      <child link="${component_name}_camera_link" />
+      <child link="${component_name_underscore}camera_link" />
       <origin xyz="${xyz}" rpy="${rpy}" />
     </joint>
     <!-- Camera Center -->
-    <link name="${component_name}_camera_center">
+    <link name="${component_name_underscore}camera_center">
       <xacro:unless value="${model == 'virtual'}">
         <visual>
@@ -188,12 +190,12 @@
       </xacro:unless>
     </link>
-    <joint name="${component_name}_camera_center_joint" type="fixed">
-      <parent link="${component_name}_camera_link"/>
-      <child link="${component_name}_camera_center"/>
+    <joint name="${component_name_underscore}camera_center_joint" type="fixed">
+      <parent link="${component_name_underscore}camera_link"/>
+      <child link="${component_name_underscore}camera_center"/>
       <origin xyz="0 0 ${height/2}" rpy="0 ${bottom_slope} 0" />
     </joint>
     <xacro:unless value="${mono}">
       <!-- Left Camera -->
-      <link name="${component_name}_left_camera_frame">
+      <link name="${component_name_underscore}left_camera_frame">
         <xacro:if value="${model == 'virtual'}">
           <visual>
@@ -214,17 +216,17 @@
         </xacro:if>
       </link>
-      <joint name="${component_name}_left_camera_joint" type="fixed">
-        <parent link="${component_name}_camera_center"/>
-        <child link="${component_name}_left_camera_frame"/>
+      <joint name="${component_name_underscore}left_camera_joint" type="fixed">
+        <parent link="${component_name_underscore}camera_center"/>
+        <child link="${component_name_underscore}left_camera_frame"/>
         <origin xyz="${optical_offset_x} ${baseline/2} 0" rpy="0 0 0" />
       </joint>
-      <link name="${component_name}_left_camera_optical_frame"/>
-      <joint name="${component_name}_left_camera_optical_joint" type="fixed">
+      <link name="${component_name_underscore}left_camera_optical_frame"/>
+      <joint name="${component_name_underscore}left_camera_optical_joint" type="fixed">
         <origin xyz="0 0 0" rpy="-${M_PI/2} 0.0 -${M_PI/2}"/>
-        <parent link="${component_name}_left_camera_frame"/>
-        <child link="${component_name}_left_camera_optical_frame"/>
+        <parent link="${component_name_underscore}left_camera_frame"/>
+        <child link="${component_name_underscore}left_camera_optical_frame"/>
       </joint>
       <!-- Right Camera -->
-      <link name="${component_name}_right_camera_frame">
+      <link name="${component_name_underscore}right_camera_frame">
         <xacro:if value="${model == 'virtual'}">
           <visual>
@@ -245,39 +247,39 @@
         </xacro:if>
       </link>
-      <joint name="${component_name}_right_camera_joint" type="fixed">
-        <parent link="${component_name}_camera_center"/>
-        <child link="${component_name}_right_camera_frame"/>
+      <joint name="${component_name_underscore}right_camera_joint" type="fixed">
+        <parent link="${component_name_underscore}camera_center"/>
+        <child link="${component_name_underscore}right_camera_frame"/>
         <origin xyz="${optical_offset_x} -${baseline/2} 0" rpy="0 0 0" />
       </joint>
-      <link name="${component_name}_right_camera_optical_frame"/>
-      <joint name="${component_name}_right_camera_optical_joint" type="fixed">
+      <link name="${component_name_underscore}right_camera_optical_frame"/>
+      <joint name="${component_name_underscore}right_camera_optical_joint" type="fixed">
         <origin xyz="0 0 0" rpy="-${M_PI/2} 0.0 -${M_PI/2}"/>
-        <parent link="${component_name}_right_camera_frame"/>
-        <child link="${component_name}_right_camera_optical_frame"/>
+        <parent link="${component_name_underscore}right_camera_frame"/>
+        <child link="${component_name_underscore}right_camera_optical_frame"/>
       </joint>
       <!-- ZED2 Sensors -->
       <xacro:if value="${model == 'zed2'}">
-        <link name="${component_name}_mag_link" />
-        <joint name="${component_name}_mag_joint" type="fixed">
-          <parent link="${component_name}_camera_center"/>
-          <child link="${component_name}_mag_link"/>
+        <link name="${component_name_underscore}mag_link" />
+        <joint name="${component_name_underscore}mag_joint" type="fixed">
+          <parent link="${component_name_underscore}camera_center"/>
+          <child link="${component_name_underscore}mag_link"/>
           <origin xyz="0 0 0" rpy="0 0 0" />
         </joint>
-        <link name="${component_name}_baro_link" />
-        <joint name="${component_name}_baro_joint" type="fixed">
-          <parent link="${component_name}_camera_center"/>
-          <child link="${component_name}_baro_link"/>
+        <link name="${component_name_underscore}baro_link" />
+        <joint name="${component_name_underscore}baro_joint" type="fixed">
+          <parent link="${component_name_underscore}camera_center"/>
+          <child link="${component_name_underscore}baro_link"/>
           <origin xyz="0 0 0" rpy="0 0 0" />
         </joint>
-        <link name="${component_name}_temp_left_link" />
-        <joint name="${component_name}_temp_left_joint" type="fixed">
-          <parent link="${component_name}_left_camera_frame"/>
-          <child link="${component_name}_temp_left_link"/>
+        <link name="${component_name_underscore}temp_left_link" />
+        <joint name="${component_name_underscore}temp_left_joint" type="fixed">
+          <parent link="${component_name_underscore}left_camera_frame"/>
+          <child link="${component_name_underscore}temp_left_link"/>
           <origin xyz="0 0 0" rpy="0 0 0" />
         </joint>
-        <link name="${component_name}_temp_right_link" />
-        <joint name="${component_name}_temp_right_joint" type="fixed">
-          <parent link="${component_name}_right_camera_frame"/>
-          <child link="${component_name}_temp_right_link"/>
+        <link name="${component_name_underscore}temp_right_link" />
+        <joint name="${component_name_underscore}temp_right_joint" type="fixed">
+          <parent link="${component_name_underscore}right_camera_frame"/>
+          <child link="${component_name_underscore}temp_right_link"/>
           <origin xyz="0 0 0" rpy="0 0 0" />
         </joint>
@@ -286,15 +288,15 @@
     <xacro:if value="${mono}">
       <!-- Camera -->
-      <link name="${component_name}_camera_frame" />
-      <joint name="${component_name}_camera_joint" type="fixed">
-        <parent link="${component_name}_camera_center"/>
-        <child link="${component_name}_camera_frame"/>
+      <link name="${component_name_underscore}camera_frame" />
+      <joint name="${component_name_underscore}camera_joint" type="fixed">
+        <parent link="${component_name_underscore}camera_center"/>
+        <child link="${component_name_underscore}camera_frame"/>
         <origin xyz="${optical_offset_x} 0 0" rpy="0 0 0" />
       </joint>
-      <link name="${component_name}_camera_optical_frame"/>
-      <joint name="${component_name}_camera_optical_joint" type="fixed">
+      <link name="${component_name_underscore}camera_optical_frame"/>
+      <joint name="${component_name_underscore}camera_optical_joint" type="fixed">
         <origin xyz="0 0 0" rpy="-${M_PI/2} 0.0 -${M_PI/2}"/>
-        <parent link="${component_name}_camera_frame"/>
-        <child link="${component_name}_camera_optical_frame"/>
+        <parent link="${component_name_underscore}camera_frame"/>
+        <child link="${component_name_underscore}camera_optical_frame"/>
       </joint>
     </xacro:if>
@@ -302,8 +304,8 @@
     <xacro:include filename="$(find husarion_components_description)/urdf/gz_sensor.urdf.xacro" ns="gz_sensor" />
     <xacro:gz_sensor.camera
-      reference="${component_name}_camera_center"
-      name="${robot_namespace_slash}${component_name}_stereolabs_zed_color"
-      topic="${robot_namespace_slash}${component_name}/zed_node/rgb/image_rect_color"
-      frame_id="${robot_namespace_slash}${component_name}_camera_center"
+      reference="${component_name_underscore}camera_center"
+      name="${robot_namespace_slash}${component_name_underscore}stereolabs_zed_color"
+      topic="${robot_namespace_slash}${component_name_slash}zed_node/rgb/image_rect_color"
+      frame_id="${robot_namespace_slash}${component_name_underscore}camera_center"
       frequency="30"
       width="1280"
@@ -311,8 +313,8 @@
       fov="${110.0/180.0*pi}" />
     <xacro:gz_sensor.depth_camera
-      reference="${component_name}_camera_center"
-      name="${robot_namespace_slash}${component_name}_stereolabs_zed_depth"
-      topic="${robot_namespace_slash}${component_name}/zed_node/depth"
-      frame_id="${robot_namespace_slash}${component_name}_camera_center"
+      reference="${component_name_underscore}camera_center"
+      name="${robot_namespace_slash}${component_name_underscore}stereolabs_zed_depth"
+      topic="${robot_namespace_slash}${component_name_slash}zed_node/depth"
+      frame_id="${robot_namespace_slash}${component_name_underscore}camera_center"
       frequency="30"
       width="1280"

Commit message: macros: add default component names

File: urdf/intel_realsense_d435.urdf.xacro (robot description, xacro)
@@ -21,4 +21,7 @@
                        robot_namespace:=''
                        component_name:=''">
+    <xacro:if value="${component_name == ''}">
+      <xacro:property name="component_name" value="d435" />
+    </xacro:if>
     <xacro:property name="robot_namespace_slash" value="${robot_namespace + '/' if robot_namespace != '' else ''}" />
     <xacro:property name="component_name_underscore" value="${component_name + '_' if component_name != '' else ''}" />

File: urdf/kinova.urdf.xacro (robot description, xacro)
@@ -48,11 +48,14 @@
                        robot_namespace:=''
                        component_name:=''">
+    <xacro:if value="${component_name == ''}">
+      <xacro:property name="component_name" value="kinova" />
+    </xacro:if>
+    <xacro:property name="robot_namespace_slash" value="${robot_namespace + '/' if robot_namespace != '' else ''}" />
+    <xacro:property name="component_name_underscore" value="${component_name + '_' if component_name != '' else ''}" />
+    <xacro:property name="component_name_slash" value="${component_name + '/' if component_name != '' else ''}" />
     <xacro:include
       filename="$(find kortex_description)/robots/kortex_robot.xacro"
       ns="kinova_manipulator"
     />
-    <xacro:property name="robot_namespace_slash" value="${robot_namespace + '/' if robot_namespace != '' else ''}" />
-    <xacro:property name="component_name_underscore" value="${component_name + '_' if component_name != '' else ''}" />
-    <xacro:property name="component_name_slash" value="${component_name + '/' if component_name != '' else ''}" />
     <!-- robot name parameter -->
     <xacro:property name="robot_name" value="kinova_arm" />

File: urdf/luxonis_depthai.urdf.xacro (robot description, xacro)
@@ -21,8 +21,11 @@
                        model:='OAK-D-PRO'
                        use_sim:=False">
-    <xacro:include filename="$(find depthai_descriptions)/urdf/include/depthai_macro.urdf.xacro" />
+    <xacro:if value="${component_name == ''}">
+      <xacro:property name="component_name" value="oak" />
+    </xacro:if>
     <xacro:property name="robot_namespace_slash" value="${robot_namespace + '/' if robot_namespace != '' else ''}" />
     <xacro:property name="component_name_underscore" value="${component_name + '_' if component_name != '' else ''}" />
     <xacro:property name="component_name_slash" value="${component_name + '/' if component_name != '' else ''}" />
+    <xacro:include filename="$(find depthai_descriptions)/urdf/include/depthai_macro.urdf.xacro" />
     <xacro:depthai_camera camera_name="${component_name}" parent="${parent_link}"
       base_frame="${robot_namespace_slash}${component_name}" camera_model="${model}"

File: urdf/orbbec_astra.urdf.xacro (robot description, xacro)
@@ -19,4 +19,7 @@
                        robot_namespace:=''
                        component_name:=''">
+    <xacro:if value="${component_name == ''}">
+      <xacro:property name="component_name" value="astra" />
+    </xacro:if>
     <xacro:property name="robot_namespace_slash" value="${robot_namespace + '/' if robot_namespace != '' else ''}" />
     <xacro:property name="component_name_underscore" value="${component_name + '_' if component_name != '' else ''}" />

File: urdf/ouster.urdf.xacro (robot description, xacro)
@@ -20,4 +20,10 @@
                        robot_namespace:=''
                        component_name:=''">
+    <xacro:if value="${component_name == ''}">
+      <xacro:property name="component_name" value="ouster" />
+    </xacro:if>
+    <xacro:property name="robot_namespace_slash" value="${robot_namespace + '/' if robot_namespace != '' else ''}" />
+    <xacro:property name="component_name_underscore" value="${component_name + '_' if component_name != '' else ''}" />
+    <xacro:property name="component_name_slash" value="${component_name + '/' if component_name != '' else ''}" />
     <xacro:if value="${model == 'os0_32'}">
       <xacro:property name="vfov" value="${radians(90.0)}" scope="parent" />
@@ -56,7 +62,4 @@
       <xacro:property name="mesh" value="ouster_os01" scope="parent"/>
     </xacro:if>
-    <xacro:property name="robot_namespace_slash" value="${robot_namespace + '/' if robot_namespace != '' else ''}" />
-    <xacro:property name="component_name_underscore" value="${component_name + '_' if component_name != '' else ''}" />
-    <xacro:property name="component_name_slash" value="${component_name + '/' if component_name != '' else ''}" />
     <joint name="${parent_link.rstrip('_link')}_to_${component_name_underscore}ouster_${model}_joint" type="fixed">
       <origin xyz="${xyz}" rpy="${rpy}" />

File: urdf/robotiq.urdf.xacro (robot description, xacro)
@@ -19,8 +19,11 @@
                        robotiq_type:=2f_85
                        component_name:=''">
+    <xacro:if value="${component_name == ''}">
+      <xacro:property name="component_name" value="robotiq" />
+    </xacro:if>
+    <xacro:property name="component_name_underscore" value="${component_name + '_' if component_name != '' else ''}" />
     <xacro:include
       filename="$(find robotiq_description)/urdf/robotiq_${robotiq_type}_macro.urdf.xacro"
       ns="gripper" />
-    <xacro:property name="component_name_underscore" value="${component_name + '_' if component_name != '' else ''}" />
     <xacro:gripper.robotiq_gripper name="${component_name}robotiq_${robotiq_type}"
       prefix="${component_name_underscore}"

File: urdf/slamtec_rplidar.urdf.xacro (robot description, xacro)
@@ -20,4 +20,7 @@
                        component_name:=''
                        model:=s3">
+    <xacro:if value="${component_name == ''}">
+      <xacro:property name="component_name" value="rplidar" />
+    </xacro:if>
     <xacro:property name="robot_namespace_slash" value="${robot_namespace + '/' if robot_namespace != '' else ''}" />
     <xacro:property name="component_name_underscore" value="${component_name + '_' if component_name != '' else ''}" />

File: urdf/stereolabs_zed.urdf.xacro (robot description, xacro)
@@ -23,4 +23,7 @@
                        robot_namespace:=''
                        component_name:=''">
+    <xacro:if value="${component_name == ''}">
+      <xacro:property name="component_name" value="zed" />
+    </xacro:if>
     <xacro:property name="robot_namespace_slash" value="${robot_namespace + '/' if robot_namespace != '' else ''}" />
     <xacro:property name="component_name_underscore" value="${component_name + '_' if component_name != '' else ''}" />

File: urdf/teltonika_003R-00253.urdf.xacro (robot description, xacro)
@@ -19,4 +19,7 @@
                        robot_namespace:=''
                        component_name:=''">
+    <xacro:if value="${component_name == ''}">
+      <xacro:property name="component_name" value="teltonika" />
+    </xacro:if>
     <xacro:property name="robot_namespace_slash" value="${robot_namespace + '/' if robot_namespace != '' else ''}" />
     <xacro:property name="component_name_underscore" value="${component_name + '_' if component_name != '' else ''}" />

File: urdf/ur.urdf.xacro (robot description, xacro)
@@ -44,6 +44,9 @@
                        component_name:=''
                        ur_type:=ur3e">
+    <xacro:if value="${component_name == ''}">
+      <xacro:property name="component_name" value="ur" />
+    </xacro:if>
+    <xacro:property name="component_name_underscore" value="${component_name + '_' if component_name != '' else ''}" />
     <xacro:include filename="$(find ur_description)/urdf/ur_macro.xacro" ns="ur_manipulator" />
-    <xacro:property name="component_name_underscore" value="${component_name + '_' if component_name != '' else ''}" />
     <xacro:property name="joint_limit_params"
       value="$(find ur_description)/config/${ur_type}/joint_limits.yaml" scope="parent" />

File: urdf/velodyne_puck.urdf.xacro (robot description, xacro)
@@ -19,4 +19,7 @@
                        robot_namespace:=''
                        component_name:=''">
+    <xacro:if value="${component_name == ''}">
+      <xacro:property name="component_name" value="velodyne" />
+    </xacro:if>
     <xacro:property name="robot_namespace_slash" value="${robot_namespace + '/' if robot_namespace != '' else ''}" />
     <xacro:property name="component_name_underscore" value="${component_name + '_' if component_name != '' else ''}" />

File: urdf/wibotic_receiver.urdf.xacro (robot description, xacro)
@@ -19,4 +19,7 @@
                        robot_namespace:=''
                        component_name:=''">
+    <xacro:if value="${component_name == ''}">
+      <xacro:property name="component_name" value="wibotic_receiver" />
+    </xacro:if>
     <xacro:property name="robot_namespace_slash" value="${robot_namespace + '/' if robot_namespace != '' else ''}" />
     <xacro:property name="component_name_underscore" value="${component_name + '_' if component_name != '' else ''}" />

File: urdf/wibotic_station.urdf.xacro (robot description, xacro)
@@ -21,4 +21,7 @@
                        rpy:='0.0 0.0 0.0'
                        component_name:=''">
+    <xacro:if value="${component_name == ''}">
+      <xacro:property name="component_name" value="wibotic_station" />
+    </xacro:if>
     <xacro:property name="component_name_underscore" value="${component_name + '_' if component_name != '' else ''}" />
     <joint name="${parent_link.rstrip('_link')}_to_${component_name_underscore}wibotic_station_joint" type="fixed">

Commit message: urdfs: set default d435 and astra names to "camera"

File: urdf/intel_realsense_d435.urdf.xacro (robot description, xacro)
@@ -22,5 +22,5 @@
                        component_name:=''">
     <xacro:if value="${component_name == ''}">
-      <xacro:property name="component_name" value="d435" />
+      <xacro:property name="component_name" value="camera" />
     </xacro:if>
     <xacro:property name="robot_namespace_slash" value="${robot_namespace + '/' if robot_namespace != '' else ''}" />

File: urdf/orbbec_astra.urdf.xacro (robot description, xacro)
@@ -20,5 +20,5 @@
                        component_name:=''">
     <xacro:if value="${component_name == ''}">
-      <xacro:property name="component_name" value="astra" />
+      <xacro:property name="component_name" value="camera" />
     </xacro:if>
     <xacro:property name="robot_namespace_slash" value="${robot_namespace + '/' if robot_namespace != '' else ''}" />
