Commit message: velodyne: remove default component name

File: urdf/velodyne_puck.urdf.xacro (robot description, xacro)
@@ -19,16 +19,19 @@
                        robot_namespace:=''
                        component_name:=''">
-    <xacro:if value="${component_name == ''}">
+    <!-- <xacro:if value="${component_name == ''}">
       <xacro:property name="component_name" value="velodyne" />
-    </xacro:if>
+    </xacro:if> -->
+    <!-- ^ removed for compatibility with hw driver -->
     <xacro:property name="robot_namespace_slash" value="${robot_namespace + '/' if robot_namespace != '' else ''}" />
     <xacro:property name="component_name_underscore" value="${component_name + '_' if component_name != '' else ''}" />
     <xacro:property name="component_name_slash" value="${component_name + '/' if component_name != '' else ''}" />
-    <joint name="${parent_link.rstrip('_link')}_to_${component_name_underscore}joint" type="fixed">
+    <xacro:property name="component_name_underscore_nonempty" value="${component_name_underscore if component_name_underscore != '' else 'velodyne_'}" />
+    <!-- ^ in case no name is provided, generate "..._link" instead of just "link" -->
+    <joint name="${parent_link.rstrip('_link')}_to_${component_name_underscore_nonempty}joint" type="fixed">
       <origin xyz="${xyz}" rpy="${rpy}" />
       <parent link="${parent_link}" />
-      <child link="${component_name_underscore}link" />
+      <child link="${component_name_underscore_nonempty}link" />
     </joint>
-    <link name="${component_name_underscore}link">
+    <link name="${component_name_underscore_nonempty}link">
       <!-- <visual>
         <origin xyz="0.0 0.0 0.0" rpy="0.0 0.0 0.0" />
@@ -61,8 +64,8 @@
       </inertial>
     </link>
-    <joint name="${component_name_underscore}to_${component_name_underscore}velodyne_joint"
+    <joint name="${component_name_underscore_nonempty}to_${component_name_underscore}velodyne_joint"
       type="fixed">
       <origin xyz="0.0 0.0 0.0378" rpy="0.0 0.0 0.0" />
-      <parent link="${component_name_underscore}link" />
+      <parent link="${component_name_underscore_nonempty}link" />
       <child link="${component_name_underscore}velodyne" />
     </joint>
