Commit message: REVIEWME: standarize frame names

File: urdf/luxonis_depthai.urdf.xacro (robot description, xacro)
@@ -29,5 +29,5 @@
     <xacro:include filename="$(find depthai_descriptions)/urdf/include/depthai_macro.urdf.xacro" />
     <xacro:depthai_camera camera_name="${component_name}" parent="${parent_link}"
-      base_frame="${robot_namespace_slash}${component_name}" camera_model="${model}"
+      base_frame="${robot_namespace_slash}${component_name_underscore}link" camera_model="${model}"
       cam_pos_x="${xyz.split()[0]}" cam_pos_y="${xyz.split()[1]}" cam_pos_z="${xyz.split()[2]}"
       cam_roll="${rpy.split()[0]}" cam_pitch="${rpy.split()[1]}" cam_yaw="${rpy.split()[2]}"
@@ -36,5 +36,5 @@
       ns="gz_sensor" />
     <xacro:gz_sensor.camera
-      reference="${robot_namespace_slash}${component_name}"
+      reference="${component_name_underscore}link"
       name="${robot_namespace_slash}${component_name_underscore}color"
       topic="${robot_namespace_slash}${component_name_slash}rgb/color"
@@ -45,5 +45,5 @@
       fov="${60.0/180.0*pi}" />
     <xacro:gz_sensor.depth_camera
-      reference="${robot_namespace_slash}${component_name}"
+      reference="${component_name_underscore}link"
       name="${robot_namespace_slash}${component_name_underscore}depth"
       topic="${robot_namespace_slash}${component_name_slash}stereo/depth"

File: urdf/orbbec_astra.urdf.xacro (robot description, xacro)
@@ -31,10 +31,10 @@
     </joint>
     <link name="${component_name_underscore}link" />
-    <joint name="${parent_link.rstrip('_link')}_to_${component_name_underscore}orbbec_astra_joint" type="fixed">
+    <joint name="${parent_link.rstrip('_link')}_to_${component_name_underscore}astra_visual_joint" type="fixed">
       <origin xyz="${xyz}" rpy="${rpy}" />
       <parent link="${parent_link}" />
-      <child link="${component_name_underscore}orbbec_astra_link" />
+      <child link="${component_name_underscore}astra_visual_frame" />
     </joint>
-    <link name="${component_name_underscore}orbbec_astra_link">
+    <link name="${component_name_underscore}astra_visual_frame">
       <!-- <visual>
         <origin xyz="0.0 0.0 0.0" rpy="0.0 0.0 0.0" />
@@ -84,5 +84,5 @@
       </inertial>
     </link>
-    <joint name="${parent_link.rstrip('_link')}_to_${component_name_underscore}color_joint" type="fixed">
+    <joint name="${component_name_underscore}to_${component_name_underscore}color_joint" type="fixed">
       <origin xyz="-0.002 0.0125 0.03325" rpy="-0.003 0.0 -0.003" />
       <parent link="${component_name_underscore}link" />
@@ -90,5 +90,5 @@
     </joint>
     <link name="${component_name_underscore}depth_frame" />
-    <joint name="${parent_link.rstrip('_link')}_to_${component_name_underscore}depth_joint" type="fixed">
+    <joint name="${component_name_underscore}to_${component_name_underscore}depth_joint" type="fixed">
       <origin xyz="0.0 0.0 0.03325" rpy="0.0 0.0 0.0" />
       <parent link="${component_name_underscore}link" />

File: urdf/ouster.urdf.xacro (robot description, xacro)
@@ -62,10 +62,10 @@
       <xacro:property name="mesh" value="ouster_os01" scope="parent"/>
     </xacro:if>
-    <joint name="${parent_link.rstrip('_link')}_to_${component_name_underscore}ouster_${model}_joint" type="fixed">
+    <joint name="${parent_link.rstrip('_link')}_to_${component_name_underscore}joint" type="fixed">
       <origin xyz="${xyz}" rpy="${rpy}" />
       <parent link="${parent_link}" />
-      <child link="${component_name_underscore}ouster_${model}_link" />
+      <child link="${component_name_underscore}link" />
     </joint>
-    <link name="${component_name_underscore}ouster_${model}_link">
+    <link name="${component_name_underscore}link">
       <!-- <visual>
         <origin xyz="0.0 0.0 0.0" rpy="0.0 0.0 0.0" />
@@ -98,14 +98,14 @@
       </inertial>
     </link>
-    <joint name="${component_name_underscore}ouster_${model}_to_${component_name_underscore}os_lidar_joint" type="fixed">
+    <joint name="${component_name_underscore}to_${component_name_underscore}lidar_joint" type="fixed">
       <origin xyz="0.0 0.0 0.03618" rpy="0.0 0.0 0.0" />
-      <parent link="${component_name_underscore}ouster_${model}_link" />
-      <child link="${component_name_underscore}os_lidar" />
+      <parent link="${component_name_underscore}link" />
+      <child link="${component_name_underscore}lidar_frame" />
     </joint>
-    <link name="${component_name_underscore}os_lidar" />
-    <gazebo reference="${component_name_underscore}os_lidar">
+    <link name="${component_name_underscore}lidar_frame" />
+    <gazebo reference="${component_name_underscore}lidar_frame">
       <!-- gpu_lidar has to be set, CPU lidar doesn't work in ignition -
       https://github.com/gazebosim/gz-sensors/issues/26 -->
-      <sensor type="gpu_lidar" name="${robot_namespace_slash}${component_name_underscore}ouster_${model}_sensor">
+      <sensor type="gpu_lidar" name="${robot_namespace_slash}${component_name_underscore}lidar">
         <visualize>false</visualize>
         <ray>
@@ -137,5 +137,5 @@
         <update_rate>20.0</update_rate>
         <topic>${robot_namespace_slash}${component_name_slash}ouster/points</topic>
-        <gz_frame_id>${robot_namespace_slash}${component_name_underscore}os_lidar</gz_frame_id>
+        <gz_frame_id>${robot_namespace_slash}${component_name_underscore}lidar_frame</gz_frame_id>
         <always_on>true</always_on>
       </sensor>

File: urdf/robotiq.urdf.xacro (robot description, xacro)
@@ -26,5 +26,5 @@
       filename="$(find robotiq_description)/urdf/robotiq_${robotiq_type}_macro.urdf.xacro"
       ns="gripper" />
-    <xacro:gripper.robotiq_gripper name="${component_name}robotiq_${robotiq_type}"
+    <xacro:gripper.robotiq_gripper name="${component_name_underscore}robotiq_${robotiq_type}"
       prefix="${component_name_underscore}"
       parent="${parent_link}"

File: urdf/slamtec_rplidar.urdf.xacro (robot description, xacro)
@@ -199,10 +199,10 @@
       </xacro:property>
     </xacro:if>
-    <joint name="${parent_link.rstrip('_link')}_to_${component_name_underscore}slamtec_rplidar_joint" type="fixed">
+    <joint name="${parent_link.rstrip('_link')}_to_${component_name_underscore}joint" type="fixed">
       <origin xyz="${xyz}" rpy="${rpy}" />
       <parent link="${parent_link}" />
-      <child link="${component_name_underscore}slamtec_rplidar_link" />
+      <child link="${component_name_underscore}link" />
     </joint>
-    <link name="${component_name_underscore}slamtec_rplidar_link">
+    <link name="${component_name_underscore}link">
       <!-- <visual>
         <origin xyz="0.0 0.0 0.0" rpy="0.0 0.0 0.0" />
@@ -225,17 +225,17 @@
       </inertial>
     </link>
-    <joint name="${component_name_underscore}slamtec_rplidar_to_${component_name_underscore}laser_joint" type="fixed">
+    <joint name="${component_name_underscore}to_${component_name_underscore}laser_joint" type="fixed">
       <xacro:insert_block name="joint" />
-      <parent link="${component_name_underscore}slamtec_rplidar_link" />
-      <child link="${component_name_underscore}laser" />
+      <parent link="${component_name_underscore}link" />
+      <child link="${component_name_underscore}laser_frame" />
     </joint>
-    <link name="${component_name_underscore}laser" />
-    <gazebo reference="${component_name_underscore}laser">
-      <sensor type="gpu_lidar" name="${robot_namespace_slash}${component_name_underscore}slamtec_rplidar_sensor">
+    <link name="${component_name_underscore}laser_frame" />
+    <gazebo reference="${component_name_underscore}laser_frame">
+      <sensor type="gpu_lidar" name="${robot_namespace_slash}${component_name_underscore}lidar">
         <always_on>false</always_on>
         <update_rate>10</update_rate>
         <visualize>false</visualize>
         <topic>${robot_namespace_slash}${component_name_slash}scan</topic>
-        <gz_frame_id>${robot_namespace_slash}${component_name_underscore}laser</gz_frame_id>
+        <gz_frame_id>${robot_namespace_slash}${component_name_underscore}laser_frame</gz_frame_id>
         <ray>
           <scan>

File: urdf/stereolabs_zed.urdf.xacro (robot description, xacro)
@@ -165,12 +165,12 @@
     </xacro:if>
     <!-- Camera mounting point (the threaded screw hole in the bottom) -->
-    <link name="${component_name_underscore}camera_link" />
-    <joint name="${component_name_underscore}base_joint" type="fixed">
+    <link name="${component_name_underscore}link" />
+    <joint name="${parent_link.rstrip('_link')}_to_${component_name_underscore}joint" type="fixed">
       <parent link="${parent_link}" />
-      <child link="${component_name_underscore}camera_link" />
+      <child link="${component_name_underscore}link" />
       <origin xyz="${xyz}" rpy="${rpy}" />
     </joint>
     <!-- Camera Center -->
-    <link name="${component_name_underscore}camera_center">
+    <link name="${component_name_underscore}camera_center_frame">
       <xacro:unless value="${model == 'virtual'}">
         <visual>
@@ -193,7 +193,7 @@
       </xacro:unless>
     </link>
-    <joint name="${component_name_underscore}camera_center_joint" type="fixed">
-      <parent link="${component_name_underscore}camera_link"/>
-      <child link="${component_name_underscore}camera_center"/>
+    <joint name="${component_name_underscore}to_${component_name_underscore}camera_center_joint" type="fixed">
+      <parent link="${component_name_underscore}link"/>
+      <child link="${component_name_underscore}camera_center_frame"/>
       <origin xyz="0 0 ${height/2}" rpy="0 ${bottom_slope} 0" />
     </joint>
@@ -220,5 +220,5 @@
       </link>
       <joint name="${component_name_underscore}left_camera_joint" type="fixed">
-        <parent link="${component_name_underscore}camera_center"/>
+        <parent link="${component_name_underscore}camera_center_frame"/>
         <child link="${component_name_underscore}left_camera_frame"/>
         <origin xyz="${optical_offset_x} ${baseline/2} 0" rpy="0 0 0" />
@@ -251,5 +251,5 @@
       </link>
       <joint name="${component_name_underscore}right_camera_joint" type="fixed">
-        <parent link="${component_name_underscore}camera_center"/>
+        <parent link="${component_name_underscore}camera_center_frame"/>
         <child link="${component_name_underscore}right_camera_frame"/>
         <origin xyz="${optical_offset_x} -${baseline/2} 0" rpy="0 0 0" />
@@ -265,5 +265,5 @@
         <link name="${component_name_underscore}mag_link" />
         <joint name="${component_name_underscore}mag_joint" type="fixed">
-          <parent link="${component_name_underscore}camera_center"/>
+          <parent link="${component_name_underscore}camera_center_frame"/>
           <child link="${component_name_underscore}mag_link"/>
           <origin xyz="0 0 0" rpy="0 0 0" />
@@ -271,5 +271,5 @@
         <link name="${component_name_underscore}baro_link" />
         <joint name="${component_name_underscore}baro_joint" type="fixed">
-          <parent link="${component_name_underscore}camera_center"/>
+          <parent link="${component_name_underscore}camera_center_frame"/>
           <child link="${component_name_underscore}baro_link"/>
           <origin xyz="0 0 0" rpy="0 0 0" />
@@ -293,5 +293,5 @@
       <link name="${component_name_underscore}camera_frame" />
       <joint name="${component_name_underscore}camera_joint" type="fixed">
-        <parent link="${component_name_underscore}camera_center"/>
+        <parent link="${component_name_underscore}camera_center_frame"/>
         <child link="${component_name_underscore}camera_frame"/>
         <origin xyz="${optical_offset_x} 0 0" rpy="0 0 0" />
@@ -307,8 +307,8 @@
     <xacro:include filename="$(find husarion_components_description)/urdf/gz_sensor.urdf.xacro" ns="gz_sensor" />
     <xacro:gz_sensor.camera
-      reference="${component_name_underscore}camera_center"
+      reference="${component_name_underscore}camera_center_frame"
       name="${robot_namespace_slash}${component_name_underscore}stereolabs_zed_color"
       topic="${robot_namespace_slash}${component_name_slash}zed_node/rgb/image_rect_color"
-      frame_id="${robot_namespace_slash}${component_name_underscore}camera_center"
+      frame_id="${robot_namespace_slash}${component_name_underscore}camera_center_frame"
       frequency="30"
       width="1280"
@@ -316,8 +316,8 @@
       fov="${110.0/180.0*pi}" />
     <xacro:gz_sensor.depth_camera
-      reference="${component_name_underscore}camera_center"
+      reference="${component_name_underscore}camera_center_frame"
       name="${robot_namespace_slash}${component_name_underscore}stereolabs_zed_depth"
       topic="${robot_namespace_slash}${component_name_slash}zed_node/depth"
-      frame_id="${robot_namespace_slash}${component_name_underscore}camera_center"
+      frame_id="${robot_namespace_slash}${component_name_underscore}camera_center_frame"
       frequency="30"
       width="1280"

File: urdf/teltonika_003R-00253.urdf.xacro (robot description, xacro)
@@ -25,11 +25,11 @@
     <xacro:property name="component_name_underscore" value="${component_name + '_' if component_name != '' else ''}" />
     <xacro:property name="component_name_slash" value="${component_name + '/' if component_name != '' else ''}" />
-    <joint name="${parent_link.rstrip('_link')}_to_${component_name_underscore}teltonika_mounting_joint"
+    <joint name="${parent_link.rstrip('_link')}_to_${component_name_underscore}joint"
       type="fixed">
       <origin xyz="${xyz}" rpy="${rpy}" />
       <parent link="${parent_link}" />
-      <child link="${component_name_underscore}teltonika_mounting_link" />
+      <child link="${component_name_underscore}link" />
     </joint>
-    <link name="${component_name_underscore}teltonika_mounting_link">
+    <link name="${component_name_underscore}link">
       <visual>
         <origin xyz="0.0 0.0 0.0" rpy="0.0 0.0 0.0" />
@@ -54,18 +54,18 @@
     </link>
     <joint
-      name="${component_name_underscore}teltonika_mounting_link_to_${component_name_underscore}teltonika_joint"
+      name="${component_name_underscore}to_${component_name_underscore}origin_joint"
       type="fixed">
       <origin xyz="0.045 0.0 0.0058" rpy="0.0 0.0 0.0" />
-      <parent link="${component_name_underscore}teltonika_mounting_link" />
-      <child link="${component_name_underscore}teltonika" />
+      <parent link="${component_name_underscore}link" />
+      <child link="${component_name_underscore}origin_frame" />
     </joint>
-    <link name="${component_name_underscore}teltonika" />
-    <gazebo reference="${component_name_underscore}teltonika">
-      <sensor name="navsat" type="navsat">
+    <link name="${component_name_underscore}origin_frame" />
+    <gazebo reference="${component_name_underscore}origin_frame">
+      <sensor name="${robot_namespace_slash}${component_name_underscore}navsat" type="navsat">
         <plugin filename="ignition-gazebo-navsat-system" name="ignition::gazebo::systems::NavSat" />
         <always_on>1</always_on>
         <update_rate>1</update_rate>
         <topic>${robot_namespace_slash}${component_name_slash}fix</topic>
-        <gz_frame_id>${robot_namespace_slash}${component_name_slash}teltonika</gz_frame_id>
+        <gz_frame_id>${robot_namespace_slash}${component_name_slash}origin_frame</gz_frame_id>
       </sensor>
     </gazebo>

File: urdf/velodyne_puck.urdf.xacro (robot description, xacro)
@@ -25,10 +25,10 @@
     <xacro:property name="component_name_underscore" value="${component_name + '_' if component_name != '' else ''}" />
     <xacro:property name="component_name_slash" value="${component_name + '/' if component_name != '' else ''}" />
-    <joint name="${parent_link.rstrip('_link')}_to_${component_name_underscore}velodyne_puck_joint" type="fixed">
+    <joint name="${parent_link.rstrip('_link')}_to_${component_name_underscore}joint" type="fixed">
       <origin xyz="${xyz}" rpy="${rpy}" />
       <parent link="${parent_link}" />
-      <child link="${component_name_underscore}velodyne_puck_link" />
+      <child link="${component_name_underscore}link" />
     </joint>
-    <link name="${component_name_underscore}velodyne_puck_link">
+    <link name="${component_name_underscore}link">
       <!-- <visual>
         <origin xyz="0.0 0.0 0.0" rpy="0.0 0.0 0.0" />
@@ -61,15 +61,15 @@
       </inertial>
     </link>
-    <joint name="${component_name_underscore}velodyne_puck_to_${component_name_underscore}velodyne_joint"
+    <joint name="${component_name_underscore}to_${component_name_underscore}lidar_joint"
       type="fixed">
       <origin xyz="0.0 0.0 0.0378" rpy="0.0 0.0 0.0" />
-      <parent link="${component_name_underscore}velodyne_puck_link" />
-      <child link="${component_name_underscore}velodyne" />
+      <parent link="${component_name_underscore}link" />
+      <child link="${component_name_underscore}lidar_frame" />
     </joint>
-    <link name="${component_name_underscore}velodyne" />
-    <gazebo reference="${component_name_underscore}velodyne">
+    <link name="${component_name_underscore}lidar_frame" />
+    <gazebo reference="${component_name_underscore}lidar_frame">
       <!-- gpu_lidar has to be set, CPU lidar doesn't work in ignition -
       https://github.com/gazebosim/gz-sensors/issues/26 -->
-      <sensor type="gpu_lidar" name="${robot_namespace_slash}${component_name_underscore}velodyne_puck_sensor">
+      <sensor type="gpu_lidar" name="${robot_namespace_slash}${component_name_underscore}lidar">
         <visualize>false</visualize>
         <update_rate>10.0</update_rate>
@@ -101,5 +101,5 @@
         </ray>
         <topic>${robot_namespace_slash}${component_name_slash}velodyne_points</topic>
-        <gz_frame_id>${robot_namespace_slash}${component_name_underscore}velodyne</gz_frame_id>
+        <gz_frame_id>${robot_namespace_slash}${component_name_underscore}lidar_frame</gz_frame_id>
         <always_on>true</always_on>
       </sensor>

File: urdf/wibotic_receiver.urdf.xacro (robot description, xacro)
@@ -24,10 +24,10 @@
     <xacro:property name="robot_namespace_slash" value="${robot_namespace + '/' if robot_namespace != '' else ''}" />
     <xacro:property name="component_name_underscore" value="${component_name + '_' if component_name != '' else ''}" />
-    <joint name="${parent_link.rstrip('_link')}_to_${component_name_underscore}wibotic_receiver_joint" type="fixed">
+    <joint name="${parent_link.rstrip('_link')}_to_${component_name_underscore}joint" type="fixed">
       <origin xyz="${xyz}" rpy="${rpy}" />
       <parent link="${parent_link}" />
-      <child link="${component_name_underscore}wibotic_receiver_link" />
+      <child link="${component_name_underscore}link" />
     </joint>
-    <link name="${component_name_underscore}wibotic_receiver_link">
+    <link name="${component_name_underscore}link">
       <!-- <visual>
         <origin xyz="0.0 0.0 0.0" rpy="0.0 0.0 ${pi/2.0}" />

File: urdf/wibotic_station.urdf.xacro (robot description, xacro)
@@ -25,10 +25,10 @@
     </xacro:if>
     <xacro:property name="component_name_underscore" value="${component_name + '_' if component_name != '' else ''}" />
-    <joint name="${parent_link.rstrip('_link')}_to_${component_name_underscore}wibotic_station_joint" type="fixed">
+    <joint name="${parent_link.rstrip('_link')}_to_${component_name_underscore}joint" type="fixed">
       <origin xyz="${xyz}" rpy="${rpy}" />
       <parent link="${parent_link}" />
-      <child link="${component_name_underscore}wibotic_station_link" />
+      <child link="${component_name_underscore}link" />
     </joint>
-    <link name="${component_name_underscore}wibotic_station_link">
+    <link name="${component_name_underscore}link">
       <!-- <visual>
         <origin xyz="0.0 0.0 0.0" rpy="0.0 0.0 ${pi/2.0}" />
@@ -63,12 +63,12 @@
       </inertial>
     </link>
-    <joint name="${component_name_underscore}wibotic_station_to_${component_name_underscore}wibotic_transmitter_joint" type="fixed">
+    <joint name="${component_name_underscore}to_${component_name_underscore}transmitter_joint" type="fixed">
       <!-- This should be when docking is released for panther-docker
       <origin xyz="0.05 0.0 0.295" rpy="0.0 0.0 ${pi}" /> -->
       <origin xyz="0.05 0.0 0.5" rpy="0.0 0.0 ${pi}" />
-      <parent link="${component_name_underscore}wibotic_station_link" />
-      <child link="${component_name_underscore}wibotic_transmitter_link" />
+      <parent link="${component_name_underscore}link" />
+      <child link="${component_name_underscore}transmitter_link" />
     </joint>
-    <link name="${component_name_underscore}wibotic_transmitter_link" />
+    <link name="${component_name_underscore}transmitter_link" />
   </xacro:macro>
   <xacro:macro name="create_apriltag"

Commit message: oak: remove default component name

File: urdf/luxonis_depthai.urdf.xacro (robot description, xacro)
@@ -21,13 +21,16 @@
                        model:='OAK-D-PRO'
                        use_sim:=False">
-    <xacro:if value="${component_name == ''}">
+    <!-- <xacro:if value="${component_name == ''}">
       <xacro:property name="component_name" value="oak" />
-    </xacro:if>
+    </xacro:if> -->
+    <!-- ^ removed for compatibility with hw driver -->
     <xacro:property name="robot_namespace_slash" value="${robot_namespace + '/' if robot_namespace != '' else ''}" />
     <xacro:property name="component_name_underscore" value="${component_name + '_' if component_name != '' else ''}" />
     <xacro:property name="component_name_slash" value="${component_name + '/' if component_name != '' else ''}" />
+    <xacro:property name="component_name_underscore_nonempty" value="${component_name_underscore if component_name_underscore != '' else 'oak_'}" />
+    <!-- ^ in case no name is provided, generate "..._link" instead of just "link" -->
     <xacro:include filename="$(find depthai_descriptions)/urdf/include/depthai_macro.urdf.xacro" />
     <xacro:depthai_camera camera_name="${component_name}" parent="${parent_link}"
-      base_frame="${robot_namespace_slash}${component_name_underscore}link" camera_model="${model}"
+      base_frame="${robot_namespace_slash}${component_name_underscore_nonempty}link" camera_model="${model}"
       cam_pos_x="${xyz.split()[0]}" cam_pos_y="${xyz.split()[1]}" cam_pos_z="${xyz.split()[2]}"
       cam_roll="${rpy.split()[0]}" cam_pitch="${rpy.split()[1]}" cam_yaw="${rpy.split()[2]}"
@@ -36,5 +39,5 @@
       ns="gz_sensor" />
     <xacro:gz_sensor.camera
-      reference="${component_name_underscore}link"
+      reference="${component_name_underscore_nonempty}link"
       name="${robot_namespace_slash}${component_name_underscore}color"
       topic="${robot_namespace_slash}${component_name_slash}rgb/color"
@@ -45,5 +48,5 @@
       fov="${60.0/180.0*pi}" />
     <xacro:gz_sensor.depth_camera
-      reference="${component_name_underscore}link"
+      reference="${component_name_underscore_nonempty}link"
       name="${robot_namespace_slash}${component_name_underscore}depth"
       topic="${robot_namespace_slash}${component_name_slash}stereo/depth"
