Commit message: Fix refactor (#10)
* gz_components.launch default component names

* ...transmitter_link -> ...wibotic_transmitter_link

* remove default component names from ouster and rplidar urdfs

* oak: remove default component name

* fix test errors

* velodyne: remove default component name

* remove oak default name from luxonis_depthai gz bridge launch

* revert oak default name removal

* allow teltonika without name, producing "gps" frame without any prefix

* remove unused imports

* fix teltonika urdf gazebo params

* fix teltonika

File: urdf/luxonis_depthai.urdf.xacro (robot description, xacro)
@@ -27,7 +27,9 @@
     <xacro:property name="component_name_underscore" value="${component_name + '_' if component_name != '' else ''}" />
     <xacro:property name="component_name_slash" value="${component_name + '/' if component_name != '' else ''}" />
+    <xacro:property name="component_name_underscore_nonempty" value="${component_name_underscore if component_name_underscore != '' else 'oak_'}" />
+    <!-- ^ in case no name is provided, generate "..._link" instead of just "link" -->
     <xacro:include filename="$(find depthai_descriptions)/urdf/include/depthai_macro.urdf.xacro" />
     <xacro:depthai_camera camera_name="${component_name}" parent="${parent_link}"
-      base_frame="${robot_namespace_slash}${component_name_underscore}link" camera_model="${model}"
+      base_frame="${robot_namespace_slash}${component_name_underscore_nonempty}link" camera_model="${model}"
       cam_pos_x="${xyz.split()[0]}" cam_pos_y="${xyz.split()[1]}" cam_pos_z="${xyz.split()[2]}"
       cam_roll="${rpy.split()[0]}" cam_pitch="${rpy.split()[1]}" cam_yaw="${rpy.split()[2]}"
@@ -36,5 +38,5 @@
       ns="gz_sensor" />
     <xacro:gz_sensor.camera
-      reference="${component_name_underscore}link"
+      reference="${component_name_underscore_nonempty}link"
       name="${robot_namespace_slash}${component_name_underscore}color"
       topic="${robot_namespace_slash}${component_name_slash}rgb/color"
@@ -45,5 +47,5 @@
       fov="${60.0/180.0*pi}" />
     <xacro:gz_sensor.depth_camera
-      reference="${component_name_underscore}link"
+      reference="${component_name_underscore_nonempty}link"
       name="${robot_namespace_slash}${component_name_underscore}depth"
       topic="${robot_namespace_slash}${component_name_slash}stereo/depth"

File: urdf/teltonika_003R-00253.urdf.xacro (robot description, xacro)
@@ -54,12 +54,12 @@
     </link>
     <joint
-      name="${component_name_underscore}to_${component_name_underscore}antenna_joint"
+      name="${component_name_underscore}to_${component_name_underscore}_joint"
       type="fixed">
       <origin xyz="0.045 0.0 0.0058" rpy="0.0 0.0 0.0" />
       <parent link="${component_name_underscore}link" />
-      <child link="${component_name_underscore}antenna" />
+      <child link="${component_name_underscore}" />
     </joint>
-    <link name="${component_name_underscore}antenna" />
-    <gazebo reference="${component_name_underscore}antenna">
+    <link name="${component_name_underscore}" />
+    <gazebo reference="${component_name_underscore}">
       <sensor name="${robot_namespace_slash}${component_name_underscore}navsat" type="navsat">
         <plugin filename="ignition-gazebo-navsat-system" name="ignition::gazebo::systems::NavSat" />
@@ -67,5 +67,5 @@
         <update_rate>1</update_rate>
         <topic>${robot_namespace_slash}${component_name_slash}fix</topic>
-        <gz_frame_id>${robot_namespace_slash}${component_name_slash}antenna</gz_frame_id>
+        <gz_frame_id>${robot_namespace_slash}${component_name_underscore}</gz_frame_id>
       </sensor>
     </gazebo>
