Commit message: fix teltonika URDF crash

File: urdf/teltonika_003R-00253.urdf.xacro (robot description, xacro)
@@ -20,11 +20,13 @@
                        device_namespace:=gps">
     <xacro:property name="ns" value="${namespace + '/' if namespace != '' else ''}" />
-    <joint name="${parent_link.rstrip('_link')}_to_antenna_joint"
+    <xacro:property name="prefix" value="${device_namespace + '_' if device_namespace != '' else ''}" />
+    <xacro:property name="device_ns" value="${device_namespace + '/' if device_namespace != '' else ''}" />
+    <joint name="${parent_link.rstrip('_link')}_to_${prefix}teltonika_mounting_joint"
       type="fixed">
       <origin xyz="${xyz}" rpy="${rpy}" />
       <parent link="${parent_link}" />
-      <child link="${device_namespace}_mounting_point" />
+      <child link="${prefix}teltonika_mounting_link" />
     </joint>
-    <link name="${device_namespace}_mounting_point">
+    <link name="${prefix}teltonika_mounting_link">
       <visual>
         <origin xyz="0.0 0.0 0.0" rpy="0.0 0.0 0.0" />
@@ -49,18 +51,18 @@
     </link>
     <joint
-      name="antenna_to_${device_namespace.rstrip('_link')}_joint"
+      name="${prefix}teltonika_mounting_link_to_${prefix}teltonika_joint"
       type="fixed">
       <origin xyz="0.045 0.0 0.0058" rpy="0.0 0.0 0.0" />
-      <parent link="${device_namespace}_mounting_point" />
-      <child link="${device_namespace}" />
+      <parent link="${prefix}teltonika_mounting_link" />
+      <child link="${prefix}teltonika" />
     </joint>
-    <link name="${device_namespace}" />
-    <gazebo reference="${device_namespace}">
+    <link name="${prefix}teltonika" />
+    <gazebo reference="${prefix}teltonika">
       <sensor name="navsat" type="navsat">
         <plugin filename="ignition-gazebo-navsat-system" name="ignition::gazebo::systems::NavSat" />
         <always_on>1</always_on>
         <update_rate>1</update_rate>
-        <topic>${ns}${device_namespace}/fix</topic>
-        <gz_frame_id>${ns}${device_namespace}</gz_frame_id>
+        <topic>${ns}${device_ns}fix</topic>
+        <gz_frame_id>${ns}${device_ns}teltonika</gz_frame_id>
       </sensor>
     </gazebo>

Commit message: urdf default name teltonika -> gps

File: urdf/teltonika_003R-00253.urdf.xacro (robot description, xacro)
@@ -20,5 +20,5 @@
                        component_name:=''">
     <xacro:if value="${component_name == ''}">
-      <xacro:property name="component_name" value="teltonika" />
+      <xacro:property name="component_name" value="gps" />
     </xacro:if>
     <xacro:property name="robot_namespace_slash" value="${robot_namespace + '/' if robot_namespace != '' else ''}" />

Commit message: rename teltonika frame

File: urdf/teltonika_003R-00253.urdf.xacro (robot description, xacro)
@@ -54,12 +54,12 @@
     </link>
     <joint
-      name="${component_name_underscore}to_${component_name_underscore}origin_joint"
+      name="${component_name_underscore}to_${component_name_underscore}antenna_joint"
       type="fixed">
       <origin xyz="0.045 0.0 0.0058" rpy="0.0 0.0 0.0" />
       <parent link="${component_name_underscore}link" />
-      <child link="${component_name_underscore}origin_frame" />
+      <child link="${component_name_underscore}antenna" />
     </joint>
-    <link name="${component_name_underscore}origin_frame" />
-    <gazebo reference="${component_name_underscore}origin_frame">
+    <link name="${component_name_underscore}antenna" />
+    <gazebo reference="${component_name_underscore}antenna">
       <sensor name="${robot_namespace_slash}${component_name_underscore}navsat" type="navsat">
         <plugin filename="ignition-gazebo-navsat-system" name="ignition::gazebo::systems::NavSat" />
@@ -67,5 +67,5 @@
         <update_rate>1</update_rate>
         <topic>${robot_namespace_slash}${component_name_slash}fix</topic>
-        <gz_frame_id>${robot_namespace_slash}${component_name_slash}origin_frame</gz_frame_id>
+        <gz_frame_id>${robot_namespace_slash}${component_name_slash}antenna</gz_frame_id>
       </sensor>
     </gazebo>

Commit message: allow teltonika without name, producing "gps" frame without any prefix

File: urdf/teltonika_003R-00253.urdf.xacro (robot description, xacro)
@@ -19,17 +19,20 @@
                        robot_namespace:=''
                        component_name:=''">
-    <xacro:if value="${component_name == ''}">
+    <!-- <xacro:if value="${component_name == ''}">
       <xacro:property name="component_name" value="gps" />
-    </xacro:if>
+    </xacro:if> -->
+    <!-- ^ removed for compatibility with hw driver -->
     <xacro:property name="robot_namespace_slash" value="${robot_namespace + '/' if robot_namespace != '' else ''}" />
     <xacro:property name="component_name_underscore" value="${component_name + '_' if component_name != '' else ''}" />
     <xacro:property name="component_name_slash" value="${component_name + '/' if component_name != '' else ''}" />
-    <joint name="${parent_link.rstrip('_link')}_to_${component_name_underscore}joint"
+    <xacro:property name="component_name_underscore_nonempty" value="${component_name_underscore if component_name_underscore != '' else 'gps_'}" />
+    <!-- ^ in case no name is provided, generate "..._link" instead of just "link" -->
+    <joint name="${parent_link.rstrip('_link')}_to_${component_name_underscore_nonempty}joint"
       type="fixed">
       <origin xyz="${xyz}" rpy="${rpy}" />
       <parent link="${parent_link}" />
-      <child link="${component_name_underscore}link" />
+      <child link="${component_name_underscore_nonempty}link" />
     </joint>
-    <link name="${component_name_underscore}link">
+    <link name="${component_name_underscore_nonempty}link">
       <visual>
         <origin xyz="0.0 0.0 0.0" rpy="0.0 0.0 0.0" />
@@ -54,13 +57,13 @@
     </link>
     <joint
-      name="${component_name_underscore}to_${component_name_underscore}antenna_joint"
+      name="${component_name_underscore_nonempty}to_${component_name_underscore}gps_joint"
       type="fixed">
       <origin xyz="0.045 0.0 0.0058" rpy="0.0 0.0 0.0" />
-      <parent link="${component_name_underscore}link" />
-      <child link="${component_name_underscore}antenna" />
+      <parent link="${component_name_underscore_nonempty}link" />
+      <child link="${component_name_underscore}gps" />
     </joint>
-    <link name="${component_name_underscore}antenna" />
-    <gazebo reference="${component_name_underscore}antenna">
-      <sensor name="${robot_namespace_slash}${component_name_underscore}navsat" type="navsat">
+    <link name="${component_name_underscore}gps" />
+    <gazebo reference="${component_name_underscore}gps">
+      <sensor name="${robot_namespace_slash}${component_name_underscore_nonempty}navsat" type="navsat">
         <plugin filename="ignition-gazebo-navsat-system" name="ignition::gazebo::systems::NavSat" />
         <always_on>1</always_on>

Commit message: fix teltonika urdf gazebo params

File: urdf/teltonika_003R-00253.urdf.xacro (robot description, xacro)
@@ -27,4 +27,5 @@
     <xacro:property name="component_name_slash" value="${component_name + '/' if component_name != '' else ''}" />
     <xacro:property name="component_name_underscore_nonempty" value="${component_name_underscore if component_name_underscore != '' else 'gps_'}" />
+    <xacro:property name="component_name_slash_nonempty" value="${component_name_slash if component_name_slash != '' else 'gps/'}" />
     <!-- ^ in case no name is provided, generate "..._link" instead of just "link" -->
     <joint name="${parent_link.rstrip('_link')}_to_${component_name_underscore_nonempty}joint"
@@ -69,6 +70,6 @@
         <always_on>1</always_on>
         <update_rate>1</update_rate>
-        <topic>${robot_namespace_slash}${component_name_slash}fix</topic>
-        <gz_frame_id>${robot_namespace_slash}${component_name_slash}antenna</gz_frame_id>
+        <topic>${robot_namespace_slash}${component_name_slash_nonempty}fix</topic>
+        <gz_frame_id>${robot_namespace_slash}${component_name_underscore}gps</gz_frame_id>
       </sensor>
     </gazebo>

Commit message: fix teltonika

File: urdf/teltonika_003R-00253.urdf.xacro (robot description, xacro)
@@ -19,21 +19,17 @@
                        robot_namespace:=''
                        component_name:=''">
-    <!-- <xacro:if value="${component_name == ''}">
+    <xacro:if value="${component_name == ''}">
       <xacro:property name="component_name" value="gps" />
-    </xacro:if> -->
-    <!-- ^ removed for compatibility with hw driver -->
+    </xacro:if>
     <xacro:property name="robot_namespace_slash" value="${robot_namespace + '/' if robot_namespace != '' else ''}" />
     <xacro:property name="component_name_underscore" value="${component_name + '_' if component_name != '' else ''}" />
     <xacro:property name="component_name_slash" value="${component_name + '/' if component_name != '' else ''}" />
-    <xacro:property name="component_name_underscore_nonempty" value="${component_name_underscore if component_name_underscore != '' else 'gps_'}" />
-    <xacro:property name="component_name_slash_nonempty" value="${component_name_slash if component_name_slash != '' else 'gps/'}" />
-    <!-- ^ in case no name is provided, generate "..._link" instead of just "link" -->
-    <joint name="${parent_link.rstrip('_link')}_to_${component_name_underscore_nonempty}joint"
+    <joint name="${parent_link.rstrip('_link')}_to_${component_name_underscore}joint"
       type="fixed">
       <origin xyz="${xyz}" rpy="${rpy}" />
       <parent link="${parent_link}" />
-      <child link="${component_name_underscore_nonempty}link" />
+      <child link="${component_name_underscore}link" />
     </joint>
-    <link name="${component_name_underscore_nonempty}link">
+    <link name="${component_name_underscore}link">
       <visual>
         <origin xyz="0.0 0.0 0.0" rpy="0.0 0.0 0.0" />
@@ -58,18 +54,18 @@
     </link>
     <joint
-      name="${component_name_underscore_nonempty}to_${component_name_underscore}gps_joint"
+      name="${component_name_underscore}to_${component_name_underscore}_joint"
       type="fixed">
       <origin xyz="0.045 0.0 0.0058" rpy="0.0 0.0 0.0" />
-      <parent link="${component_name_underscore_nonempty}link" />
-      <child link="${component_name_underscore}gps" />
+      <parent link="${component_name_underscore}link" />
+      <child link="${component_name_underscore}" />
     </joint>
-    <link name="${component_name_underscore}gps" />
-    <gazebo reference="${component_name_underscore}gps">
-      <sensor name="${robot_namespace_slash}${component_name_underscore_nonempty}navsat" type="navsat">
+    <link name="${component_name_underscore}" />
+    <gazebo reference="${component_name_underscore}">
+      <sensor name="${robot_namespace_slash}${component_name_underscore}navsat" type="navsat">
         <plugin filename="ignition-gazebo-navsat-system" name="ignition::gazebo::systems::NavSat" />
         <always_on>1</always_on>
         <update_rate>1</update_rate>
-        <topic>${robot_namespace_slash}${component_name_slash_nonempty}fix</topic>
-        <gz_frame_id>${robot_namespace_slash}${component_name_underscore}gps</gz_frame_id>
+        <topic>${robot_namespace_slash}${component_name_slash}fix</topic>
+        <gz_frame_id>${robot_namespace_slash}${component_name_underscore}</gz_frame_id>
       </sensor>
     </gazebo>

Commit message: Fixed teltonika antenna link
Signed-off-by: Jakub Delicat <jakub.delicat@husarion.com>

File: urdf/teltonika_003R-00253.urdf.xacro (robot description, xacro)
@@ -58,8 +58,8 @@
       <origin xyz="0.045 0.0 0.0058" rpy="0.0 0.0 0.0" />
       <parent link="${component_name_underscore}link" />
-      <child link="${component_name_underscore}" />
+      <child link="${component_name_underscore}antenna" />
     </joint>
-    <link name="${component_name_underscore}" />
-    <gazebo reference="${component_name_underscore}">
+    <link name="${component_name_underscore}antenna" />
+    <gazebo reference="${component_name_underscore}antenna">
       <sensor name="${robot_namespace_slash}${component_name_underscore}navsat" type="navsat">
         <plugin filename="ignition-gazebo-navsat-system" name="ignition::gazebo::systems::NavSat" />
@@ -67,5 +67,5 @@
         <update_rate>1</update_rate>
         <topic>${robot_namespace_slash}${component_name_slash}fix</topic>
-        <gz_frame_id>${robot_namespace_slash}${component_name_underscore}</gz_frame_id>
+        <gz_frame_id>${robot_namespace_slash}${component_name_underscore}antenna</gz_frame_id>
       </sensor>
     </gazebo>
