Commit message: ...transmitter_link -> ...wibotic_transmitter_link

File: urdf/wibotic_station.urdf.xacro (robot description, xacro)
@@ -63,12 +63,12 @@
       </inertial>
     </link>
-    <joint name="${component_name_underscore}to_${component_name_underscore}transmitter_joint" type="fixed">
+    <joint name="${component_name_underscore}to_${component_name_underscore}wibotic_transmitter_joint" type="fixed">
       <!-- This should be when docking is released for panther-docker
       <origin xyz="0.05 0.0 0.295" rpy="0.0 0.0 ${pi}" /> -->
       <origin xyz="0.05 0.0 0.5" rpy="0.0 0.0 ${pi}" />
       <parent link="${component_name_underscore}link" />
-      <child link="${component_name_underscore}transmitter_link" />
+      <child link="${component_name_underscore}wibotic_transmitter_link" />
     </joint>
-    <link name="${component_name_underscore}transmitter_link" />
+    <link name="${component_name_underscore}wibotic_transmitter_link" />
   </xacro:macro>
   <xacro:macro name="create_apriltag"

Commit message: Make wibotic station more universal (change root_link, edit height of elements)

File: urdf/wibotic_station.urdf.xacro (robot description, xacro)
@@ -13,8 +13,15 @@
 -->
 <robot xmlns:xacro="http://www.ros.org/wiki/xacro" name="wibotic_station">
+  <xacro:arg name="apriltag_height" default="0.5" />
+  <xacro:arg name="apriltag_image" default="" />
+  <xacro:arg name="apriltag_size" default="0.08" />
   <xacro:arg name="component_name" default="" />
-  <xacro:arg name="apriltag_image_path" default="" />
-  <xacro:arg name="apriltag_size" default="0.07" />
-  <xacro:macro name="wibotic_station"
+  <xacro:arg name="root_link" default="apriltag_link" />
+  <xacro:arg name="transmitter_height" default="0.3" />
+  <!-- The AprilTag serves as the root element of the Wibotic Station.
+       This design ensures that docking functionality can detect stations via AprilTags,
+       and maintains a single root in the TF tree for proper frame hierarchy.
+       You can change the root manipulating root_link, parent_link, xyz and rpy parameters -->
+    <xacro:macro name="wibotic_station"
                params="parent_link
                        xyz:='0.0 0.0 0.0'
@@ -26,10 +33,10 @@
     </xacro:if>
     <xacro:property name="component_name_underscore" value="${component_name + '_' if component_name != '' else ''}" />
-    <joint name="${parent_link.rstrip('_link')}_to_${component_name_underscore}joint" type="fixed">
+    <joint name="${parent_link}to_${component_name_underscore}wibotic_station_link_joint" type="fixed">
       <origin xyz="${xyz}" rpy="${rpy}" />
       <parent link="${parent_link}" />
-      <child link="${component_name_underscore}link" />
+      <child link="${component_name_underscore}wibotic_station_link" />
     </joint>
-  <link name="${component_name_underscore}link">
+    <link name="${component_name_underscore}wibotic_station_link">
       <visual>
         <origin xyz="0.0 0.0 0.0" rpy="0.0 0.0 0.0" />
@@ -40,12 +47,12 @@
       <!-- Fake collision fit to dae -->
       <collision>
-        <origin xyz="-0.2 0.0  0.4" rpy="0.0 0.0 0.0" />
+        <origin xyz="-0.2 0.0  0.45" rpy="0.0 0.0 0.0" />
         <geometry>
-          <box size="0.4 0.5 0.8" />
+          <box size="0.4 0.5 0.9" />
         </geometry>
       </collision>
       <!-- Fake inertia -->
       <inertial>
-        <origin xyz="-0.15 0.0 0.3" rpy="0.0 0.0 0.0" />
+        <origin xyz="-0.2 0.0  0.45" rpy="0.0 0.0 0.0" />
         <mass value="15.0" />
         <inertia ixx="0.001111" ixy="0.0"      ixz="0.0"
@@ -54,7 +61,7 @@
       </inertial>
     </link>
-    <joint name="${component_name_underscore}to_${component_name_underscore}wibotic_transmitter_joint" type="fixed">
-      <origin xyz="0.0 0.0 ${transmitter_height}" rpy="0.0 0.0 0.0" />
-      <parent link="${component_name_underscore}link" />
+    <joint name="${component_name_underscore}wibotic_station_link_to_${component_name_underscore}wibotic_transmitter_joint" type="fixed">
+      <origin xyz="0.0 0.0 ${transmitter_height + 0.135}" rpy="0.0 0.0 0.0" /> <!-- 0.135 is offset from mesh origin to bottom of transmitter case -->
+      <parent link="${component_name_underscore}wibotic_station_link" />
       <child link="${component_name_underscore}wibotic_transmitter_link" />
     </joint>
@@ -67,25 +74,25 @@
       </visual>
     </link>
+    <!-- Additional link for as a destination for docking -->
+    <joint name="${component_name_underscore}wibotic_transmitter_link_to_${component_name_underscore}wibotic_dock_frame_joint" type="fixed">
+      <origin xyz="0.05 0.0 0.0" rpy="0.0 0.0 ${pi}" />
+      <parent link="${component_name_underscore}wibotic_transmitter_link" />
+      <child link="${component_name_underscore}wibotic_dock_frame" />
+    </joint>
+    <link name="${component_name_underscore}wibotic_dock_frame" />
   </xacro:macro>
-  <xacro:macro name="create_apriltag"
-    params="name size:=$(arg apriltag_size) component_name:=''">
+  <xacro:macro name="apriltag"
+               params="parent_link
+                       xyz:='0.0 0.0 0.0'
+                       rpy:='0.0 0.0 0.0'
+                       component_name:=''
+                       size:=0.08">
     <xacro:property name="component_name_underscore" value="${component_name + '_' if component_name != '' else ''}" />
-    <link name="${component_name_underscore}${name}_link">
-      <visual>
-        <origin xyz="0 0 0" rpy="0 0 0" />
-        <geometry>
-          <box size="${size+0.02} ${size+0.02} 0.00005" />
-        </geometry>
-        <material name="White">
-          <color rgba="1.0 1.0 1.0 1.0" />
-        </material>
-      </visual>
-      </link>
-    <joint name="${name}_to_${name}_${component_name_underscore}image_link_joint" type="fixed">
-      <origin xyz="0 0 0" rpy="0 -${pi/2.0} ${pi/2.0}" />
-      <parent link="${component_name_underscore}${name}_link" />
-      <child link="${component_name_underscore}${name}_image_link" />
+    <joint name="${parent_link}_to_${component_name_underscore}image_link_joint" type="fixed">
+      <origin xyz="${xyz}" rpy="${rpy}" />
+      <parent link="${parent_link}" />
+      <child link="${component_name_underscore}image_link" />
     </joint>
-    <link name="${component_name_underscore}${name}_image_link">
+    <link name="${component_name_underscore}image_link">
       <visual>
         <origin xyz="0 0 0" rpy="0 ${pi/2.0} 0" />
@@ -100,9 +107,9 @@
         <origin xyz="0 0 0" rpy="0 ${pi/2.0} 0" />
         <geometry>
-          <box size="${size+0.02} ${size+0.02} 0.0001" />
+          <box size="${size} ${size} 0.0001" />
         </geometry>
       </collision>
     </link>
-    <gazebo reference="${component_name_underscore}${name}_image_link">
+    <gazebo reference="${component_name_underscore}image_link">
       <visual>
         <material>
@@ -114,5 +121,5 @@
           <pbr>
             <metal>
-              <albedo_map>$(arg apriltag_image_path)</albedo_map>
+              <albedo_map>$(arg apriltag_image)</albedo_map>
             </metal>
           </pbr>
@@ -120,9 +127,13 @@
       </visual>
     </gazebo>
-    <xacro:property name="apriltag_size_prop" value="$(arg apriltag_size)" />
-    <xacro:wibotic_station
-      component_name="$(arg component_name)" parent_link="${component_name_underscore}${name}_image_link"  xyz="0.0 0.0 0.5"
-      rpy="${pi} 0 0" transmitter_height="$(arg transmitter_height)" />
   </xacro:macro>
-  <xacro:create_apriltag name="apriltag" component_name="$(arg component_name)" size="$(arg apriltag_size)" />
+  <xacro:property name="component_name_prop" value="$(arg component_name)" />
+  <xacro:property name="apriltag_name" value="${component_name_prop + '_apriltag' if component_name_prop != '' else 'apriltag'}" />
+  <link name="$(arg root_link)" />
+  <!-- AprilTag as root -->
+  <xacro:apriltag parent_link="$(arg root_link)" xyz="0 0 0" rpy="0 -${pi/2.0} ${pi/2.0}" component_name="${apriltag_name}" size="$(arg apriltag_size)" />
+  <xacro:wibotic_station parent_link="$(arg root_link)" xyz="0 -$(arg apriltag_height) 0" rpy="${pi} -${pi/2.0} ${pi/2.0}" component_name="$(arg component_name)" transmitter_height="$(arg transmitter_height)" />
+  <!-- Station as root -->
+  <!-- <xacro:wibotic_station parent_link="$(arg root_link)" component_name="$(arg component_name)" transmitter_height="$(arg transmitter_height)" />
+  <xacro:apriltag parent_link="$(arg root_link)" xyz="0 0 $(arg apriltag_height)" rpy="${pi} 0 0" component_name="${apriltag_name}" size="$(arg apriltag_size)" /> -->
 </robot>
