Commit message: Fix collistion

File: urdf/wibotic_receiver.urdf.xacro (robot description, xacro)
@@ -31,5 +31,5 @@
     <link name="${component_name_underscore}mount_link">
       <visual>
-        <origin xyz="0.0 0.0 0.0" rpy="0.0 0.0 0.0" />
+        <origin xyz="0.01 0.0 0.0" rpy="0.0 0.0 0.0" />
         <geometry>
           <mesh filename="package://husarion_components_description/meshes/wibotic_receiver.dae" />
@@ -40,5 +40,5 @@
       </visual>
       <collision>
-        <origin xyz="-0.028 0.0 0.085" rpy="0.0 0.0 0.0" />
+        <origin xyz="-0.018 0.0 0.085" rpy="0.0 0.0 0.0" />
         <geometry>
           <box size="0.015 0.135 0.19" />
@@ -46,5 +46,5 @@
       </collision>
       <collision>
-        <origin xyz="-0.006 0.0 0.115" rpy="0.0 0.0 0.0" />
+        <origin xyz="0.004 0.0 0.115" rpy="0.0 ${pi/2} 0.0" />
         <geometry>
           <cylinder length="0.03" radius="0.07" />
@@ -53,5 +53,5 @@
     </link>
     <joint name="${component_name_underscore}mount_link_to_${component_name_underscore}coil_joint" type="fixed">
-      <origin xyz="0.0095 0.0 0.115" rpy="0.0 0.0 0.0" />
+      <origin xyz="0.018 0.0 0.115" rpy="0.0 0.0 0.0" />
       <parent link="${component_name_underscore}mount_link" />
       <child link="${component_name_underscore}coil_link" />
