Commit message: Fix ouster visual

File: urdf/ouster.urdf.xacro (robot description, xacro)
@@ -73,5 +73,5 @@
       <!-- TODO Remove simple visuals when mesh is ready -->
       <visual>
-        <origin xyz="0.0 0.0 0.0" rpy="0.0 0.0 0.0" />
+        <origin xyz="0.0 0.0 ${0.072/2.0}" rpy="0.0 0.0 0.0" />
         <geometry>
           <cylinder radius="${0.085/2.0}" length="0.073" />

Commit message: revert ouster/velodyne/rplidar/zed reading frame changes

File: urdf/ouster.urdf.xacro (robot description, xacro)
@@ -98,11 +98,11 @@
       </inertial>
     </link>
-    <joint name="${component_name_underscore}to_${component_name_underscore}lidar_joint" type="fixed">
+    <joint name="${component_name_underscore}to_${component_name_underscore}os_lidar_joint" type="fixed">
       <origin xyz="0.0 0.0 0.03618" rpy="0.0 0.0 0.0" />
       <parent link="${component_name_underscore}link" />
-      <child link="${component_name_underscore}lidar_frame" />
+      <child link="${component_name_underscore}os_lidar" />
     </joint>
-    <link name="${component_name_underscore}lidar_frame" />
-    <gazebo reference="${component_name_underscore}lidar_frame">
+    <link name="${component_name_underscore}os_lidar" />
+    <gazebo reference="${component_name_underscore}os_lidar">
       <!-- gpu_lidar has to be set, CPU lidar doesn't work in ignition -
       https://github.com/gazebosim/gz-sensors/issues/26 -->
@@ -137,5 +137,5 @@
         <update_rate>20.0</update_rate>
         <topic>${robot_namespace_slash}${component_name_slash}ouster/points</topic>
-        <gz_frame_id>${robot_namespace_slash}${component_name_underscore}lidar_frame</gz_frame_id>
+        <gz_frame_id>${robot_namespace_slash}${component_name_underscore}os_lidar</gz_frame_id>
         <always_on>true</always_on>
       </sensor>

File: urdf/slamtec_rplidar.urdf.xacro (robot description, xacro)
@@ -228,8 +228,8 @@
       <xacro:insert_block name="joint" />
       <parent link="${component_name_underscore}link" />
-      <child link="${component_name_underscore}laser_frame" />
+      <child link="${component_name_underscore}laser" />
     </joint>
-    <link name="${component_name_underscore}laser_frame" />
-    <gazebo reference="${component_name_underscore}laser_frame">
+    <link name="${component_name_underscore}laser" />
+    <gazebo reference="${component_name_underscore}laser">
       <sensor type="gpu_lidar" name="${robot_namespace_slash}${component_name_underscore}lidar">
         <always_on>false</always_on>
@@ -237,5 +237,5 @@
         <visualize>false</visualize>
         <topic>${robot_namespace_slash}${component_name_slash}scan</topic>
-        <gz_frame_id>${robot_namespace_slash}${component_name_underscore}laser_frame</gz_frame_id>
+        <gz_frame_id>${robot_namespace_slash}${component_name_underscore}laser</gz_frame_id>
         <ray>
           <scan>

File: urdf/stereolabs_zed.urdf.xacro (robot description, xacro)
@@ -172,5 +172,5 @@
     </joint>
     <!-- Camera Center -->
-    <link name="${component_name_underscore}camera_center_frame">
+    <link name="${component_name_underscore}camera_center">
       <xacro:unless value="${model == 'virtual'}">
         <visual>
@@ -195,5 +195,5 @@
     <joint name="${component_name_underscore}to_${component_name_underscore}camera_center_joint" type="fixed">
       <parent link="${component_name_underscore}link"/>
-      <child link="${component_name_underscore}camera_center_frame"/>
+      <child link="${component_name_underscore}camera_center"/>
       <origin xyz="0 0 ${height/2}" rpy="0 ${bottom_slope} 0" />
     </joint>
@@ -220,5 +220,5 @@
       </link>
       <joint name="${component_name_underscore}left_camera_joint" type="fixed">
-        <parent link="${component_name_underscore}camera_center_frame"/>
+        <parent link="${component_name_underscore}camera_center"/>
         <child link="${component_name_underscore}left_camera_frame"/>
         <origin xyz="${optical_offset_x} ${baseline/2} 0" rpy="0 0 0" />
@@ -251,5 +251,5 @@
       </link>
       <joint name="${component_name_underscore}right_camera_joint" type="fixed">
-        <parent link="${component_name_underscore}camera_center_frame"/>
+        <parent link="${component_name_underscore}camera_center"/>
         <child link="${component_name_underscore}right_camera_frame"/>
         <origin xyz="${optical_offset_x} -${baseline/2} 0" rpy="0 0 0" />
@@ -265,5 +265,5 @@
         <link name="${component_name_underscore}mag_link" />
         <joint name="${component_name_underscore}mag_joint" type="fixed">
-          <parent link="${component_name_underscore}camera_center_frame"/>
+          <parent link="${component_name_underscore}camera_center"/>
           <child link="${component_name_underscore}mag_link"/>
           <origin xyz="0 0 0" rpy="0 0 0" />
@@ -271,5 +271,5 @@
         <link name="${component_name_underscore}baro_link" />
         <joint name="${component_name_underscore}baro_joint" type="fixed">
-          <parent link="${component_name_underscore}camera_center_frame"/>
+          <parent link="${component_name_underscore}camera_center"/>
           <child link="${component_name_underscore}baro_link"/>
           <origin xyz="0 0 0" rpy="0 0 0" />
@@ -293,5 +293,5 @@
       <link name="${component_name_underscore}camera_frame" />
       <joint name="${component_name_underscore}camera_joint" type="fixed">
-        <parent link="${component_name_underscore}camera_center_frame"/>
+        <parent link="${component_name_underscore}camera_center"/>
         <child link="${component_name_underscore}camera_frame"/>
         <origin xyz="${optical_offset_x} 0 0" rpy="0 0 0" />
@@ -307,8 +307,8 @@
     <xacro:include filename="$(find husarion_components_description)/urdf/gz_sensor.urdf.xacro" ns="gz_sensor" />
     <xacro:gz_sensor.camera
-      reference="${component_name_underscore}camera_center_frame"
+      reference="${component_name_underscore}camera_center"
       name="${robot_namespace_slash}${component_name_underscore}stereolabs_zed_color"
       topic="${robot_namespace_slash}${component_name_slash}zed_node/rgb/image_rect_color"
-      frame_id="${robot_namespace_slash}${component_name_underscore}camera_center_frame"
+      frame_id="${robot_namespace_slash}${component_name_underscore}camera_center"
       frequency="30"
       width="1280"
@@ -316,8 +316,8 @@
       fov="${110.0/180.0*pi}" />
     <xacro:gz_sensor.depth_camera
-      reference="${component_name_underscore}camera_center_frame"
+      reference="${component_name_underscore}camera_center"
       name="${robot_namespace_slash}${component_name_underscore}stereolabs_zed_depth"
       topic="${robot_namespace_slash}${component_name_slash}zed_node/depth"
-      frame_id="${robot_namespace_slash}${component_name_underscore}camera_center_frame"
+      frame_id="${robot_namespace_slash}${component_name_underscore}camera_center"
       frequency="30"
       width="1280"

File: urdf/velodyne_puck.urdf.xacro (robot description, xacro)
@@ -61,12 +61,12 @@
       </inertial>
     </link>
-    <joint name="${component_name_underscore}to_${component_name_underscore}lidar_joint"
+    <joint name="${component_name_underscore}to_${component_name_underscore}velodyne_joint"
       type="fixed">
       <origin xyz="0.0 0.0 0.0378" rpy="0.0 0.0 0.0" />
       <parent link="${component_name_underscore}link" />
-      <child link="${component_name_underscore}lidar_frame" />
+      <child link="${component_name_underscore}velodyne" />
     </joint>
-    <link name="${component_name_underscore}lidar_frame" />
-    <gazebo reference="${component_name_underscore}lidar_frame">
+    <link name="${component_name_underscore}velodyne" />
+    <gazebo reference="${component_name_underscore}velodyne">
       <!-- gpu_lidar has to be set, CPU lidar doesn't work in ignition -
       https://github.com/gazebosim/gz-sensors/issues/26 -->
@@ -101,5 +101,5 @@
         </ray>
         <topic>${robot_namespace_slash}${component_name_slash}velodyne_points</topic>
-        <gz_frame_id>${robot_namespace_slash}${component_name_underscore}lidar_frame</gz_frame_id>
+        <gz_frame_id>${robot_namespace_slash}${component_name_underscore}velodyne</gz_frame_id>
         <always_on>true</always_on>
       </sensor>

Commit message: remove default component names from ouster and rplidar urdfs

File: urdf/ouster.urdf.xacro (robot description, xacro)
@@ -20,10 +20,13 @@
                        robot_namespace:=''
                        component_name:=''">
-    <xacro:if value="${component_name == ''}">
+    <!-- <xacro:if value="${component_name == ''}">
       <xacro:property name="component_name" value="ouster" />
-    </xacro:if>
+    </xacro:if> -->
+    <!-- ^ removed for compatibility with hw driver -->
     <xacro:property name="robot_namespace_slash" value="${robot_namespace + '/' if robot_namespace != '' else ''}" />
     <xacro:property name="component_name_underscore" value="${component_name + '_' if component_name != '' else ''}" />
     <xacro:property name="component_name_slash" value="${component_name + '/' if component_name != '' else ''}" />
+    <xacro:property name="component_name_underscore_nonempty" value="${component_name_underscore if component_name_underscore != '' else 'ouster_'}" />
+    <!-- ^ in case no name is provided, generate "..._link" instead of just "link" -->
     <xacro:if value="${model == 'os0_32'}">
       <xacro:property name="vfov" value="${radians(90.0)}" scope="parent" />
@@ -62,10 +65,10 @@
       <xacro:property name="mesh" value="ouster_os01" scope="parent"/>
     </xacro:if>
-    <joint name="${parent_link.rstrip('_link')}_to_${component_name_underscore}joint" type="fixed">
+    <joint name="${parent_link.rstrip('_link')}_to_${component_name_underscore_nonempty}joint" type="fixed">
       <origin xyz="${xyz}" rpy="${rpy}" />
       <parent link="${parent_link}" />
-      <child link="${component_name_underscore}link" />
+      <child link="${component_name_underscore_nonempty}link" />
     </joint>
-    <link name="${component_name_underscore}link">
+    <link name="${component_name_underscore_nonempty}link">
       <!-- <visual>
         <origin xyz="0.0 0.0 0.0" rpy="0.0 0.0 0.0" />
@@ -98,7 +101,7 @@
       </inertial>
     </link>
-    <joint name="${component_name_underscore}to_${component_name_underscore}os_lidar_joint" type="fixed">
+    <joint name="${component_name_underscore_nonempty}to_${component_name_underscore}os_lidar_joint" type="fixed">
       <origin xyz="0.0 0.0 0.03618" rpy="0.0 0.0 0.0" />
-      <parent link="${component_name_underscore}link" />
+      <parent link="${component_name_underscore_nonempty}link" />
       <child link="${component_name_underscore}os_lidar" />
     </joint>

File: urdf/slamtec_rplidar.urdf.xacro (robot description, xacro)
@@ -20,10 +20,13 @@
                        component_name:=''
                        model:=s3">
-    <xacro:if value="${component_name == ''}">
+    <!-- <xacro:if value="${component_name == ''}">
       <xacro:property name="component_name" value="rplidar" />
-    </xacro:if>
+    </xacro:if> -->
+    <!-- ^ removed for compatibility with hw driver -->
     <xacro:property name="robot_namespace_slash" value="${robot_namespace + '/' if robot_namespace != '' else ''}" />
     <xacro:property name="component_name_underscore" value="${component_name + '_' if component_name != '' else ''}" />
     <xacro:property name="component_name_slash" value="${component_name + '/' if component_name != '' else ''}" />
+    <xacro:property name="component_name_underscore_nonempty" value="${component_name_underscore if component_name_underscore != '' else 'rplidar_'}" />
+    <!-- ^ in case no name is provided, generate "..._link" instead of just "link" -->
     <xacro:if value="${model == 's3'}">
       <!-- Spec: https://www.slamtec.ai/wp-content/uploads/2023/11/SLAMTEC_rplidar_datasheet_S3_v1.0_en.pdf -->
@@ -199,10 +202,10 @@
       </xacro:property>
     </xacro:if>
-    <joint name="${parent_link.rstrip('_link')}_to_${component_name_underscore}joint" type="fixed">
+    <joint name="${parent_link.rstrip('_link')}_to_${component_name_underscore_nonempty}joint" type="fixed">
       <origin xyz="${xyz}" rpy="${rpy}" />
       <parent link="${parent_link}" />
-      <child link="${component_name_underscore}link" />
+      <child link="${component_name_underscore_nonempty}link" />
     </joint>
-    <link name="${component_name_underscore}link">
+    <link name="${component_name_underscore_nonempty}link">
       <!-- <visual>
         <origin xyz="0.0 0.0 0.0" rpy="0.0 0.0 0.0" />
@@ -225,7 +228,7 @@
       </inertial>
     </link>
-    <joint name="${component_name_underscore}to_${component_name_underscore}laser_joint" type="fixed">
+    <joint name="${component_name_underscore_nonempty}to_${component_name_underscore}laser_joint" type="fixed">
       <xacro:insert_block name="joint" />
-      <parent link="${component_name_underscore}link" />
+      <parent link="${component_name_underscore_nonempty}link" />
       <child link="${component_name_underscore}laser" />
     </joint>

Commit message: Add Ouster mesh

File: urdf/ouster.urdf.xacro (robot description, xacro)
@@ -71,19 +71,9 @@
     </joint>
     <link name="${component_name_underscore_nonempty}link">
-      <!-- <visual>
+      <visual>
         <origin xyz="0.0 0.0 0.0" rpy="0.0 0.0 0.0" />
         <geometry>
           <mesh filename="package://husarion_components_description/meshes/${mesh}.dae" />
         </geometry>
-      </visual> -->
-      <!-- TODO Remove simple visuals when mesh is ready -->
-      <visual>
-        <origin xyz="0.0 0.0 ${0.072/2.0}" rpy="0.0 0.0 0.0" />
-        <geometry>
-          <cylinder radius="${0.085/2.0}" length="0.073" />
-        </geometry>
-        <material name="LightGrey">
-          <color rgba="0.6 0.6 0.6 1.0" />
-        </material>
       </visual>
       <collision>

Commit message: Add wibotic meshes and fixes

File: urdf/ouster.urdf.xacro (robot description, xacro)
@@ -78,7 +78,7 @@
       </visual>
       <collision>
-        <origin xyz="0.0 0.0 ${0.072/2.0}" rpy="0.0 0.0 0.0" />
+        <origin xyz="0.0 0.0 ${0.015+0.074/2.0}" rpy="0.0 0.0 0.0" />
         <geometry>
-          <cylinder radius="${0.085/2.0}" length="0.073" />
+          <cylinder radius="${0.085/2.0}" length="${0.015+0.074}" /> <!-- base + lidar height -->
         </geometry>
       </collision>

File: urdf/wibotic_receiver.urdf.xacro (robot description, xacro)
@@ -27,37 +27,18 @@
       <origin xyz="${xyz}" rpy="${rpy}" />
       <parent link="${parent_link}" />
-      <child link="${component_name_underscore}link" />
+      <child link="${component_name_underscore}mount_link" />
     </joint>
-    <link name="${component_name_underscore}link">
-      <!-- <visual>
-        <origin xyz="0.0 0.0 0.0" rpy="0.0 0.0 ${pi/2.0}" />
+    <link name="${component_name_underscore}mount_link">
+      <visual>
+        <origin xyz="0.0 0.0 0.0" rpy="0.0 0.0 0.0" />
         <geometry>
-          <mesh filename="package://husarion_components_description/meshes/wibotic_receiver.stl" />
+          <mesh filename="package://husarion_components_description/meshes/wibotic_receiver.dae" />
         </geometry>
         <material name="Grey">
           <color rgba="0.15 0.15 0.15 1.0" />
         </material>
-      </visual> -->
-      <!-- TODO Remove simple visuals when mesh is ready -->
-      <visual>
-        <origin xyz="-0.008 0.0 0.085" rpy="0.0 0.0 0.0" />
-        <geometry>
-          <box size="0.015 0.135 0.19" />
-        </geometry>
-        <material name="DarkGrey">
-          <color rgba="0.2 0.2 0.2 1.0" />
-        </material>
-      </visual>
-      <visual>
-        <origin xyz="0.014 0.0 0.115" rpy="0.0 ${pi/2.0} 0.0" />
-        <geometry>
-          <cylinder length="0.03" radius="0.07" />
-        </geometry>
-        <material name="DarkGrey">
-          <color rgba="0.2 0.2 0.2 1.0" />
-        </material>
       </visual>
       <collision>
-        <origin xyz="-0.008 0.0 0.085" rpy="0.0 0.0 0.0" />
+        <origin xyz="-0.028 0.0 0.085" rpy="0.0 0.0 0.0" />
         <geometry>
           <box size="0.015 0.135 0.19" />
@@ -65,5 +46,5 @@
       </collision>
       <collision>
-        <origin xyz="0.014 0.0 0.115" rpy="0.0 ${pi/2.0} 0.0" />
+        <origin xyz="-0.006 0.0 0.115" rpy="0.0 0.0 0.0" />
         <geometry>
           <cylinder length="0.03" radius="0.07" />
@@ -71,4 +52,10 @@
       </collision>
     </link>
+    <joint name="${component_name_underscore}mount_link_to_${component_name_underscore}coil_joint" type="fixed">
+      <origin xyz="0.0095 0.0 0.115" rpy="0.0 0.0 0.0" />
+      <parent link="${component_name_underscore}mount_link" />
+      <child link="${component_name_underscore}coil_link" />
+    </joint>
+    <link name="${component_name_underscore}coil_link" />
   </xacro:macro>
 </robot>

File: urdf/wibotic_station.urdf.xacro (robot description, xacro)
@@ -20,5 +20,6 @@
                        xyz:='0.0 0.0 0.0'
                        rpy:='0.0 0.0 0.0'
-                       component_name:=''">
+                       component_name:=''
+                       transmitter_height:=0.3">
     <xacro:if value="${component_name == ''}">
       <xacro:property name="component_name" value="wibotic_station" />
@@ -30,22 +31,12 @@
       <child link="${component_name_underscore}link" />
     </joint>
-    <link name="${component_name_underscore}link">
-      <!-- <visual>
-        <origin xyz="0.0 0.0 0.0" rpy="0.0 0.0 ${pi/2.0}" />
+  <link name="${component_name_underscore}link">
+      <visual>
+        <origin xyz="0.0 0.0 0.0" rpy="0.0 0.0 0.0" />
         <geometry>
-          <mesh filename="package://husarion_components_description/meshes/wibotic_station.stl" />
+          <mesh filename="package://husarion_components_description/meshes/wibotic_frame.dae" />
         </geometry>
-      </visual> -->
-      <!-- TODO Remove simple visuals when mesh is ready -->
-      <visual>
-        <origin xyz="-0.2 0.0  0.4" rpy="0.0 0.0 0.0" />
-        <geometry>
-          <box size="0.4 0.5 0.8" />
-        </geometry>
-        <material name="LightGrey">
-          <color rgba="0.6 0.6 0.6 1.0" />
-        </material>
       </visual>
-      <!-- Fake collision fit to STL -->
+      <!-- Fake collision fit to dae -->
       <collision>
         <origin xyz="-0.2 0.0  0.4" rpy="0.0 0.0 0.0" />
@@ -56,5 +47,5 @@
       <!-- Fake inertia -->
       <inertial>
-        <origin xyz="-0.2 0.0 0.0" rpy="0.0 0.0 0.0" />
+        <origin xyz="-0.15 0.0 0.3" rpy="0.0 0.0 0.0" />
         <mass value="15.0" />
         <inertia ixx="0.001111" ixy="0.0"      ixz="0.0"
@@ -64,11 +55,16 @@
     </link>
     <joint name="${component_name_underscore}to_${component_name_underscore}wibotic_transmitter_joint" type="fixed">
-      <!-- This should be when docking is released for panther-docker
-      <origin xyz="0.05 0.0 0.295" rpy="0.0 0.0 ${pi}" /> -->
-      <origin xyz="0.05 0.0 0.5" rpy="0.0 0.0 ${pi}" />
+      <origin xyz="0.0 0.0 ${transmitter_height}" rpy="0.0 0.0 0.0" />
       <parent link="${component_name_underscore}link" />
       <child link="${component_name_underscore}wibotic_transmitter_link" />
     </joint>
-    <link name="${component_name_underscore}wibotic_transmitter_link" />
+    <link name="${component_name_underscore}wibotic_transmitter_link">
+      <visual>
+        <origin xyz="0.0 0.0 0.0" rpy="0.0 0.0 0.0" />
+        <geometry>
+          <mesh filename="package://husarion_components_description/meshes/wibotic_transmitter.dae" />
+        </geometry>
+      </visual>
+    </link>
   </xacro:macro>
   <xacro:macro name="create_apriltag"
@@ -92,10 +88,4 @@
     </joint>
     <link name="${component_name_underscore}${name}_image_link">
-      <collision>
-        <origin xyz="0 0 0" rpy="0 ${pi/2.0} 0" />
-        <geometry>
-          <box size="${size+0.02} ${size+0.02} 0.0001" />
-        </geometry>
-      </collision>
       <visual>
         <origin xyz="0 0 0" rpy="0 ${pi/2.0} 0" />
@@ -107,9 +97,10 @@
         </material>
       </visual>
-      <inertial>
-        <mass value="1e-5" />
-        <origin xyz="0 0 0" rpy="0 0 0" />
-        <inertia ixx="1e-6" ixy="0" ixz="0" iyy="1e-6" iyz="0" izz="1e-6" />
-      </inertial>
+      <collision>
+        <origin xyz="0 0 0" rpy="0 ${pi/2.0} 0" />
+        <geometry>
+          <box size="${size+0.02} ${size+0.02} 0.0001" />
+        </geometry>
+      </collision>
     </link>
     <gazebo reference="${component_name_underscore}${name}_image_link">
@@ -132,5 +123,5 @@
     <xacro:wibotic_station
       component_name="$(arg component_name)" parent_link="${component_name_underscore}${name}_image_link"  xyz="0.0 0.0 0.5"
-      rpy="${pi} 0 0 " />
+      rpy="${pi} 0 0" transmitter_height="$(arg transmitter_height)" />
   </xacro:macro>
   <xacro:create_apriltag name="apriltag" component_name="$(arg component_name)" size="$(arg apriltag_size)" />
