Commit message: Add meshes (#13)
* Add Ouster mesh

* Add wibotic meshes and fixes

* Make wibotic station more universal (change root_link, edit height of elements)

* Fix pre-commit

* Fix test

* Fix collistion

* apriltag_height -> apriltag_mount_height

File: urdf/ouster.urdf.xacro (robot description, xacro)
@@ -71,24 +71,14 @@
     </joint>
     <link name="${component_name_underscore_nonempty}link">
-      <!-- <visual>
+      <visual>
         <origin xyz="0.0 0.0 0.0" rpy="0.0 0.0 0.0" />
         <geometry>
           <mesh filename="package://husarion_components_description/meshes/${mesh}.dae" />
         </geometry>
-      </visual> -->
-      <!-- TODO Remove simple visuals when mesh is ready -->
-      <visual>
-        <origin xyz="0.0 0.0 ${0.072/2.0}" rpy="0.0 0.0 0.0" />
-        <geometry>
-          <cylinder radius="${0.085/2.0}" length="0.073" />
-        </geometry>
-        <material name="LightGrey">
-          <color rgba="0.6 0.6 0.6 1.0" />
-        </material>
       </visual>
       <collision>
-        <origin xyz="0.0 0.0 ${0.072/2.0}" rpy="0.0 0.0 0.0" />
+        <origin xyz="0.0 0.0 ${0.015+0.074/2.0}" rpy="0.0 0.0 0.0" />
         <geometry>
-          <cylinder radius="${0.085/2.0}" length="0.073" />
+          <cylinder radius="${0.085/2.0}" length="${0.015+0.074}" /> <!-- base + lidar height -->
         </geometry>
       </collision>

File: urdf/wibotic_receiver.urdf.xacro (robot description, xacro)
@@ -27,37 +27,18 @@
       <origin xyz="${xyz}" rpy="${rpy}" />
       <parent link="${parent_link}" />
-      <child link="${component_name_underscore}link" />
+      <child link="${component_name_underscore}mount_link" />
     </joint>
-    <link name="${component_name_underscore}link">
-      <!-- <visual>
-        <origin xyz="0.0 0.0 0.0" rpy="0.0 0.0 ${pi/2.0}" />
+    <link name="${component_name_underscore}mount_link">
+      <visual>
+        <origin xyz="0.01 0.0 0.0" rpy="0.0 0.0 0.0" />
         <geometry>
-          <mesh filename="package://husarion_components_description/meshes/wibotic_receiver.stl" />
+          <mesh filename="package://husarion_components_description/meshes/wibotic_receiver.dae" />
         </geometry>
         <material name="Grey">
           <color rgba="0.15 0.15 0.15 1.0" />
         </material>
-      </visual> -->
-      <!-- TODO Remove simple visuals when mesh is ready -->
-      <visual>
-        <origin xyz="-0.008 0.0 0.085" rpy="0.0 0.0 0.0" />
-        <geometry>
-          <box size="0.015 0.135 0.19" />
-        </geometry>
-        <material name="DarkGrey">
-          <color rgba="0.2 0.2 0.2 1.0" />
-        </material>
-      </visual>
-      <visual>
-        <origin xyz="0.014 0.0 0.115" rpy="0.0 ${pi/2.0} 0.0" />
-        <geometry>
-          <cylinder length="0.03" radius="0.07" />
-        </geometry>
-        <material name="DarkGrey">
-          <color rgba="0.2 0.2 0.2 1.0" />
-        </material>
       </visual>
       <collision>
-        <origin xyz="-0.008 0.0 0.085" rpy="0.0 0.0 0.0" />
+        <origin xyz="-0.018 0.0 0.085" rpy="0.0 0.0 0.0" />
         <geometry>
           <box size="0.015 0.135 0.19" />
@@ -65,5 +46,5 @@
       </collision>
       <collision>
-        <origin xyz="0.014 0.0 0.115" rpy="0.0 ${pi/2.0} 0.0" />
+        <origin xyz="0.004 0.0 0.115" rpy="0.0 ${pi/2} 0.0" />
         <geometry>
           <cylinder length="0.03" radius="0.07" />
@@ -71,4 +52,10 @@
       </collision>
     </link>
+    <joint name="${component_name_underscore}mount_link_to_${component_name_underscore}coil_joint" type="fixed">
+      <origin xyz="0.018 0.0 0.115" rpy="0.0 0.0 0.0" />
+      <parent link="${component_name_underscore}mount_link" />
+      <child link="${component_name_underscore}coil_link" />
+    </joint>
+    <link name="${component_name_underscore}coil_link" />
   </xacro:macro>
 </robot>

File: urdf/wibotic_station.urdf.xacro (robot description, xacro)
@@ -13,48 +13,46 @@
 -->
 <robot xmlns:xacro="http://www.ros.org/wiki/xacro" name="wibotic_station">
+  <xacro:arg name="apriltag_mount_height" default="0.5" />
+  <xacro:arg name="apriltag_image" default="" />
+  <xacro:arg name="apriltag_size" default="0.08" />
   <xacro:arg name="component_name" default="" />
-  <xacro:arg name="apriltag_image_path" default="" />
-  <xacro:arg name="apriltag_size" default="0.07" />
-  <xacro:macro name="wibotic_station"
+  <xacro:arg name="root_link" default="apriltag_link" />
+  <xacro:arg name="transmitter_height" default="0.3" />
+  <!-- The AprilTag serves as the root element of the Wibotic Station.
+       This design ensures that docking functionality can detect stations via AprilTags,
+       and maintains a single root in the TF tree for proper frame hierarchy.
+       You can change the root manipulating root_link, parent_link, xyz and rpy parameters -->
+    <xacro:macro name="wibotic_station"
                params="parent_link
                        xyz:='0.0 0.0 0.0'
                        rpy:='0.0 0.0 0.0'
-                       component_name:=''">
+                       component_name:=''
+                       transmitter_height:=0.3">
     <xacro:if value="${component_name == ''}">
       <xacro:property name="component_name" value="wibotic_station" />
     </xacro:if>
     <xacro:property name="component_name_underscore" value="${component_name + '_' if component_name != '' else ''}" />
-    <joint name="${parent_link.rstrip('_link')}_to_${component_name_underscore}joint" type="fixed">
+    <joint name="${parent_link}to_${component_name_underscore}wibotic_station_link_joint" type="fixed">
       <origin xyz="${xyz}" rpy="${rpy}" />
       <parent link="${parent_link}" />
-      <child link="${component_name_underscore}link" />
+      <child link="${component_name_underscore}wibotic_station_link" />
     </joint>
-    <link name="${component_name_underscore}link">
-      <!-- <visual>
-        <origin xyz="0.0 0.0 0.0" rpy="0.0 0.0 ${pi/2.0}" />
+    <link name="${component_name_underscore}wibotic_station_link">
+      <visual>
+        <origin xyz="0.0 0.0 0.0" rpy="0.0 0.0 0.0" />
         <geometry>
-          <mesh filename="package://husarion_components_description/meshes/wibotic_station.stl" />
+          <mesh filename="package://husarion_components_description/meshes/wibotic_frame.dae" />
         </geometry>
-      </visual> -->
-      <!-- TODO Remove simple visuals when mesh is ready -->
-      <visual>
-        <origin xyz="-0.2 0.0  0.4" rpy="0.0 0.0 0.0" />
+      </visual>
+      <!-- Fake collision fit to dae -->
+      <collision>
+        <origin xyz="-0.2 0.0  0.45" rpy="0.0 0.0 0.0" />
         <geometry>
-          <box size="0.4 0.5 0.8" />
-        </geometry>
-        <material name="LightGrey">
-          <color rgba="0.6 0.6 0.6 1.0" />
-        </material>
-      </visual>
-      <!-- Fake collision fit to STL -->
-      <collision>
-        <origin xyz="-0.2 0.0  0.4" rpy="0.0 0.0 0.0" />
-        <geometry>
-          <box size="0.4 0.5 0.8" />
+          <box size="0.4 0.5 0.9" />
         </geometry>
       </collision>
       <!-- Fake inertia -->
       <inertial>
-        <origin xyz="-0.2 0.0 0.0" rpy="0.0 0.0 0.0" />
+        <origin xyz="-0.2 0.0  0.45" rpy="0.0 0.0 0.0" />
         <mass value="15.0" />
         <inertia ixx="0.001111" ixy="0.0"      ixz="0.0"
@@ -63,39 +61,38 @@
       </inertial>
     </link>
-    <joint name="${component_name_underscore}to_${component_name_underscore}wibotic_transmitter_joint" type="fixed">
-      <!-- This should be when docking is released for panther-docker
-      <origin xyz="0.05 0.0 0.295" rpy="0.0 0.0 ${pi}" /> -->
-      <origin xyz="0.05 0.0 0.5" rpy="0.0 0.0 ${pi}" />
-      <parent link="${component_name_underscore}link" />
+    <joint name="${component_name_underscore}wibotic_station_link_to_${component_name_underscore}wibotic_transmitter_joint" type="fixed">
+      <origin xyz="0.0 0.0 ${transmitter_height + 0.135}" rpy="0.0 0.0 0.0" /> <!-- 0.135 is offset from mesh origin to bottom of transmitter case -->
+      <parent link="${component_name_underscore}wibotic_station_link" />
       <child link="${component_name_underscore}wibotic_transmitter_link" />
     </joint>
-    <link name="${component_name_underscore}wibotic_transmitter_link" />
+    <link name="${component_name_underscore}wibotic_transmitter_link">
+      <visual>
+        <origin xyz="0.0 0.0 0.0" rpy="0.0 0.0 0.0" />
+        <geometry>
+          <mesh filename="package://husarion_components_description/meshes/wibotic_transmitter.dae" />
+        </geometry>
+      </visual>
+    </link>
+    <!-- Additional link for as a destination for docking -->
+    <joint name="${component_name_underscore}wibotic_transmitter_link_to_${component_name_underscore}wibotic_dock_frame_joint" type="fixed">
+      <origin xyz="0.05 0.0 0.0" rpy="0.0 0.0 ${pi}" />
+      <parent link="${component_name_underscore}wibotic_transmitter_link" />
+      <child link="${component_name_underscore}wibotic_dock_frame" />
+    </joint>
+    <link name="${component_name_underscore}wibotic_dock_frame" />
   </xacro:macro>
-  <xacro:macro name="create_apriltag"
-    params="name size:=$(arg apriltag_size) component_name:=''">
+  <xacro:macro name="apriltag"
+               params="parent_link
+                       xyz:='0.0 0.0 0.0'
+                       rpy:='0.0 0.0 0.0'
+                       component_name:=''
+                       size:=0.08">
     <xacro:property name="component_name_underscore" value="${component_name + '_' if component_name != '' else ''}" />
-    <link name="${component_name_underscore}${name}_link">
-      <visual>
-        <origin xyz="0 0 0" rpy="0 0 0" />
-        <geometry>
-          <box size="${size+0.02} ${size+0.02} 0.00005" />
-        </geometry>
-        <material name="White">
-          <color rgba="1.0 1.0 1.0 1.0" />
-        </material>
-      </visual>
-      </link>
-    <joint name="${name}_to_${name}_${component_name_underscore}image_link_joint" type="fixed">
-      <origin xyz="0 0 0" rpy="0 -${pi/2.0} ${pi/2.0}" />
-      <parent link="${component_name_underscore}${name}_link" />
-      <child link="${component_name_underscore}${name}_image_link" />
+    <joint name="${parent_link}_to_${component_name_underscore}image_link_joint" type="fixed">
+      <origin xyz="${xyz}" rpy="${rpy}" />
+      <parent link="${parent_link}" />
+      <child link="${component_name_underscore}image_link" />
     </joint>
-    <link name="${component_name_underscore}${name}_image_link">
-      <collision>
-        <origin xyz="0 0 0" rpy="0 ${pi/2.0} 0" />
-        <geometry>
-          <box size="${size+0.02} ${size+0.02} 0.0001" />
-        </geometry>
-      </collision>
+    <link name="${component_name_underscore}image_link">
       <visual>
         <origin xyz="0 0 0" rpy="0 ${pi/2.0} 0" />
@@ -107,11 +104,12 @@
         </material>
       </visual>
-      <inertial>
-        <mass value="1e-5" />
-        <origin xyz="0 0 0" rpy="0 0 0" />
-        <inertia ixx="1e-6" ixy="0" ixz="0" iyy="1e-6" iyz="0" izz="1e-6" />
-      </inertial>
+      <collision>
+        <origin xyz="0 0 0" rpy="0 ${pi/2.0} 0" />
+        <geometry>
+          <box size="${size} ${size} 0.0001" />
+        </geometry>
+      </collision>
     </link>
-    <gazebo reference="${component_name_underscore}${name}_image_link">
+    <gazebo reference="${component_name_underscore}image_link">
       <visual>
         <material>
@@ -123,5 +121,5 @@
           <pbr>
             <metal>
-              <albedo_map>$(arg apriltag_image_path)</albedo_map>
+              <albedo_map>$(arg apriltag_image)</albedo_map>
             </metal>
           </pbr>
@@ -129,9 +127,13 @@
       </visual>
     </gazebo>
-    <xacro:property name="apriltag_size_prop" value="$(arg apriltag_size)" />
-    <xacro:wibotic_station
-      component_name="$(arg component_name)" parent_link="${component_name_underscore}${name}_image_link"  xyz="0.0 0.0 0.5"
-      rpy="${pi} 0 0 " />
   </xacro:macro>
-  <xacro:create_apriltag name="apriltag" component_name="$(arg component_name)" size="$(arg apriltag_size)" />
+  <xacro:property name="component_name_prop" value="$(arg component_name)" />
+  <xacro:property name="apriltag_name" value="${component_name_prop + '_apriltag' if component_name_prop != '' else 'apriltag'}" />
+  <link name="$(arg root_link)" />
+  <!-- AprilTag as root -->
+  <xacro:apriltag parent_link="$(arg root_link)" xyz="0 0 0" rpy="0 -${pi/2.0} ${pi/2.0}" component_name="${apriltag_name}" size="$(arg apriltag_size)" />
+  <xacro:wibotic_station parent_link="$(arg root_link)" xyz="0 -$(arg apriltag_mount_height) 0" rpy="${pi} -${pi/2.0} ${pi/2.0}" component_name="$(arg component_name)" transmitter_height="$(arg transmitter_height)" />
+  <!-- Station as root -->
+  <!-- <xacro:wibotic_station parent_link="$(arg root_link)" component_name="$(arg component_name)" transmitter_height="$(arg transmitter_height)" />
+  <xacro:apriltag parent_link="$(arg root_link)" xyz="0 0 $(arg apriltag_mount_height)" rpy="${pi} 0 0" component_name="${apriltag_name}" size="$(arg apriltag_size)" /> -->
 </robot>

Commit message: Improve ouster diffrent version simulation

File: urdf/ouster.urdf.xacro (robot description, xacro)
@@ -33,37 +33,49 @@
     <xacro:if value="${model == 'os0_32'}">
       <xacro:property name="vfov" value="${radians(90.0)}" scope="parent" />
-      <xacro:property name="lidar_range" value="50" scope="parent"/>
+      <xacro:property name="range_min" value="50" scope="parent"/>
+      <xacro:property name="range_max" value="50" scope="parent"/>
       <xacro:property name="layers" value="32" scope="parent"/>
       <xacro:property name="mesh" value="ouster_os01" scope="parent"/>
+      <xacro:property name="precision" value="0.008" scope="parent"/>
     </xacro:if>
     <xacro:if value="${model == 'os0_64'}">
       <xacro:property name="vfov" value="${radians(90.0)}" scope="parent" />
-      <xacro:property name="lidar_range" value="50" scope="parent" />
+      <xacro:property name="range_min" value="0.4" scope="parent" />
+      <xacro:property name="range_max" value="35" scope="parent" />
       <xacro:property name="layers" value="64" scope="parent" />
       <xacro:property name="mesh" value="ouster_os01" scope="parent"/>
+      <xacro:property name="precision" value="0.008" scope="parent"/>
     </xacro:if>
     <xacro:if value="${model == 'os0_128'}">
       <xacro:property name="vfov" value="${radians(90.0)}" scope="parent" />
-      <xacro:property name="lidar_range" value="50" scope="parent" />
+      <xacro:property name="range_min" value="0.4" scope="parent" />
+      <xacro:property name="range_max" value="35" scope="parent" />
       <xacro:property name="layers" value="128" scope="parent" />
       <xacro:property name="mesh" value="ouster_os01" scope="parent"/>
+      <xacro:property name="precision" value="0.008" scope="parent"/>
     </xacro:if>
     <xacro:if value="${model == 'os1_32'}">
-      <xacro:property name="vfov" value="${radians(45.0)}" scope="parent" />
-      <xacro:property name="lidar_range" value="120" scope="parent" />
+      <xacro:property name="vfov" value="${radians(42.4)}" scope="parent" />
+      <xacro:property name="range_min" value="0.5" scope="parent" />
+      <xacro:property name="range_max" value="90" scope="parent" />
       <xacro:property name="layers" value="32" scope="parent" />
       <xacro:property name="mesh" value="ouster_os01" scope="parent"/>
+      <xacro:property name="precision" value="0.005" scope="parent"/>
     </xacro:if>
     <xacro:if value="${model == 'os1_64'}">
-      <xacro:property name="vfov" value="${radians(45.0)}" scope="parent" />
-      <xacro:property name="lidar_range" value="120" scope="parent" />
+      <xacro:property name="vfov" value="${radians(42.4)}" scope="parent" />
+      <xacro:property name="range_min" value="0.5" scope="parent" />
+      <xacro:property name="range_max" value="90" scope="parent" />
       <xacro:property name="layers" value="64" scope="parent" />
       <xacro:property name="mesh" value="ouster_os01" scope="parent"/>
+      <xacro:property name="precision" value="0.005" scope="parent"/>
     </xacro:if>
     <xacro:if value="${model == 'os1_128'}">
-      <xacro:property name="vfov" value="${radians(45.0)}" scope="parent" />
-      <xacro:property name="lidar_range" value="120" scope="parent" />
+      <xacro:property name="vfov" value="${radians(42.4)}" scope="parent" />
+      <xacro:property name="range_min" value="0.5" scope="parent" />
+      <xacro:property name="range_max" value="90" scope="parent" />
       <xacro:property name="layers" value="128" scope="parent" />
       <xacro:property name="mesh" value="ouster_os01" scope="parent"/>
+      <xacro:property name="precision" value="0.005" scope="parent"/>
     </xacro:if>
     <joint name="${parent_link.rstrip('_link')}_to_${component_name_underscore_nonempty}joint" type="fixed">
@@ -120,12 +132,12 @@
           </scan>
           <range>
-            <min>0.8</min>
-            <max>${lidar_range}</max>
-            <resolution>0.003</resolution>
+            <min>${range_min}</min>
+            <max>${range_max}</max>
+            <resolution>0.001</resolution>
           </range>
           <noise>
             <type>gaussian</type>
             <mean>0.0</mean>
-            <stddev>0.0008</stddev>
+            <stddev>${precision}</stddev>
           </noise>
         </ray>

Commit message: Fix os0-32 ranges

File: urdf/ouster.urdf.xacro (robot description, xacro)
@@ -33,6 +33,6 @@
     <xacro:if value="${model == 'os0_32'}">
       <xacro:property name="vfov" value="${radians(90.0)}" scope="parent" />
-      <xacro:property name="range_min" value="50" scope="parent"/>
-      <xacro:property name="range_max" value="50" scope="parent"/>
+      <xacro:property name="range_min" value="0.4" scope="parent"/>
+      <xacro:property name="range_max" value="35" scope="parent"/>
       <xacro:property name="layers" value="32" scope="parent"/>
       <xacro:property name="mesh" value="ouster_os01" scope="parent"/>
