Commit message: fix collision

File: urdf/reling.urdf.xacro (robot description, xacro)
@@ -47,5 +47,5 @@
          <origin xyz="${component['xyz']}" rpy="${component['rpy']}" />
         <geometry>
-          <box size="0.0202 0.0202 ${component['length']}" />
+          <box size="${component['length']} 0.0202 0.0202" />
         </geometry>
       </collision>
