Commit message: Revert zed collision

File: urdf/stereolabs_zed.urdf.xacro (robot description, xacro)
@@ -33,4 +33,10 @@
       <xacro:property name="optical_offset_x" value="-0.01" />
       <xacro:property name="mono" value="false" />
+      <xacro:property name="collision">
+        <origin xyz="${screw_offset_x-0.02} 0 ${screw_offset_z}" rpy="0.0 0.0 0.0" />
+        <geometry>
+          <box size="0.033 0.175 0.03" />
+        </geometry>
+      </xacro:property>
     </xacro:if>
     <xacro:if value="${model == 'zedm'}">
@@ -42,4 +48,10 @@
       <xacro:property name="optical_offset_x" value="0.0" />
       <xacro:property name="mono" value="false" />
+      <xacro:property name="collision">
+        <origin xyz="${screw_offset_x-0.015} 0.008 ${screw_offset_z}" rpy="0.0 0.0 0.0" />
+        <geometry>
+          <box size="0.026 0.124 0.03" />
+        </geometry>
+      </xacro:property>
     </xacro:if>
     <xacro:if value="${model == 'zed2'}">
@@ -51,4 +63,10 @@
       <xacro:property name="optical_offset_x" value="-0.01" />
       <xacro:property name="mono" value="false" />
+      <xacro:property name="collision">
+        <origin xyz="${screw_offset_x-0.02} 0 ${screw_offset_z}" rpy="0.0 0.0 0.0" />
+        <geometry>
+          <box size="0.033 0.175 0.03" />
+        </geometry>
+      </xacro:property>
     </xacro:if>
     <xacro:if value="${model == 'zed2i'}">
@@ -60,4 +78,10 @@
       <xacro:property name="optical_offset_x" value="-0.01" />
       <xacro:property name="mono" value="false" />
+      <xacro:property name="collision">
+        <origin xyz="${screw_offset_x-0.015} 0 ${screw_offset_z}" rpy="0.0 0.0 0.0" />
+        <geometry>
+          <box size="0.043 0.175 0.03" />
+        </geometry>
+      </xacro:property>
     </xacro:if>
     <xacro:if value="${model == 'zedx'}">
@@ -69,4 +93,10 @@
       <xacro:property name="optical_offset_x" value="-0.01" />
       <xacro:property name="mono" value="false" />
+      <xacro:property name="collision">
+        <origin xyz="${screw_offset_z-0.01} 0 0" rpy="0.0 0.0 0.0" />
+        <geometry>
+          <box size="0.037 0.163 0.032" />
+        </geometry>
+      </xacro:property>
     </xacro:if>
     <xacro:if value="${model == 'zedxm'}">
@@ -78,4 +108,10 @@
       <xacro:property name="optical_offset_x" value="-0.01" />
       <xacro:property name="mono" value="false" />
+      <xacro:property name="collision">
+        <origin xyz="${screw_offset_z-0.01} 0 0" rpy="0.0 0.0 0.0" />
+        <geometry>
+          <box size="0.037 0.094 0.032" />
+        </geometry>
+      </xacro:property>
     </xacro:if>
     <xacro:if value="${model == 'virtual'}">
@@ -87,4 +123,10 @@
       <xacro:property name="optical_offset_x" value="0.0" />
       <xacro:property name="mono" value="false" />
+      <xacro:property name="collision">
+        <origin xyz="${screw_offset_z-0.01} 0 0" rpy="0.0 0.0 0.0" />
+        <geometry>
+          <box size="0.05 0.25 0.25" />
+        </geometry>
+      </xacro:property>
     </xacro:if>
     <xacro:if value="${model == 'zedxonegs'}">
@@ -96,4 +138,10 @@
       <xacro:property name="optical_offset_x" value="0.0" />
       <xacro:property name="mono" value="true" />
+      <xacro:property name="collision">
+        <origin xyz="${screw_offset_z-0.01} 0 0" rpy="0.0 0.0 0.0" />
+        <geometry>
+          <box size="0.05 0.25 0.25" />
+        </geometry>
+      </xacro:property>
     </xacro:if>
     <xacro:if value="${model == 'zedxone4k'}">
@@ -105,7 +153,12 @@
       <xacro:property name="optical_offset_x" value="0.0" />
       <xacro:property name="mono" value="true" />
+      <xacro:property name="collision">
+        <origin xyz="${screw_offset_z-0.01} 0 0" rpy="0.0 0.0 0.0" />
+        <geometry>
+          <box size="0.05 0.25 0.25" />
+        </geometry>
+      </xacro:property>
     </xacro:if>
     <!-- Camera mounting point (the threaded screw hole in the bottom) -->
-        <!-- Camera mounting point (the threaded screw hole in the bottom) -->
     <link name="${device_namespace}_camera_link" />
     <joint name="${device_namespace}_base_joint" type="fixed">
@@ -125,8 +178,10 @@
         </visual>
         <collision>
-          <origin xyz="${screw_offset_x} 0 ${screw_offset_z}" rpy="0 0 0"/>
+          <xacro:insert_block name="collision" />
+          <!-- Use simple collision -->
+          <!-- <origin xyz="${screw_offset_x} 0 ${screw_offset_z}" rpy="0 0 0"/>
           <geometry>
             <mesh filename="package://zed_msgs/meshes/${model}.stl" />
-          </geometry>
+          </geometry> -->
         </collision>
       </xacro:unless>

Commit message: Fix origin

File: urdf/stereolabs_zed.urdf.xacro (robot description, xacro)
@@ -49,5 +49,5 @@
       <xacro:property name="mono" value="false" />
       <xacro:property name="collision">
-        <origin xyz="${screw_offset_x-0.015} 0.008 ${screw_offset_z}" rpy="0.0 0.0 0.0" />
+        <origin xyz="${screw_offset_x+0.01} 0.008 ${screw_offset_z}" rpy="0.0 0.0 0.0" />
         <geometry>
           <box size="0.026 0.124 0.03" />
@@ -64,5 +64,5 @@
       <xacro:property name="mono" value="false" />
       <xacro:property name="collision">
-        <origin xyz="${screw_offset_x-0.02} 0 ${screw_offset_z}" rpy="0.0 0.0 0.0" />
+        <origin xyz="${screw_offset_x} 0 ${screw_offset_z}" rpy="0.0 0.0 0.0" />
         <geometry>
           <box size="0.033 0.175 0.03" />
@@ -79,5 +79,5 @@
       <xacro:property name="mono" value="false" />
       <xacro:property name="collision">
-        <origin xyz="${screw_offset_x-0.015} 0 ${screw_offset_z}" rpy="0.0 0.0 0.0" />
+        <origin xyz="${screw_offset_x} 0 ${screw_offset_z}" rpy="0.0 0.0 0.0" />
         <geometry>
           <box size="0.043 0.175 0.03" />
@@ -94,5 +94,5 @@
       <xacro:property name="mono" value="false" />
       <xacro:property name="collision">
-        <origin xyz="${screw_offset_z-0.01} 0 0" rpy="0.0 0.0 0.0" />
+        <origin xyz="${screw_offset_x} 0 0" rpy="0.0 0.0 0.0" />
         <geometry>
           <box size="0.037 0.163 0.032" />
@@ -109,5 +109,5 @@
       <xacro:property name="mono" value="false" />
       <xacro:property name="collision">
-        <origin xyz="${screw_offset_z-0.01} 0 0" rpy="0.0 0.0 0.0" />
+        <origin xyz="${screw_offset_z} 0 0" rpy="0.0 0.0 0.0" />
         <geometry>
           <box size="0.037 0.094 0.032" />

Commit message: Fix offset z -> x

File: urdf/stereolabs_zed.urdf.xacro (robot description, xacro)
@@ -109,5 +109,5 @@
       <xacro:property name="mono" value="false" />
       <xacro:property name="collision">
-        <origin xyz="${screw_offset_z} 0 0" rpy="0.0 0.0 0.0" />
+        <origin xyz="${screw_offset_x} 0 0" rpy="0.0 0.0 0.0" />
         <geometry>
           <box size="0.037 0.094 0.032" />
@@ -124,5 +124,5 @@
       <xacro:property name="mono" value="false" />
       <xacro:property name="collision">
-        <origin xyz="${screw_offset_z-0.01} 0 0" rpy="0.0 0.0 0.0" />
+        <origin xyz="${screw_offset_x} 0 0" rpy="0.0 0.0 0.0" />
         <geometry>
           <box size="0.05 0.25 0.25" />
@@ -139,5 +139,5 @@
       <xacro:property name="mono" value="true" />
       <xacro:property name="collision">
-        <origin xyz="${screw_offset_z-0.01} 0 0" rpy="0.0 0.0 0.0" />
+        <origin xyz="${screw_offset_x} 0 0" rpy="0.0 0.0 0.0" />
         <geometry>
           <box size="0.05 0.25 0.25" />
@@ -154,5 +154,5 @@
       <xacro:property name="mono" value="true" />
       <xacro:property name="collision">
-        <origin xyz="${screw_offset_z-0.01} 0 0" rpy="0.0 0.0 0.0" />
+        <origin xyz="${screw_offset_x} 0 0" rpy="0.0 0.0 0.0" />
         <geometry>
           <box size="0.05 0.25 0.25" />

Commit message: Update urdf/stereolabs_zed.urdf.xacro

File: urdf/stereolabs_zed.urdf.xacro (robot description, xacro)
@@ -156,5 +156,5 @@
         <origin xyz="${screw_offset_x} 0 0" rpy="0.0 0.0 0.0" />
         <geometry>
-          <box size="0.05 0.25 0.25" />
+          <box size="0.058 0.03 0.03" />
         </geometry>
       </xacro:property>

Commit message: Apply suggestions from code review

File: urdf/stereolabs_zed.urdf.xacro (robot description, xacro)
@@ -126,5 +126,5 @@
         <origin xyz="${screw_offset_x} 0 0" rpy="0.0 0.0 0.0" />
         <geometry>
-          <box size="0.05 0.25 0.25" />
+          <box size="0.05 0.03 0.03" />
         </geometry>
       </xacro:property>
@@ -141,5 +141,5 @@
         <origin xyz="${screw_offset_x} 0 0" rpy="0.0 0.0 0.0" />
         <geometry>
-          <box size="0.05 0.25 0.25" />
+          <box size="0.052 0.03 0.03" />
         </geometry>
       </xacro:property>

Commit message: Apply suggestions from code review

File: urdf/stereolabs_zed.urdf.xacro (robot description, xacro)
@@ -141,5 +141,5 @@
         <origin xyz="${screw_offset_x} 0 0" rpy="0.0 0.0 0.0" />
         <geometry>
-          <box size="0.052 0.03 0.03" />
+          <box size="0.052 0.031 0.031" />
         </geometry>
       </xacro:property>
@@ -156,5 +156,5 @@
         <origin xyz="${screw_offset_x} 0 0" rpy="0.0 0.0 0.0" />
         <geometry>
-          <box size="0.058 0.03 0.03" />
+          <box size="0.058 0.031 0.031" />
         </geometry>
       </xacro:property>

Commit message: Remove stereolabs materials

File: urdf/stereolabs_zed.urdf.xacro (robot description, xacro)
@@ -15,5 +15,4 @@
 <!-- Reference: https://github.com/stereolabs/zed-ros2-wrapper/blob/master/zed_wrapper/urdf/zed_macro.urdf.xacro -->
 <robot xmlns:xacro="http://wiki.ros.org/xacro">
-  <xacro:include filename="$(find husarion_components_description)/urdf/include/stereolabs_zed_materials.urdf.xacro" />
   <xacro:property name="M_PI" value="3.1415926535897931" />
   <xacro:macro name="zed_camera"
@@ -79,5 +78,5 @@
       <xacro:property name="mono" value="false" />
       <xacro:property name="collision">
-        <origin xyz="${screw_offset_x} 0 ${screw_offset_z}" rpy="0.0 0.0 0.0" />
+        <origin xyz="${screw_offset_x+0.005} 0 ${screw_offset_z}" rpy="0.0 0.0 0.0" />
         <geometry>
           <box size="0.043 0.175 0.03" />
@@ -94,5 +93,5 @@
       <xacro:property name="mono" value="false" />
       <xacro:property name="collision">
-        <origin xyz="${screw_offset_x} 0 0" rpy="0.0 0.0 0.0" />
+        <origin xyz="${screw_offset_x-0.005} 0 0" rpy="0.0 0.0 0.0" />
         <geometry>
           <box size="0.037 0.163 0.032" />
@@ -109,5 +108,5 @@
       <xacro:property name="mono" value="false" />
       <xacro:property name="collision">
-        <origin xyz="${screw_offset_x} 0 0" rpy="0.0 0.0 0.0" />
+        <origin xyz="${screw_offset_x-0.015} 0 0" rpy="0.0 0.0 0.0" />
         <geometry>
           <box size="0.037 0.094 0.032" />
@@ -175,5 +174,7 @@
           <mesh filename="package://zed_msgs/meshes/${model}.stl" />
           </geometry>
-          <material name="${model}_mat" />
+          <material name="mat">
+            <color rgba="0.25 0.25 0.25 0.99" />
+          </material>
         </visual>
         <collision>
@@ -201,5 +202,7 @@
               <mesh filename="package://zed_msgs/meshes/${model}.stl" />
             </geometry>
-            <material name="${model}_mat" />
+            <material name="mat">
+              <color rgba="0.25 0.25 0.25 0.99" />
+            </material>
           </visual>
           <collision>
@@ -230,5 +233,7 @@
               <mesh filename="package://zed_msgs/meshes/${model}.stl" />
             </geometry>
-            <material name="${model}_mat" />
+            <material name="mat">
+              <color rgba="0.25 0.25 0.25 0.99" />
+            </material>
           </visual>
           <collision>

Commit message: Fix origin (#7)
* Revert zed collision

* Fix origin

* Fix offset z -> x

* comment

* Update urdf/stereolabs_zed.urdf.xacro

* Apply suggestions from code review

* Apply suggestions from code review

* Remove stereolabs materials

File: urdf/stereolabs_zed.urdf.xacro (robot description, xacro)
@@ -15,5 +15,4 @@
 <!-- Reference: https://github.com/stereolabs/zed-ros2-wrapper/blob/master/zed_wrapper/urdf/zed_macro.urdf.xacro -->
 <robot xmlns:xacro="http://wiki.ros.org/xacro">
-  <xacro:include filename="$(find husarion_components_description)/urdf/include/stereolabs_zed_materials.urdf.xacro" />
   <xacro:property name="M_PI" value="3.1415926535897931" />
   <xacro:macro name="zed_camera"
@@ -33,4 +32,10 @@
       <xacro:property name="optical_offset_x" value="-0.01" />
       <xacro:property name="mono" value="false" />
+      <xacro:property name="collision">
+        <origin xyz="${screw_offset_x-0.02} 0 ${screw_offset_z}" rpy="0.0 0.0 0.0" />
+        <geometry>
+          <box size="0.033 0.175 0.03" />
+        </geometry>
+      </xacro:property>
     </xacro:if>
     <xacro:if value="${model == 'zedm'}">
@@ -42,4 +47,10 @@
       <xacro:property name="optical_offset_x" value="0.0" />
       <xacro:property name="mono" value="false" />
+      <xacro:property name="collision">
+        <origin xyz="${screw_offset_x+0.01} 0.008 ${screw_offset_z}" rpy="0.0 0.0 0.0" />
+        <geometry>
+          <box size="0.026 0.124 0.03" />
+        </geometry>
+      </xacro:property>
     </xacro:if>
     <xacro:if value="${model == 'zed2'}">
@@ -51,4 +62,10 @@
       <xacro:property name="optical_offset_x" value="-0.01" />
       <xacro:property name="mono" value="false" />
+      <xacro:property name="collision">
+        <origin xyz="${screw_offset_x} 0 ${screw_offset_z}" rpy="0.0 0.0 0.0" />
+        <geometry>
+          <box size="0.033 0.175 0.03" />
+        </geometry>
+      </xacro:property>
     </xacro:if>
     <xacro:if value="${model == 'zed2i'}">
@@ -60,4 +77,10 @@
       <xacro:property name="optical_offset_x" value="-0.01" />
       <xacro:property name="mono" value="false" />
+      <xacro:property name="collision">
+        <origin xyz="${screw_offset_x+0.005} 0 ${screw_offset_z}" rpy="0.0 0.0 0.0" />
+        <geometry>
+          <box size="0.043 0.175 0.03" />
+        </geometry>
+      </xacro:property>
     </xacro:if>
     <xacro:if value="${model == 'zedx'}">
@@ -69,4 +92,10 @@
       <xacro:property name="optical_offset_x" value="-0.01" />
       <xacro:property name="mono" value="false" />
+      <xacro:property name="collision">
+        <origin xyz="${screw_offset_x-0.005} 0 0" rpy="0.0 0.0 0.0" />
+        <geometry>
+          <box size="0.037 0.163 0.032" />
+        </geometry>
+      </xacro:property>
     </xacro:if>
     <xacro:if value="${model == 'zedxm'}">
@@ -78,4 +107,10 @@
       <xacro:property name="optical_offset_x" value="-0.01" />
       <xacro:property name="mono" value="false" />
+      <xacro:property name="collision">
+        <origin xyz="${screw_offset_x-0.015} 0 0" rpy="0.0 0.0 0.0" />
+        <geometry>
+          <box size="0.037 0.094 0.032" />
+        </geometry>
+      </xacro:property>
     </xacro:if>
     <xacro:if value="${model == 'virtual'}">
@@ -87,4 +122,10 @@
       <xacro:property name="optical_offset_x" value="0.0" />
       <xacro:property name="mono" value="false" />
+      <xacro:property name="collision">
+        <origin xyz="${screw_offset_x} 0 0" rpy="0.0 0.0 0.0" />
+        <geometry>
+          <box size="0.05 0.03 0.03" />
+        </geometry>
+      </xacro:property>
     </xacro:if>
     <xacro:if value="${model == 'zedxonegs'}">
@@ -96,4 +137,10 @@
       <xacro:property name="optical_offset_x" value="0.0" />
       <xacro:property name="mono" value="true" />
+      <xacro:property name="collision">
+        <origin xyz="${screw_offset_x} 0 0" rpy="0.0 0.0 0.0" />
+        <geometry>
+          <box size="0.052 0.031 0.031" />
+        </geometry>
+      </xacro:property>
     </xacro:if>
     <xacro:if value="${model == 'zedxone4k'}">
@@ -105,7 +152,12 @@
       <xacro:property name="optical_offset_x" value="0.0" />
       <xacro:property name="mono" value="true" />
+      <xacro:property name="collision">
+        <origin xyz="${screw_offset_x} 0 0" rpy="0.0 0.0 0.0" />
+        <geometry>
+          <box size="0.058 0.031 0.031" />
+        </geometry>
+      </xacro:property>
     </xacro:if>
     <!-- Camera mounting point (the threaded screw hole in the bottom) -->
-        <!-- Camera mounting point (the threaded screw hole in the bottom) -->
     <link name="${device_namespace}_camera_link" />
     <joint name="${device_namespace}_base_joint" type="fixed">
@@ -122,11 +174,15 @@
           <mesh filename="package://zed_msgs/meshes/${model}.stl" />
           </geometry>
-          <material name="${model}_mat" />
+          <material name="mat">
+            <color rgba="0.25 0.25 0.25 0.99" />
+          </material>
         </visual>
         <collision>
-          <origin xyz="${screw_offset_x} 0 ${screw_offset_z}" rpy="0 0 0"/>
+          <!-- <origin xyz="${screw_offset_x} 0 ${screw_offset_z}" rpy="0 0 0"/>
           <geometry>
             <mesh filename="package://zed_msgs/meshes/${model}.stl" />
-          </geometry>
+          </geometry> -->
+          <!-- Use simple collision instead default stl -->
+          <xacro:insert_block name="collision" />
         </collision>
       </xacro:unless>
@@ -146,5 +202,7 @@
               <mesh filename="package://zed_msgs/meshes/${model}.stl" />
             </geometry>
-            <material name="${model}_mat" />
+            <material name="mat">
+              <color rgba="0.25 0.25 0.25 0.99" />
+            </material>
           </visual>
           <collision>
@@ -175,5 +233,7 @@
               <mesh filename="package://zed_msgs/meshes/${model}.stl" />
             </geometry>
-            <material name="${model}_mat" />
+            <material name="mat">
+              <color rgba="0.25 0.25 0.25 0.99" />
+            </material>
           </visual>
           <collision>
