Commit message: Add zed description

File: urdf/stereolabs_zed.urdf.xacro (robot description, xacro)
@@ -31,283 +31,15 @@
     <xacro:property name="component_name_underscore" value="${component_name + '_' if component_name != '' else ''}" />
     <xacro:property name="component_name_slash" value="${component_name + '/' if component_name != '' else ''}" />
-    <xacro:if value="${model == 'zed'}">
-      <xacro:property name="baseline" value="0.12" />
-      <xacro:property name="height" value="0.03" />
-      <xacro:property name="bottom_slope" value="0.05" />
-      <xacro:property name="screw_offset_x" value="0.0" />
-      <xacro:property name="screw_offset_z" value="0.0" />
-      <xacro:property name="optical_offset_x" value="-0.01" />
-      <xacro:property name="mono" value="false" />
-      <xacro:property name="collision">
-        <origin xyz="${screw_offset_x-0.02} 0 ${screw_offset_z}" rpy="0.0 0.0 0.0" />
-        <geometry>
-          <box size="0.033 0.175 0.03" />
-        </geometry>
-      </xacro:property>
-    </xacro:if>
-    <xacro:if value="${model == 'zedm'}">
-      <xacro:property name="baseline" value="0.063" />
-      <xacro:property name="height" value="0.0265" />
-      <xacro:property name="bottom_slope" value="0.0" />
-      <xacro:property name="screw_offset_x" value="0.0" />
-      <xacro:property name="screw_offset_z" value="0.0" />
-      <xacro:property name="optical_offset_x" value="0.0" />
-      <xacro:property name="mono" value="false" />
-      <xacro:property name="collision">
-        <origin xyz="${screw_offset_x+0.01} 0.008 ${screw_offset_z}" rpy="0.0 0.0 0.0" />
-        <geometry>
-          <box size="0.026 0.124 0.03" />
-        </geometry>
-      </xacro:property>
-    </xacro:if>
-    <xacro:if value="${model == 'zed2'}">
-      <xacro:property name="baseline" value="0.12" />
-      <xacro:property name="height" value="0.03" />
-      <xacro:property name="bottom_slope" value="0.05" />
-      <xacro:property name="screw_offset_x" value="0.0" />
-      <xacro:property name="screw_offset_z" value="0.0" />
-      <xacro:property name="optical_offset_x" value="-0.01" />
-      <xacro:property name="mono" value="false" />
-      <xacro:property name="collision">
-        <origin xyz="${screw_offset_x} 0 ${screw_offset_z}" rpy="0.0 0.0 0.0" />
-        <geometry>
-          <box size="0.033 0.175 0.03" />
-        </geometry>
-      </xacro:property>
-    </xacro:if>
-    <xacro:if value="${model == 'zed2i'}">
-      <xacro:property name="baseline" value="0.12" />
-      <xacro:property name="height" value="0.03" />
-      <xacro:property name="bottom_slope" value="0.0" />
-      <xacro:property name="screw_offset_x" value="-0.01" />
-      <xacro:property name="screw_offset_z" value="0.0" />
-      <xacro:property name="optical_offset_x" value="-0.01" />
-      <xacro:property name="mono" value="false" />
-      <xacro:property name="collision">
-        <origin xyz="${screw_offset_x+0.005} 0 ${screw_offset_z}" rpy="0.0 0.0 0.0" />
-        <geometry>
-          <box size="0.043 0.175 0.03" />
-        </geometry>
-      </xacro:property>
-    </xacro:if>
-    <xacro:if value="${model == 'zedx'}">
-      <xacro:property name="baseline" value="0.12" />
-      <xacro:property name="height" value="0.032" />
-      <xacro:property name="bottom_slope" value="0.0" />
-      <xacro:property name="screw_offset_x" value="0.0" />
-      <xacro:property name="screw_offset_z" value="-0.016" />
-      <xacro:property name="optical_offset_x" value="-0.01" />
-      <xacro:property name="mono" value="false" />
-      <xacro:property name="collision">
-        <origin xyz="${screw_offset_x-0.005} 0 0" rpy="0.0 0.0 0.0" />
-        <geometry>
-          <box size="0.037 0.163 0.032" />
-        </geometry>
-      </xacro:property>
-    </xacro:if>
-    <xacro:if value="${model == 'zedxm'}">
-      <xacro:property name="baseline" value="0.05" />
-      <xacro:property name="height" value="0.032" />
-      <xacro:property name="bottom_slope" value="0.0" />
-      <xacro:property name="screw_offset_x" value="0.0" />
-      <xacro:property name="screw_offset_z" value="-0.016" />
-      <xacro:property name="optical_offset_x" value="-0.01" />
-      <xacro:property name="mono" value="false" />
-      <xacro:property name="collision">
-        <origin xyz="${screw_offset_x-0.015} 0 0" rpy="0.0 0.0 0.0" />
-        <geometry>
-          <box size="0.037 0.094 0.032" />
-        </geometry>
-      </xacro:property>
-    </xacro:if>
-    <xacro:if value="${model == 'virtual'}">
-      <xacro:property name="baseline" value="${custom_baseline}" />
-      <xacro:property name="height" value="0.031" />
-      <xacro:property name="bottom_slope" value="0.0" />
-      <xacro:property name="screw_offset_x" value="0.00" />
-      <xacro:property name="screw_offset_z" value="-0.0155" />
-      <xacro:property name="optical_offset_x" value="0.0" />
-      <xacro:property name="mono" value="false" />
-      <xacro:property name="collision">
-        <origin xyz="${screw_offset_x} 0 0" rpy="0.0 0.0 0.0" />
-        <geometry>
-          <box size="0.05 0.03 0.03" />
-        </geometry>
-      </xacro:property>
-    </xacro:if>
-    <xacro:if value="${model == 'zedxonegs'}">
-      <xacro:property name="baseline" value="0.0" />
-      <xacro:property name="height" value="0.031" />
-      <xacro:property name="bottom_slope" value="0.0" />
-      <xacro:property name="screw_offset_x" value="0.0" />
-      <xacro:property name="screw_offset_z" value="-0.0155" />
-      <xacro:property name="optical_offset_x" value="0.0" />
-      <xacro:property name="mono" value="true" />
-      <xacro:property name="collision">
-        <origin xyz="${screw_offset_x} 0 0" rpy="0.0 0.0 0.0" />
-        <geometry>
-          <box size="0.052 0.031 0.031" />
-        </geometry>
-      </xacro:property>
-    </xacro:if>
-    <xacro:if value="${model == 'zedxone4k'}">
-      <xacro:property name="baseline" value="0.0" />
-      <xacro:property name="height" value="0.031" />
-      <xacro:property name="bottom_slope" value="0.0" />
-      <xacro:property name="screw_offset_x" value="0.00" />
-      <xacro:property name="screw_offset_z" value="-0.0155" />
-      <xacro:property name="optical_offset_x" value="0.0" />
-      <xacro:property name="mono" value="true" />
-      <xacro:property name="collision">
-        <origin xyz="${screw_offset_x} 0 0" rpy="0.0 0.0 0.0" />
-        <geometry>
-          <box size="0.058 0.031 0.031" />
-        </geometry>
-      </xacro:property>
-    </xacro:if>
-    <!-- Camera mounting point (the threaded screw hole in the bottom) -->
-    <link name="${component_name_underscore}link" />
-    <joint name="${parent_link.rstrip('_link')}_to_${component_name_underscore}joint" type="fixed">
-      <parent link="${parent_link}" />
-      <child link="${component_name_underscore}link" />
+    <xacro:include filename="$(find zed_description)/urdf/zed_macro.urdf.xacro" />
+    <joint name="${parent_link}_to_${component_name_underscore}joint" type="fixed">
       <origin xyz="${xyz}" rpy="${rpy}" />
+      <parent link="${parent_link}"/>
+      <child link="${component_name}_camera_link" />
     </joint>
-    <!-- Camera Center -->
-    <link name="${component_name_underscore}camera_center">
-      <xacro:unless value="${model == 'virtual'}">
-        <visual>
-          <origin xyz="${screw_offset_x} 0 ${screw_offset_z}" rpy="0 0 0"/>
-          <geometry>
-          <mesh filename="package://zed_msgs/meshes/${model}.stl" />
-          </geometry>
-          <material name="mat">
-            <color rgba="0.25 0.25 0.25 0.99" />
-          </material>
-        </visual>
-        <collision>
-          <!-- <origin xyz="${screw_offset_x} 0 ${screw_offset_z}" rpy="0 0 0"/>
-          <geometry>
-            <mesh filename="package://zed_msgs/meshes/${model}.stl" />
-          </geometry> -->
-          <!-- Use simple collision instead default stl -->
-          <xacro:insert_block name="collision" />
-        </collision>
-      </xacro:unless>
-    </link>
-    <joint name="${component_name_underscore}to_${component_name_underscore}camera_center_joint" type="fixed">
-      <parent link="${component_name_underscore}link"/>
-      <child link="${component_name_underscore}camera_center"/>
-      <origin xyz="0 0 ${height/2}" rpy="0 ${bottom_slope} 0" />
-    </joint>
-    <xacro:unless value="${mono}">
-      <!-- Left Camera -->
-      <link name="${component_name_underscore}left_camera_frame">
-        <xacro:if value="${model == 'virtual'}">
-          <visual>
-            <origin xyz="0 0 0" rpy="0 0 0"/>
-            <geometry>
-              <mesh filename="package://zed_msgs/meshes/${model}.stl" />
-            </geometry>
-            <material name="mat">
-              <color rgba="0.25 0.25 0.25 0.99" />
-            </material>
-          </visual>
-          <collision>
-            <origin xyz="0 0 0" rpy="0 0 0"/>
-            <geometry>
-              <mesh filename="package://zed_msgs/meshes/${model}.stl" />
-            </geometry>
-          </collision>
-        </xacro:if>
-      </link>
-      <joint name="${component_name_underscore}left_camera_joint" type="fixed">
-        <parent link="${component_name_underscore}camera_center"/>
-        <child link="${component_name_underscore}left_camera_frame"/>
-        <origin xyz="${optical_offset_x} ${baseline/2} 0" rpy="0 0 0" />
-      </joint>
-      <link name="${component_name_underscore}left_camera_optical_frame"/>
-      <joint name="${component_name_underscore}left_camera_optical_joint" type="fixed">
-        <origin xyz="0 0 0" rpy="-${M_PI/2} 0.0 -${M_PI/2}"/>
-        <parent link="${component_name_underscore}left_camera_frame"/>
-        <child link="${component_name_underscore}left_camera_optical_frame"/>
-      </joint>
-      <!-- Right Camera -->
-      <link name="${component_name_underscore}right_camera_frame">
-        <xacro:if value="${model == 'virtual'}">
-          <visual>
-            <origin xyz="0 0 0" rpy="0 0 0"/>
-            <geometry>
-              <mesh filename="package://zed_msgs/meshes/${model}.stl" />
-            </geometry>
-            <material name="mat">
-              <color rgba="0.25 0.25 0.25 0.99" />
-            </material>
-          </visual>
-          <collision>
-            <origin xyz="0 0 0" rpy="0 0 0"/>
-            <geometry>
-              <mesh filename="package://zed_msgs/meshes/${model}.stl" />
-            </geometry>
-          </collision>
-        </xacro:if>
-      </link>
-      <joint name="${component_name_underscore}right_camera_joint" type="fixed">
-        <parent link="${component_name_underscore}camera_center"/>
-        <child link="${component_name_underscore}right_camera_frame"/>
-        <origin xyz="${optical_offset_x} -${baseline/2} 0" rpy="0 0 0" />
-      </joint>
-      <link name="${component_name_underscore}right_camera_optical_frame"/>
-      <joint name="${component_name_underscore}right_camera_optical_joint" type="fixed">
-        <origin xyz="0 0 0" rpy="-${M_PI/2} 0.0 -${M_PI/2}"/>
-        <parent link="${component_name_underscore}right_camera_frame"/>
-        <child link="${component_name_underscore}right_camera_optical_frame"/>
-      </joint>
-      <!-- ZED2 Sensors -->
-      <xacro:if value="${model == 'zed2'}">
-        <link name="${component_name_underscore}mag_link" />
-        <joint name="${component_name_underscore}mag_joint" type="fixed">
-          <parent link="${component_name_underscore}camera_center"/>
-          <child link="${component_name_underscore}mag_link"/>
-          <origin xyz="0 0 0" rpy="0 0 0" />
-        </joint>
-        <link name="${component_name_underscore}baro_link" />
-        <joint name="${component_name_underscore}baro_joint" type="fixed">
-          <parent link="${component_name_underscore}camera_center"/>
-          <child link="${component_name_underscore}baro_link"/>
-          <origin xyz="0 0 0" rpy="0 0 0" />
-        </joint>
-        <link name="${component_name_underscore}temp_left_link" />
-        <joint name="${component_name_underscore}temp_left_joint" type="fixed">
-          <parent link="${component_name_underscore}left_camera_frame"/>
-          <child link="${component_name_underscore}temp_left_link"/>
-          <origin xyz="0 0 0" rpy="0 0 0" />
-        </joint>
-        <link name="${component_name_underscore}temp_right_link" />
-        <joint name="${component_name_underscore}temp_right_joint" type="fixed">
-          <parent link="${component_name_underscore}right_camera_frame"/>
-          <child link="${component_name_underscore}temp_right_link"/>
-          <origin xyz="0 0 0" rpy="0 0 0" />
-        </joint>
-      </xacro:if>
-    </xacro:unless>
-    <xacro:if value="${mono}">
-      <!-- Camera -->
-      <link name="${component_name_underscore}camera_frame" />
-      <joint name="${component_name_underscore}camera_joint" type="fixed">
-        <parent link="${component_name_underscore}camera_center"/>
-        <child link="${component_name_underscore}camera_frame"/>
-        <origin xyz="${optical_offset_x} 0 0" rpy="0 0 0" />
-      </joint>
-      <link name="${component_name_underscore}camera_optical_frame"/>
-      <joint name="${component_name_underscore}camera_optical_joint" type="fixed">
-        <origin xyz="0 0 0" rpy="-${M_PI/2} 0.0 -${M_PI/2}"/>
-        <parent link="${component_name_underscore}camera_frame"/>
-        <child link="${component_name_underscore}camera_optical_frame"/>
-      </joint>
-    </xacro:if>
+    <xacro:zed_camera name="${component_name}" model="${model}" enable_gnss="false" />
     <!-- GAZEBO -->
     <xacro:include filename="$(find husarion_components_description)/urdf/gz_sensor.urdf.xacro" ns="gz_sensor" />
     <xacro:gz_sensor.camera
-      reference="${component_name_underscore}camera_center"
+      reference="${component_name_underscore}_camera_center"
       name="${robot_namespace_slash}${component_name_underscore}camera_color"
       topic="${robot_namespace_slash}${component_name_slash}zed_node/rgb/image_rect_color"

Commit message: Bump zed_description

File: urdf/stereolabs_zed.urdf.xacro (robot description, xacro)
@@ -29,20 +29,20 @@
     <xacro:property name="robot_namespace_slash" value="${robot_namespace + '/' if robot_namespace != '' else ''}" />
     <xacro:property name="tf_prefix" value="${robot_namespace_slash if use_tf_prefix in ['True', True] else ''}" />
-    <xacro:property name="component_name_underscore" value="${component_name + '_' if component_name != '' else ''}" />
-    <xacro:property name="component_name_slash" value="${component_name + '/' if component_name != '' else ''}" />
     <xacro:include filename="$(find zed_description)/urdf/zed_macro.urdf.xacro" />
-    <joint name="${parent_link}_to_${component_name_underscore}joint" type="fixed">
+    <joint name="${parent_link}_to_${component_name}_joint" type="fixed">
       <origin xyz="${xyz}" rpy="${rpy}" />
       <parent link="${parent_link}"/>
       <child link="${component_name}_camera_link" />
     </joint>
-    <xacro:zed_camera name="${component_name}" model="${model}" enable_gnss="false" />
+    <xacro:zed_camera name="${component_name}" model="${model}" enable_gnss="false" >
+      <origin xyz="0 0 0" rpy="0 0 0"/>
+    </xacro:zed_camera>
     <!-- GAZEBO -->
     <xacro:include filename="$(find husarion_components_description)/urdf/gz_sensor.urdf.xacro" ns="gz_sensor" />
     <xacro:gz_sensor.camera
-      reference="${component_name_underscore}camera_center"
-      name="${robot_namespace_slash}${component_name_underscore}camera_color"
-      topic="${robot_namespace_slash}${component_name_slash}zed_node/rgb/image_rect_color"
-      frame_id="${tf_prefix}${component_name_underscore}camera_center"
+      reference="${component_name}_camera_center"
+      name="${robot_namespace_slash}${component_name}_camera_color"
+      topic="${robot_namespace_slash}${component_name}/zed_node/rgb/image_rect_color"
+      frame_id="${tf_prefix}${component_name}_camera_center"
       frequency="30"
       width="1280"
@@ -50,8 +50,8 @@
       fov="${110.0/180.0*pi}" />
     <xacro:gz_sensor.depth_camera
-      reference="${component_name_underscore}camera_center"
-      name="${robot_namespace_slash}${component_name_underscore}camera_depth"
-      topic="${robot_namespace_slash}${component_name_slash}zed_node/depth"
-      frame_id="${tf_prefix}${component_name_underscore}camera_center"
+      reference="${component_name}_camera_center"
+      name="${robot_namespace_slash}${component_name}_camera_depth"
+      topic="${robot_namespace_slash}${component_name}/zed_node/depth"
+      frame_id="${tf_prefix}${component_name}_camera_center"
       frequency="30"
       width="1280"
