Commit message: Add velodyne and astra meshes; Improve rplidar: s1, s2

File: urdf/orbbec_astra.urdf.xacro (robot description, xacro)
@@ -39,28 +39,9 @@
     </joint>
     <link name="${component_name_underscore}astra_visual_frame">
-      <!-- <visual>
-        <origin xyz="0.0 0.0 0.0" rpy="0.0 0.0 0.0" />
+      <visual>
+        <origin xyz="0.0 0.0 0.0" rpy="${pi/2} 0.0 0.0" />
         <geometry>
-          <mesh filename="package://husarion_components_description/meshes/orbbec_astra.dae" />
+          <mesh filename="package://husarion_components_description/meshes/orbbec_astra.glb" />
         </geometry>
-      </visual> -->
-      <!-- TODO Remove simple visuals when mesh is ready -->
-      <visual>
-        <origin xyz="${0.0225-0.04/2.0} 0.0 ${0.019+0.03/2.0}" rpy="0.0 0.0 0.0" />
-        <geometry>
-          <box size="0.04 0.165 0.03" />
-        </geometry>
-        <material name="LightGrey">
-          <color rgba="0.6 0.6 0.6 1.0" />
-        </material>
-      </visual>
-      <visual>
-        <origin xyz="${0.0235-0.06/2.0} 0.0 ${0.019/2.0}" rpy="0.0 0.0 0.0" />
-        <geometry>
-          <box size="0.06 0.06 0.019" />
-        </geometry>
-        <material name="LightGrey">
-          <color rgba="0.6 0.6 0.6 1.0" />
-        </material>
       </visual>
       <!-- camera module collision -->

File: urdf/velodyne_puck.urdf.xacro (robot description, xacro)
@@ -36,19 +36,9 @@
     </joint>
     <link name="${component_name_underscore_nonempty}link">
-      <!-- <visual>
-        <origin xyz="0.0 0.0 0.0" rpy="0.0 0.0 0.0" />
+      <visual>
+        <origin xyz="0.0 0.0 0.0" rpy="${pi/2} 0.0 0.0" />
         <geometry>
-          <mesh filename="package://husarion_components_description/meshes/velodyne_puck.dae" />
+          <mesh filename="package://husarion_components_description/meshes/velodyne_puck.glb" />
         </geometry>
-      </visual> -->
-      <!-- TODO Remove simple visuals when mesh is ready -->
-      <visual>
-        <origin xyz="0.0 0.0 ${0.072/2.0}" rpy="0.0 0.0 0.0" />
-        <geometry>
-          <cylinder radius="${0.103/2.0}" length="0.072" />
-        </geometry>
-        <material name="LightGrey">
-          <color rgba="0.6 0.6 0.6 1.0" />
-        </material>
       </visual>
       <collision>
