Commit message: Zed add CAM05 and update ZED urdf

File: urdf/components.urdf.xacro (robot description, xacro)
@@ -107,4 +107,5 @@
           ('CAM03', 'zed2'),
           ('CAM04', 'zed2i'),
+          ('CAM05', 'zedm'),
           ('CAM06', 'zedx'),
           ])}" />

File: urdf/stereolabs_zed.urdf.xacro (robot description, xacro)
@@ -13,5 +13,7 @@
 limitations under the License.
 -->
+<!-- Reference: https://github.com/stereolabs/zed-ros2-wrapper/blob/master/zed_wrapper/urdf/zed_macro.urdf.xacro -->
 <robot xmlns:xacro="http://wiki.ros.org/xacro">
+  <xacro:include filename="$(find husarion_components_description)/urdf/include/stereolabs_zed_materials.urdf.xacro" />
   <xacro:property name="M_PI" value="3.1415926535897931" />
   <xacro:macro name="zed_camera"
@@ -30,13 +32,8 @@
       <xacro:property name="screw_offset_z" value="0.0" />
       <xacro:property name="optical_offset_x" value="-0.01" />
-      <xacro:property name="collision">
-        <origin xyz="${screw_offset_x-0.02} 0 ${screw_offset_z}" rpy="0.0 0.0 0.0" />
-        <geometry>
-          <box size="0.033 0.175 0.03" />
-        </geometry>
-      </xacro:property>
+      <xacro:property name="mono" value="false" />
     </xacro:if>
     <xacro:if value="${model == 'zedm'}">
-      <xacro:property name="baseline" value="0.06" />
+      <xacro:property name="baseline" value="0.063" />
       <xacro:property name="height" value="0.0265" />
       <xacro:property name="bottom_slope" value="0.0" />
@@ -44,10 +41,5 @@
       <xacro:property name="screw_offset_z" value="0.0" />
       <xacro:property name="optical_offset_x" value="0.0" />
-      <xacro:property name="collision">
-        <origin xyz="${screw_offset_x-0.015} 0.008 ${screw_offset_z}" rpy="0.0 0.0 0.0" />
-        <geometry>
-          <box size="0.026 0.124 0.03" />
-        </geometry>
-      </xacro:property>
+      <xacro:property name="mono" value="false" />
     </xacro:if>
     <xacro:if value="${model == 'zed2'}">
@@ -58,10 +50,5 @@
       <xacro:property name="screw_offset_z" value="0.0" />
       <xacro:property name="optical_offset_x" value="-0.01" />
-      <xacro:property name="collision">
-        <origin xyz="${screw_offset_x-0.02} 0 ${screw_offset_z}" rpy="0.0 0.0 0.0" />
-        <geometry>
-          <box size="0.033 0.175 0.03" />
-        </geometry>
-      </xacro:property>
+      <xacro:property name="mono" value="false" />
     </xacro:if>
     <xacro:if value="${model == 'zed2i'}">
@@ -72,10 +59,5 @@
       <xacro:property name="screw_offset_z" value="0.0" />
       <xacro:property name="optical_offset_x" value="-0.01" />
-      <xacro:property name="collision">
-        <origin xyz="${screw_offset_x-0.015} 0 ${screw_offset_z}" rpy="0.0 0.0 0.0" />
-        <geometry>
-          <box size="0.043 0.175 0.03" />
-        </geometry>
-      </xacro:property>
+      <xacro:property name="mono" value="false" />
     </xacro:if>
     <xacro:if value="${model == 'zedx'}">
@@ -86,10 +68,5 @@
       <xacro:property name="screw_offset_z" value="-0.016" />
       <xacro:property name="optical_offset_x" value="-0.01" />
-      <xacro:property name="collision">
-        <origin xyz="${screw_offset_z-0.01} 0 0" rpy="0.0 0.0 0.0" />
-        <geometry>
-          <box size="0.037 0.163 0.032" />
-        </geometry>
-      </xacro:property>
+      <xacro:property name="mono" value="false" />
     </xacro:if>
     <xacro:if value="${model == 'zedxm'}">
@@ -100,92 +77,164 @@
       <xacro:property name="screw_offset_z" value="-0.016" />
       <xacro:property name="optical_offset_x" value="-0.01" />
-      <xacro:property name="collision">
-        <origin xyz="${screw_offset_z-0.01} 0 0" rpy="0.0 0.0 0.0" />
-        <geometry>
-          <box size="0.037 0.094 0.032" />
-        </geometry>
-      </xacro:property>
+      <xacro:property name="mono" value="false" />
+    </xacro:if>
+    <xacro:if value="${model == 'virtual'}">
+      <xacro:property name="baseline" value="${custom_baseline}" />
+      <xacro:property name="height" value="0.031" />
+      <xacro:property name="bottom_slope" value="0.0" />
+      <xacro:property name="screw_offset_x" value="0.00" />
+      <xacro:property name="screw_offset_z" value="-0.0155" />
+      <xacro:property name="optical_offset_x" value="0.0" />
+      <xacro:property name="mono" value="false" />
+    </xacro:if>
+    <xacro:if value="${model == 'zedxonegs'}">
+      <xacro:property name="baseline" value="0.0" />
+      <xacro:property name="height" value="0.031" />
+      <xacro:property name="bottom_slope" value="0.0" />
+      <xacro:property name="screw_offset_x" value="0.0" />
+      <xacro:property name="screw_offset_z" value="-0.0155" />
+      <xacro:property name="optical_offset_x" value="0.0" />
+      <xacro:property name="mono" value="true" />
+    </xacro:if>
+    <xacro:if value="${model == 'zedxone4k'}">
+      <xacro:property name="baseline" value="0.0" />
+      <xacro:property name="height" value="0.031" />
+      <xacro:property name="bottom_slope" value="0.0" />
+      <xacro:property name="screw_offset_x" value="0.00" />
+      <xacro:property name="screw_offset_z" value="-0.0155" />
+      <xacro:property name="optical_offset_x" value="0.0" />
+      <xacro:property name="mono" value="true" />
     </xacro:if>
     <!-- Camera mounting point (the threaded screw hole in the bottom) -->
-    <link name="${device_namespace}_link" />
+        <!-- Camera mounting point (the threaded screw hole in the bottom) -->
+    <link name="${device_namespace}_camera_link" />
     <joint name="${device_namespace}_base_joint" type="fixed">
       <parent link="${parent_link}" />
-      <child link="${device_namespace}_link" />
+      <child link="${device_namespace}_camera_link" />
       <origin xyz="${xyz}" rpy="${rpy}" />
     </joint>
     <!-- Camera Center -->
-    <link name="${device_namespace}_center">
-      <visual>
-        <!-- 0.02 in x is caused because the visual model is in the frame -->
-        <origin xyz="${screw_offset_x-0.02} 0 ${screw_offset_z}" rpy="0 0 0" />
-        <geometry>
+    <link name="${device_namespace}_camera_center">
+      <xacro:unless value="${model == 'virtual'}">
+        <visual>
+          <origin xyz="${screw_offset_x} 0 ${screw_offset_z}" rpy="0 0 0"/>
+          <geometry>
           <mesh filename="package://zed_msgs/meshes/${model}.stl" />
-        </geometry>
-        <material name="mat">
-          <color rgba="0.25 0.25 0.25 0.99" />
-        </material>
-      </visual>
-      <collision>
-        <xacro:insert_block name="collision" />
-      </collision>
+          </geometry>
+          <material name="${model}_mat" />
+        </visual>
+        <collision>
+          <origin xyz="${screw_offset_x} 0 ${screw_offset_z}" rpy="0 0 0"/>
+          <geometry>
+            <mesh filename="package://zed_msgs/meshes/${model}.stl" />
+          </geometry>
+        </collision>
+      </xacro:unless>
     </link>
     <joint name="${device_namespace}_camera_center_joint" type="fixed">
-      <parent link="${device_namespace}_link" />
-      <child link="${device_namespace}_center" />
-      <!-- 0.02 in x is caused because the visual model is in the frame -->
-      <origin xyz="0.02 0 ${height/2}" rpy="0 ${bottom_slope} 0" />
+      <parent link="${device_namespace}_camera_link"/>
+      <child link="${device_namespace}_camera_center"/>
+      <origin xyz="0 0 ${height/2}" rpy="0 ${bottom_slope} 0" />
     </joint>
-    <!-- Artificially Created Camera Center -->
-    <link name="${device_namespace}_center_optical_frame" />
-    <joint name="${device_namespace}_center_joint" type="fixed">
-      <parent link="${device_namespace}_center" />
-      <child link="${device_namespace}_center_optical_frame" />
-      <origin xyz="0.0 0.0 0.0" rpy="${-pi/2.0} 0 ${-pi/2.0}" />
-    </joint>
-    <!-- Left Camera -->
-    <link name="${device_namespace}_left_camera_frame" />
-    <joint name="${device_namespace}_left_camera_joint" type="fixed">
-      <parent link="${device_namespace}_center" />
-      <child link="${device_namespace}_left_camera_frame" />
-      <origin xyz="${optical_offset_x} ${baseline/2} 0" rpy="0 0 0" />
-    </joint>
-    <link name="${device_namespace}_left_camera_optical_frame" />
-    <joint name="${device_namespace}_left_camera_optical_joint" type="fixed">
-      <origin xyz="0 0 0" rpy="-${M_PI/2} 0.0 -${M_PI/2}" />
-      <parent link="${device_namespace}_left_camera_frame" />
-      <child link="${device_namespace}_left_camera_optical_frame" />
-    </joint>
-    <!-- Right Camera -->
-    <link name="${device_namespace}_right_camera_frame" />
-    <joint name="${device_namespace}_right_camera_joint" type="fixed">
-      <parent link="${device_namespace}_center" />
-      <child link="${device_namespace}_right_camera_frame" />
-      <origin xyz="${optical_offset_x} -${baseline/2} 0" rpy="0 0 0" />
-    </joint>
-    <link name="${device_namespace}_right_camera_optical_frame" />
-    <joint name="${device_namespace}_right_camera_optical_joint" type="fixed">
-      <origin xyz="0 0 0" rpy="-${M_PI/2} 0.0 -${M_PI/2}" />
-      <parent link="${device_namespace}_right_camera_frame" />
-      <child link="${device_namespace}_right_camera_optical_frame" />
-    </joint>
-    <!-- ZED2 Sensors -->
-    <xacro:if value="${model == 'zed2'}">
-      <link name="${device_namespace}_mag_link" />
-      <joint name="${device_namespace}_mag_joint" type="fixed">
-        <parent link="${device_namespace}_center" />
-        <child link="${device_namespace}_mag_link" />
-        <origin xyz="0 0 0" rpy="0 0 0" />
-      </joint>
-      <link name="${device_namespace}_baro_link" />
-      <joint name="${device_namespace}_baro_joint" type="fixed">
-        <parent link="${device_namespace}_center" />
-        <child link="${device_namespace}_baro_link" />
-        <origin xyz="0 0 0" rpy="0 0 0" />
-      </joint>
-      <link name="${device_namespace}_temp_left_link" />
-      <joint name="${device_namespace}_temp_left_joint" type="fixed">
-        <parent link="${device_namespace}_left_camera_frame" />
-        <child link="${device_namespace}_temp_left_link" />
-        <origin xyz="0 0 0" rpy="0 0 0" />
+    <xacro:unless value="${mono}">
+      <!-- Left Camera -->
+      <link name="${device_namespace}_left_camera_frame">
+        <xacro:if value="${model == 'virtual'}">
+          <visual>
+            <origin xyz="0 0 0" rpy="0 0 0"/>
+            <geometry>
+              <mesh filename="package://zed_msgs/meshes/${model}.stl" />
+            </geometry>
+            <material name="${model}_mat" />
+          </visual>
+          <collision>
+            <origin xyz="0 0 0" rpy="0 0 0"/>
+            <geometry>
+              <mesh filename="package://zed_msgs/meshes/${model}.stl" />
+            </geometry>
+          </collision>
+        </xacro:if>
+      </link>
+      <joint name="${device_namespace}_left_camera_joint" type="fixed">
+        <parent link="${device_namespace}_camera_center"/>
+        <child link="${device_namespace}_left_camera_frame"/>
+        <origin xyz="${optical_offset_x} ${baseline/2} 0" rpy="0 0 0" />
+      </joint>
+      <link name="${device_namespace}_left_camera_optical_frame"/>
+      <joint name="${device_namespace}_left_camera_optical_joint" type="fixed">
+        <origin xyz="0 0 0" rpy="-${M_PI/2} 0.0 -${M_PI/2}"/>
+        <parent link="${device_namespace}_left_camera_frame"/>
+        <child link="${device_namespace}_left_camera_optical_frame"/>
+      </joint>
+      <!-- Right Camera -->
+      <link name="${device_namespace}_right_camera_frame">
+        <xacro:if value="${model == 'virtual'}">
+          <visual>
+            <origin xyz="0 0 0" rpy="0 0 0"/>
+            <geometry>
+              <mesh filename="package://zed_msgs/meshes/${model}.stl" />
+            </geometry>
+            <material name="${model}_mat" />
+          </visual>
+          <collision>
+            <origin xyz="0 0 0" rpy="0 0 0"/>
+            <geometry>
+              <mesh filename="package://zed_msgs/meshes/${model}.stl" />
+            </geometry>
+          </collision>
+        </xacro:if>
+      </link>
+      <joint name="${device_namespace}_right_camera_joint" type="fixed">
+        <parent link="${device_namespace}_camera_center"/>
+        <child link="${device_namespace}_right_camera_frame"/>
+        <origin xyz="${optical_offset_x} -${baseline/2} 0" rpy="0 0 0" />
+      </joint>
+      <link name="${device_namespace}_right_camera_optical_frame"/>
+      <joint name="${device_namespace}_right_camera_optical_joint" type="fixed">
+        <origin xyz="0 0 0" rpy="-${M_PI/2} 0.0 -${M_PI/2}"/>
+        <parent link="${device_namespace}_right_camera_frame"/>
+        <child link="${device_namespace}_right_camera_optical_frame"/>
+      </joint>
+      <!-- ZED2 Sensors -->
+      <xacro:if value="${model == 'zed2'}">
+        <link name="${device_namespace}_mag_link" />
+        <joint name="${device_namespace}_mag_joint" type="fixed">
+          <parent link="${device_namespace}_camera_center"/>
+          <child link="${device_namespace}_mag_link"/>
+          <origin xyz="0 0 0" rpy="0 0 0" />
+        </joint>
+        <link name="${device_namespace}_baro_link" />
+        <joint name="${device_namespace}_baro_joint" type="fixed">
+          <parent link="${device_namespace}_camera_center"/>
+          <child link="${device_namespace}_baro_link"/>
+          <origin xyz="0 0 0" rpy="0 0 0" />
+        </joint>
+        <link name="${device_namespace}_temp_left_link" />
+        <joint name="${device_namespace}_temp_left_joint" type="fixed">
+          <parent link="${device_namespace}_left_camera_frame"/>
+          <child link="${device_namespace}_temp_left_link"/>
+          <origin xyz="0 0 0" rpy="0 0 0" />
+        </joint>
+        <link name="${device_namespace}_temp_right_link" />
+        <joint name="${device_namespace}_temp_right_joint" type="fixed">
+          <parent link="${device_namespace}_right_camera_frame"/>
+          <child link="${device_namespace}_temp_right_link"/>
+          <origin xyz="0 0 0" rpy="0 0 0" />
+        </joint>
+      </xacro:if>
+    </xacro:unless>
+    <xacro:if value="${mono}">
+      <!-- Camera -->
+      <link name="${device_namespace}_camera_frame" />
+      <joint name="${device_namespace}_camera_joint" type="fixed">
+        <parent link="${device_namespace}_camera_center"/>
+        <child link="${device_namespace}_camera_frame"/>
+        <origin xyz="${optical_offset_x} 0 0" rpy="0 0 0" />
+      </joint>
+      <link name="${device_namespace}_camera_optical_frame"/>
+      <joint name="${device_namespace}_camera_optical_joint" type="fixed">
+        <origin xyz="0 0 0" rpy="-${M_PI/2} 0.0 -${M_PI/2}"/>
+        <parent link="${device_namespace}_camera_frame"/>
+        <child link="${device_namespace}_camera_optical_frame"/>
       </joint>
     </xacro:if>
@@ -193,20 +242,20 @@
     <xacro:include filename="$(find husarion_components_description)/urdf/gz_sensor.urdf.xacro" ns="gz_sensor" />
     <xacro:gz_sensor.camera
-      reference="${device_namespace}_center"
+      reference="${device_namespace}_camera_center"
       name="${ns}${device_namespace}_stereolabs_zed_color"
       topic="${ns}${device_namespace}/zed_node/rgb/image_rect_color"
-      frame_id="${ns}${device_namespace}_center_optical_frame"
+      frame_id="${ns}${device_namespace}_camera_center"
       frequency="30"
-      width="1920"
-      height="1080"
+      width="1280"
+      height="720"
       fov="${110.0/180.0*pi}" />
     <xacro:gz_sensor.depth_camera
-      reference="${device_namespace}_center"
+      reference="${device_namespace}_camera_center"
       name="${ns}${device_namespace}_stereolabs_zed_depth"
       topic="${ns}${device_namespace}/zed_node/depth"
-      frame_id="${ns}${device_namespace}_center_optical_frame"
+      frame_id="${ns}${device_namespace}_camera_center"
       frequency="30"
-      width="1920"
-      height="1080"
+      width="1280"
+      height="720"
       fov="${110.0/180.0*pi}"
       min_dist="0.3"
