Commit message: urdf: rename namespace arg to robot_namespace

File: urdf/components.urdf.xacro (robot description, xacro)
@@ -68,5 +68,5 @@
             xyz="${xyz}"
             rpy="${rpy}"
-            namespace="${ns}"
+            robot_namespace="${ns}"
             device_namespace="${device_ns}"
           />
@@ -83,5 +83,5 @@
             xyz="${xyz}"
             rpy="${rpy}"
-            namespace="${ns}"
+            robot_namespace="${ns}"
             device_namespace="${device_ns}"
           />
@@ -98,5 +98,5 @@
             xyz="${xyz}"
             rpy="${rpy}"
-            namespace="${ns}"
+            robot_namespace="${ns}"
             device_namespace="${device_ns}"
             use_nominal_extrinsics="${use_sim}"
@@ -121,5 +121,5 @@
             xyz="${xyz}"
             rpy="${rpy}"
-            namespace="${ns}"
+            robot_namespace="${ns}"
             device_namespace="${device_ns}"
             model="${zed_models_dict[type]}"
@@ -142,5 +142,5 @@
             xyz="${xyz}"
             rpy="${rpy}"
-            namespace="${ns}"
+            robot_namespace="${ns}"
             device_namespace="${device_ns}"
             model="${luxonis_models_dict[type]}"
@@ -164,5 +164,5 @@
             xyz="${xyz}"
             rpy="${rpy}"
-            namespace="${ns}"
+            robot_namespace="${ns}"
             device_namespace="${device_ns}"
             model="${rplidar_models_dict[type]}"
@@ -187,5 +187,5 @@
             xyz="${xyz}"
             rpy="${rpy}"
-            namespace="${ns}"
+            robot_namespace="${ns}"
             device_namespace="${device_ns}"
             model="${ouster_models_dict[type]}"
@@ -201,5 +201,5 @@
             xyz="${xyz}"
             rpy="${rpy}"
-            namespace="${ns}"
+            robot_namespace="${ns}"
             device_namespace="${device_ns}"
           />
@@ -240,5 +240,5 @@
             xyz="${xyz}"
             rpy="${rpy}"
-            namespace="${ns}"
+            robot_namespace="${ns}"
             device_namespace="${device_ns}"
             kinova_type="gen3"
@@ -257,5 +257,5 @@
             xyz="${xyz}"
             rpy="${rpy}"
-            namespace="${ns}"
+            robot_namespace="${ns}"
             device_namespace="${device_ns}"
             kinova_type="gen3"
@@ -274,5 +274,5 @@
             xyz="${xyz}"
             rpy="${rpy}"
-            namespace="${ns}"
+            robot_namespace="${ns}"
             device_namespace="${device_ns}"
             kinova_type="gen3"
@@ -291,5 +291,5 @@
             xyz="${xyz}"
             rpy="${rpy}"
-            namespace="${ns}"
+            robot_namespace="${ns}"
             kinova_type="gen3"
             dof="7"
@@ -318,5 +318,5 @@
             xyz="${xyz}"
             rpy="${rpy}"
-            namespace="${ns}"
+            robot_namespace="${ns}"
             device_namespace="${device_ns}"
           />

File: urdf/intel_realsense_d435.urdf.xacro (robot description, xacro)
@@ -19,7 +19,7 @@
                        rpy:='0.0 0.0 0.0'
                        use_nominal_extrinsics:=false
-                       namespace:=''
+                       robot_namespace:=''
                        device_namespace:=camera">
-    <xacro:property name="ns" value="${namespace + '/' if namespace != '' else ''}" />
+    <xacro:property name="ns" value="${robot_namespace + '/' if robot_namespace != '' else ''}" />
     <!-- The following values are approximate, and the camera node
       publishing TF values with actual calibrated camera extrinsic values -->

File: urdf/kinova.urdf.xacro (robot description, xacro)
@@ -46,5 +46,5 @@
                        gripper:=''
                        vision:=false
-                       namespace:=''
+                       robot_namespace:=''
                        device_namespace:=''">
     <xacro:include
@@ -52,5 +52,5 @@
       ns="kinova_manipulator"
     />
-    <xacro:property name="ns" value="${namespace + '/' if namespace != '' else ''}" />
+    <xacro:property name="ns" value="${robot_namespace + '/' if robot_namespace != '' else ''}" />
     <xacro:property name="prefix" value="${device_namespace + '_' if device_namespace != '' else ''}" />
     <!-- robot name parameter -->

File: urdf/luxonis_depthai.urdf.xacro (robot description, xacro)
@@ -17,10 +17,10 @@
                        xyz:='0.0 0.0 0.0'
                        rpy:='0.0 0.0 0.0'
-                       namespace:=''
+                       robot_namespace:=''
                        device_namespace:='oak'
                        model:='OAK-D-PRO'
                        use_sim:=False">
     <xacro:include filename="$(find depthai_descriptions)/urdf/include/depthai_macro.urdf.xacro" />
-    <xacro:property name="ns" value="${namespace + '/' if namespace != '' else ''}" />
+    <xacro:property name="ns" value="${robot_namespace + '/' if robot_namespace != '' else ''}" />
     <xacro:depthai_camera camera_name="${device_namespace}" parent="${parent_link}"
       base_frame="${ns}${device_namespace}" camera_model="${model}"

File: urdf/orbbec_astra.urdf.xacro (robot description, xacro)
@@ -17,7 +17,7 @@
                        xyz:='0.0 0.0 0.0'
                        rpy:='0.0 0.0 0.0'
-                       namespace:=''
+                       robot_namespace:=''
                        device_namespace:=camera">
-    <xacro:property name="ns" value="${namespace + '/' if namespace != '' else ''}" />
+    <xacro:property name="ns" value="${robot_namespace + '/' if robot_namespace != '' else ''}" />
     <joint name="${parent_link.rstrip('_link')}_to_${device_namespace}_joint" type="fixed">
       <origin xyz="${xyz}" rpy="${rpy}" />

File: urdf/ouster.urdf.xacro (robot description, xacro)
@@ -18,5 +18,5 @@
                        rpy:='0.0 0.0 0.0'
                        model:=os1_32
-                       namespace:=''
+                       robot_namespace:=''
                        device_namespace:=''">
     <xacro:if value="${model == 'os0_32'}">
@@ -56,5 +56,5 @@
       <xacro:property name="mesh" value="ouster_os01" scope="parent"/>
     </xacro:if>
-    <xacro:property name="ns" value="${namespace + '/' if namespace != '' else ''}" />
+    <xacro:property name="ns" value="${robot_namespace + '/' if robot_namespace != '' else ''}" />
     <xacro:property name="prefix" value="${device_namespace + '_' if device_namespace != '' else ''}" />
     <xacro:property name="device_ns" value="${device_namespace + '/' if device_namespace != '' else ''}" />

File: urdf/slamtec_rplidar.urdf.xacro (robot description, xacro)
@@ -17,8 +17,8 @@
                        xyz:='0.0 0.0 0.0'
                        rpy:='0.0 0.0 0.0'
-                       namespace:=''
+                       robot_namespace:=''
                        device_namespace:=''
                        model:=s3">
-    <xacro:property name="ns" value="${namespace + '/' if namespace != '' else ''}" />
+    <xacro:property name="ns" value="${robot_namespace + '/' if robot_namespace != '' else ''}" />
     <xacro:property name="prefix" value="${device_namespace + '_' if device_namespace != '' else ''}" />
     <xacro:property name="device_ns" value="${device_namespace + '/' if device_namespace != '' else ''}" />

File: urdf/stereolabs_zed.urdf.xacro (robot description, xacro)
@@ -21,7 +21,7 @@
                        rpy:='0.0 0.0 0.0'
                        model:=zed
-                       namespace:=''
+                       robot_namespace:=''
                        device_namespace:=zed">
-    <xacro:property name="ns" value="${namespace + '/' if namespace != '' else ''}" />
+    <xacro:property name="ns" value="${robot_namespace + '/' if robot_namespace != '' else ''}" />
     <xacro:if value="${model == 'zed'}">
       <xacro:property name="baseline" value="0.12" />

File: urdf/teltonika_003R-00253.urdf.xacro (robot description, xacro)
@@ -17,7 +17,7 @@
                        xyz:='0.0 0.0 0.0'
                        rpy:='0.0 0.0 0.0'
-                       namespace:=''
+                       robot_namespace:=''
                        device_namespace:=gps">
-    <xacro:property name="ns" value="${namespace + '/' if namespace != '' else ''}" />
+    <xacro:property name="ns" value="${robot_namespace + '/' if robot_namespace != '' else ''}" />
     <xacro:property name="prefix" value="${device_namespace + '_' if device_namespace != '' else ''}" />
     <xacro:property name="device_ns" value="${device_namespace + '/' if device_namespace != '' else ''}" />

File: urdf/velodyne_puck.urdf.xacro (robot description, xacro)
@@ -17,7 +17,7 @@
                        xyz:='0.0 0.0 0.0'
                        rpy:='0.0 0.0 0.0'
-                       namespace:=''
+                       robot_namespace:=''
                        device_namespace:=''">
-    <xacro:property name="ns" value="${namespace + '/' if namespace != '' else ''}" />
+    <xacro:property name="ns" value="${robot_namespace + '/' if robot_namespace != '' else ''}" />
     <xacro:property name="prefix" value="${device_namespace + '_' if device_namespace != '' else ''}" />
     <xacro:property name="device_ns" value="${device_namespace + '/' if device_namespace != '' else ''}" />

File: urdf/wibotic_receiver.urdf.xacro (robot description, xacro)
@@ -17,7 +17,7 @@
                        xyz:='0.0 0.0 0.0'
                        rpy:='0.0 0.0 0.0'
-                       namespace:=''
+                       robot_namespace:=''
                        device_namespace:=''">
-    <xacro:property name="ns" value="${namespace + '/' if namespace != '' else ''}" />
+    <xacro:property name="ns" value="${robot_namespace + '/' if robot_namespace != '' else ''}" />
     <xacro:property name="prefix" value="${device_namespace + '_' if device_namespace != '' else ''}" />
     <joint name="${parent_link.rstrip('_link')}_to_${prefix}wibotic_receiver_joint" type="fixed">

Commit message: components.urdf: remove default component names

File: urdf/components.urdf.xacro (robot description, xacro)
@@ -76,7 +76,4 @@
             filename="$(find husarion_components_description)/urdf/orbbec_astra.urdf.xacro"
             ns="camera" />
-          <xacro:if value="${device_ns == ''}">
-            <xacro:property name="device_ns" value="camera" scope="parent" />
-          </xacro:if>
           <xacro:camera.orbbec_astra
             parent_link="${parent_link}"
@@ -91,7 +88,4 @@
             filename="$(find husarion_components_description)/urdf/intel_realsense_d435.urdf.xacro"
             ns="camera" />
-          <xacro:if value="${device_ns == ''}">
-            <xacro:property name="device_ns" value="camera" scope="parent" />
-          </xacro:if>
           <xacro:camera.intel_realsense_d435
             parent_link="${parent_link}"
@@ -114,7 +108,4 @@
             filename="$(find husarion_components_description)/urdf/stereolabs_zed.urdf.xacro"
             ns="camera" />
-          <xacro:if value="${device_ns == ''}">
-            <xacro:property name="device_ns" value="zed" scope="parent" />
-          </xacro:if>
           <xacro:camera.zed_camera
             parent_link="${parent_link}"
@@ -135,7 +126,4 @@
             filename="$(find husarion_components_description)/urdf/luxonis_depthai.urdf.xacro"
             ns="camera" />
-          <xacro:if value="${device_ns == ''}">
-            <xacro:property name="device_ns" value="oak" scope="parent" />
-          </xacro:if>
           <xacro:camera.luxonis_depthai
             parent_link="${parent_link}"
