Commit message: device_namespace -> component_name

File: urdf/components.urdf.xacro (robot description, xacro)
@@ -59,5 +59,5 @@
         <xacro:property name="xyz" value="${component['xyz'] if 'xyz' in component else '0.0 0.0 0.0'}" scope="parent" />
         <xacro:property name="rpy" value="${component['rpy'] if 'rpy' in component else '0.0 0.0 0.0'}" scope="parent" />
-        <xacro:property name="device_ns" value="${component['device_namespace'] if 'device_namespace' in component else ''}" scope="parent" />
+        <xacro:property name="component_name" value="${component['name'] if 'name' in component else ''}" scope="parent" />
         <xacro:if value="${type == 'ANT02'}">
           <xacro:include
@@ -69,5 +69,5 @@
             rpy="${rpy}"
             robot_namespace="${ns}"
-            device_namespace="${device_ns}"
+            component_name="${component_name}"
           />
         </xacro:if>
@@ -81,5 +81,5 @@
             rpy="${rpy}"
             robot_namespace="${ns}"
-            device_namespace="${device_ns}"
+            component_name="${component_name}"
           />
         </xacro:if>
@@ -93,5 +93,5 @@
             rpy="${rpy}"
             robot_namespace="${ns}"
-            device_namespace="${device_ns}"
+            component_name="${component_name}"
             use_nominal_extrinsics="${use_sim}"
           />
@@ -113,5 +113,5 @@
             rpy="${rpy}"
             robot_namespace="${ns}"
-            device_namespace="${device_ns}"
+            component_name="${component_name}"
             model="${zed_models_dict[type]}"
           />
@@ -131,5 +131,5 @@
             rpy="${rpy}"
             robot_namespace="${ns}"
-            device_namespace="${device_ns}"
+            component_name="${component_name}"
             model="${luxonis_models_dict[type]}"
           />
@@ -153,5 +153,5 @@
             rpy="${rpy}"
             robot_namespace="${ns}"
-            device_namespace="${device_ns}"
+            component_name="${component_name}"
             model="${rplidar_models_dict[type]}"
           />
@@ -176,5 +176,5 @@
             rpy="${rpy}"
             robot_namespace="${ns}"
-            device_namespace="${device_ns}"
+            component_name="${component_name}"
             model="${ouster_models_dict[type]}"
           />
@@ -190,5 +190,5 @@
             rpy="${rpy}"
             robot_namespace="${ns}"
-            device_namespace="${device_ns}"
+            component_name="${component_name}"
           />
         </xacro:if>
@@ -202,5 +202,5 @@
             xyz="${xyz}"
             rpy="${rpy}"
-            device_namespace="${device_ns}"
+            component_name="${component_name}"
             ur_type="ur3e"
           />
@@ -215,5 +215,5 @@
             xyz="${xyz}"
             rpy="${rpy}"
-            device_namespace="${device_ns}"
+            component_name="${component_name}"
             ur_type="ur5e"
           />
@@ -229,5 +229,5 @@
             rpy="${rpy}"
             robot_namespace="${ns}"
-            device_namespace="${device_ns}"
+            component_name="${component_name}"
             kinova_type="gen3"
             dof="6"
@@ -246,5 +246,5 @@
             rpy="${rpy}"
             robot_namespace="${ns}"
-            device_namespace="${device_ns}"
+            component_name="${component_name}"
             kinova_type="gen3"
             dof="6"
@@ -263,5 +263,5 @@
             rpy="${rpy}"
             robot_namespace="${ns}"
-            device_namespace="${device_ns}"
+            component_name="${component_name}"
             kinova_type="gen3"
             dof="7"
@@ -284,5 +284,5 @@
             gripper="robotiq_2f_85"
             vision="true"
-            device_namespace="${device_ns}"
+            component_name="${component_name}"
           />
         </xacro:if>
@@ -294,5 +294,5 @@
             xyz="${xyz}"
             rpy="${rpy}"
-            device_namespace="${device_ns}"
+            component_name="${component_name}"
             robotiq_type="2f_85"
           />
@@ -307,5 +307,5 @@
             rpy="${rpy}"
             robot_namespace="${ns}"
-            device_namespace="${device_ns}"
+            component_name="${component_name}"
           />
         </xacro:if>

File: urdf/intel_realsense_d435.urdf.xacro (robot description, xacro)
@@ -20,5 +20,5 @@
                        use_nominal_extrinsics:=false
                        robot_namespace:=''
-                       device_namespace:=camera">
+                       component_name:=camera">
     <xacro:property name="ns" value="${robot_namespace + '/' if robot_namespace != '' else ''}" />
     <!-- The following values are approximate, and the camera node
@@ -41,17 +41,17 @@
     <xacro:property name="d435_cam_depth_pz" value="${d435_cam_height/2}" />
     <!-- camera body, with origin at bottom screw mount -->
-    <joint name="${parent_link.rstrip('_link')}_to_${device_namespace}_bottom_screw_joint" type="fixed">
+    <joint name="${parent_link.rstrip('_link')}_to_${component_name}_bottom_screw_joint" type="fixed">
       <origin xyz="${xyz}" rpy="${rpy}" />
       <parent link="${parent_link}" />
-      <child link="${device_namespace}_bottom_screw_frame" />
+      <child link="${component_name}_bottom_screw_frame" />
     </joint>
-    <link name="${device_namespace}_bottom_screw_frame" />
-    <joint name="${device_namespace}_bottom_screw_to_${device_namespace}_joint" type="fixed">
+    <link name="${component_name}_bottom_screw_frame" />
+    <joint name="${component_name}_bottom_screw_to_${component_name}_joint" type="fixed">
       <origin xyz="0.0 ${d435_cam_depth_py} ${d435_cam_depth_pz}"
         rpy="0.0 0.0 0.0" />
-      <parent link="${device_namespace}_bottom_screw_frame" />
-      <child link="${device_namespace}_link" />
+      <parent link="${component_name}_bottom_screw_frame" />
+      <child link="${component_name}_link" />
     </joint>
-    <link name="${device_namespace}_link">
+    <link name="${component_name}_link">
       <visual>
         <origin xyz="${d435_cam_mount_from_center_offset} ${-d435_cam_depth_py} 0.0" rpy="${pi/2.0} 0.0 ${pi/2.0}" />
@@ -79,55 +79,55 @@
     <xacro:if value="${use_nominal_extrinsics}">
       <!-- camera depth joints and links -->
-      <joint name="${device_namespace}_to_${device_namespace}_depth_joint" type="fixed">
+      <joint name="${component_name}_to_${component_name}_depth_joint" type="fixed">
         <origin xyz="0.0 0.0 0.0" rpy="0.0 0.0 0.0" />
-        <parent link="${device_namespace}_link" />
-        <child link="${device_namespace}_depth_frame" />
+        <parent link="${component_name}_link" />
+        <child link="${component_name}_depth_frame" />
       </joint>
-      <link name="${device_namespace}_depth_frame" />
-      <joint name="${device_namespace}_depth_to_${device_namespace}_depth_optical_joint" type="fixed">
+      <link name="${component_name}_depth_frame" />
+      <joint name="${component_name}_depth_to_${component_name}_depth_optical_joint" type="fixed">
         <origin xyz="0.0 0.0 0.0" rpy="${-pi/2.0} 0.0 ${-pi/2.0}" />
-        <parent link="${device_namespace}_depth_frame" />
-        <child link="${device_namespace}_depth_optical_frame" />
+        <parent link="${component_name}_depth_frame" />
+        <child link="${component_name}_depth_optical_frame" />
       </joint>
-      <link name="${device_namespace}_depth_optical_frame" />
+      <link name="${component_name}_depth_optical_frame" />
       <!-- camera left IR joints and links -->
-      <joint name="${device_namespace}_to_${device_namespace}_infra1_joint" type="fixed">
+      <joint name="${component_name}_to_${component_name}_infra1_joint" type="fixed">
         <origin xyz="0.0 ${d435_cam_depth_to_infra1_offset} 0.0" rpy="0.0 0.0 0.0" />
-        <parent link="${device_namespace}_link" />
-        <child link="${device_namespace}_infra1_frame" />
+        <parent link="${component_name}_link" />
+        <child link="${component_name}_infra1_frame" />
       </joint>
-      <link name="${device_namespace}_infra1_frame" />
-      <joint name="${device_namespace}_infra1_to_${device_namespace}_infra1_optical_joint" type="fixed">
+      <link name="${component_name}_infra1_frame" />
+      <joint name="${component_name}_infra1_to_${component_name}_infra1_optical_joint" type="fixed">
         <origin xyz="0.0 0.0 0.0" rpy="${-pi/2.0} 0.0 ${-pi/2.0}" />
-        <parent link="${device_namespace}_infra1_frame" />
-        <child link="${device_namespace}_infra1_optical_frame" />
+        <parent link="${component_name}_infra1_frame" />
+        <child link="${component_name}_infra1_optical_frame" />
       </joint>
-      <link name="${device_namespace}_infra1_optical_frame" />
+      <link name="${component_name}_infra1_optical_frame" />
       <!-- camera right IR joints and links -->
-      <joint name="${device_namespace}_to_${device_namespace}_infra2_joint" type="fixed">
+      <joint name="${component_name}_to_${component_name}_infra2_joint" type="fixed">
         <origin xyz="0.0 ${d435_cam_depth_to_infra2_offset} 0.0" rpy="0.0 0.0 0.0" />
-        <parent link="${device_namespace}_link" />
-        <child link="${device_namespace}_infra2_frame" />
+        <parent link="${component_name}_link" />
+        <child link="${component_name}_infra2_frame" />
       </joint>
-      <link name="${device_namespace}_infra2_frame" />
-      <joint name="${device_namespace}_infra2_to_${device_namespace}_infra2_optical_joint" type="fixed">
+      <link name="${component_name}_infra2_frame" />
+      <joint name="${component_name}_infra2_to_${component_name}_infra2_optical_joint" type="fixed">
         <origin xyz="0.0 0.0 0.0" rpy="${-pi/2.0} 0.0 ${-pi/2.0}" />
-        <parent link="${device_namespace}_infra2_frame" />
-        <child link="${device_namespace}_infra2_optical_frame" />
+        <parent link="${component_name}_infra2_frame" />
+        <child link="${component_name}_infra2_optical_frame" />
       </joint>
-      <link name="${device_namespace}_infra2_optical_frame" />
+      <link name="${component_name}_infra2_optical_frame" />
       <!-- camera color joints and links -->
-      <joint name="${device_namespace}_to_${device_namespace}_color_joint" type="fixed">
+      <joint name="${component_name}_to_${component_name}_color_joint" type="fixed">
         <origin xyz="0.0 ${d435_cam_depth_to_color_offset} 0.0" rpy="0.0 0.0 0.0" />
-        <parent link="${device_namespace}_link" />
-        <child link="${device_namespace}_color_frame" />
+        <parent link="${component_name}_link" />
+        <child link="${component_name}_color_frame" />
       </joint>
-      <link name="${device_namespace}_color_frame" />
-      <joint name="${device_namespace}_color_to_${device_namespace}_color_optical_joint" type="fixed">
+      <link name="${component_name}_color_frame" />
+      <joint name="${component_name}_color_to_${component_name}_color_optical_joint" type="fixed">
         <origin xyz="0.0 0.0 0.0" rpy="${-pi/2.0} 0.0 ${-pi/2.0}" />
-        <parent link="${device_namespace}_color_frame" />
-        <child link="${device_namespace}_color_optical_frame" />
+        <parent link="${component_name}_color_frame" />
+        <child link="${component_name}_color_optical_frame" />
       </joint>
-      <link name="${device_namespace}_color_optical_frame" />
+      <link name="${component_name}_color_optical_frame" />
     </xacro:if>
     <xacro:include filename="$(find husarion_components_description)/urdf/gz_sensor.urdf.xacro" ns="gz_sensor" />
@@ -136,8 +136,8 @@
     <!-- https://github.com/IntelRealSense/realsense-ros#published-topics -->
     <xacro:gz_sensor.camera
-      reference="${device_namespace}_link"
-      name="${ns}${device_namespace}_intel_realsense_d435_color"
-      topic="${ns}${device_namespace}/color/image_raw"
-      frame_id="${ns}${device_namespace}_color_optical_frame"
+      reference="${component_name}_link"
+      name="${ns}${component_name}_intel_realsense_d435_color"
+      topic="${ns}${component_name}/color/image_raw"
+      frame_id="${ns}${component_name}_color_optical_frame"
       frequency="30"
       width="1280"
@@ -145,8 +145,8 @@
       fov="${69.0/180.0*pi}" />
     <xacro:gz_sensor.depth_camera
-      reference="${device_namespace}_link"
-      name="${ns}${device_namespace}_intel_realsense_d435_depth"
-      topic="${ns}${device_namespace}/depth/image_rect_raw"
-      frame_id="${ns}${device_namespace}_depth_optical_frame"
+      reference="${component_name}_link"
+      name="${ns}${component_name}_intel_realsense_d435_depth"
+      topic="${ns}${component_name}/depth/image_rect_raw"
+      frame_id="${ns}${component_name}_depth_optical_frame"
       frequency="30"
       width="1280"

File: urdf/kinova.urdf.xacro (robot description, xacro)
@@ -47,5 +47,5 @@
                        vision:=false
                        robot_namespace:=''
-                       device_namespace:=''">
+                       component_name:=''">
     <xacro:include
       filename="$(find kortex_description)/robots/kortex_robot.xacro"
@@ -53,5 +53,5 @@
     />
     <xacro:property name="ns" value="${robot_namespace + '/' if robot_namespace != '' else ''}" />
-    <xacro:property name="prefix" value="${device_namespace + '_' if device_namespace != '' else ''}" />
+    <xacro:property name="prefix" value="${component_name + '_' if component_name != '' else ''}" />
     <!-- robot name parameter -->
     <xacro:property name="robot_name" value="kinova_arm" />
@@ -126,6 +126,6 @@
     </xacro:unless>
     <xacro:if value="${vision}">
-      <gazebo reference="${device_namespace}_camera_color_frame">
-        <sensor name="${ns}${device_namespace}_camera_sensor" type="rgbd_camera">
+      <gazebo reference="${component_name}_camera_color_frame">
+        <sensor name="${ns}${component_name}_camera_sensor" type="rgbd_camera">
           <camera>
             <horizontal_fov>1.047</horizontal_fov>
@@ -177,11 +177,11 @@
               </clip>
             </depth_camera>
-            <optical_frame_id>${device_namespace}_color_optical_frame</optical_frame_id>
+            <optical_frame_id>${component_name}_color_optical_frame</optical_frame_id>
           </camera>
-          <gz_frame_id>${device_namespace}_camera_color_frame</gz_frame_id>
+          <gz_frame_id>${component_name}_camera_color_frame</gz_frame_id>
           <always_on>1</always_on>
           <update_rate>${camera_fps}</update_rate>
           <visualize>true</visualize>
-          <topic>${ns}${device_namespace}/wrist_mounted_camera</topic>
+          <topic>${ns}${component_name}/wrist_mounted_camera</topic>
           <enable_metrics>false</enable_metrics>
         </sensor>

File: urdf/luxonis_depthai.urdf.xacro (robot description, xacro)
@@ -18,11 +18,11 @@
                        rpy:='0.0 0.0 0.0'
                        robot_namespace:=''
-                       device_namespace:='oak'
+                       component_name:='oak'
                        model:='OAK-D-PRO'
                        use_sim:=False">
     <xacro:include filename="$(find depthai_descriptions)/urdf/include/depthai_macro.urdf.xacro" />
     <xacro:property name="ns" value="${robot_namespace + '/' if robot_namespace != '' else ''}" />
-    <xacro:depthai_camera camera_name="${device_namespace}" parent="${parent_link}"
-      base_frame="${ns}${device_namespace}" camera_model="${model}"
+    <xacro:depthai_camera camera_name="${component_name}" parent="${parent_link}"
+      base_frame="${ns}${component_name}" camera_model="${model}"
       cam_pos_x="${xyz.split()[0]}" cam_pos_y="${xyz.split()[1]}" cam_pos_z="${xyz.split()[2]}"
       cam_roll="${rpy.split()[0]}" cam_pitch="${rpy.split()[1]}" cam_yaw="${rpy.split()[2]}"
@@ -31,8 +31,8 @@
       ns="gz_sensor" />
     <xacro:gz_sensor.camera
-      reference="${ns}${device_namespace}"
-      name="${ns}${device_namespace}_color"
-      topic="${ns}${device_namespace}/rgb/color"
-      frame_id="${ns}${device_namespace}_rgb_camera_frame"
+      reference="${ns}${component_name}"
+      name="${ns}${component_name}_color"
+      topic="${ns}${component_name}/rgb/color"
+      frame_id="${ns}${component_name}_rgb_camera_frame"
       frequency="30"
       width="1280"
@@ -40,8 +40,8 @@
       fov="${60.0/180.0*pi}" />
     <xacro:gz_sensor.depth_camera
-      reference="${ns}${device_namespace}"
-      name="${ns}${device_namespace}_depth"
-      topic="${ns}${device_namespace}/stereo/depth"
-      frame_id="${ns}${device_namespace}_rgb_camera_frame"
+      reference="${ns}${component_name}"
+      name="${ns}${component_name}_depth"
+      topic="${ns}${component_name}/stereo/depth"
+      frame_id="${ns}${component_name}_rgb_camera_frame"
       frequency="30"
       width="1280"

File: urdf/orbbec_astra.urdf.xacro (robot description, xacro)
@@ -18,18 +18,18 @@
                        rpy:='0.0 0.0 0.0'
                        robot_namespace:=''
-                       device_namespace:=camera">
+                       component_name:=camera">
     <xacro:property name="ns" value="${robot_namespace + '/' if robot_namespace != '' else ''}" />
-    <joint name="${parent_link.rstrip('_link')}_to_${device_namespace}_joint" type="fixed">
+    <joint name="${parent_link.rstrip('_link')}_to_${component_name}_joint" type="fixed">
       <origin xyz="${xyz}" rpy="${rpy}" />
       <parent link="${parent_link}" />
-      <child link="${device_namespace}_link" />
+      <child link="${component_name}_link" />
     </joint>
-    <link name="${device_namespace}_link" />
-    <joint name="${parent_link.rstrip('_link')}_to_${device_namespace}_orbbec_astra_joint" type="fixed">
+    <link name="${component_name}_link" />
+    <joint name="${parent_link.rstrip('_link')}_to_${component_name}_orbbec_astra_joint" type="fixed">
       <origin xyz="${xyz}" rpy="${rpy}" />
       <parent link="${parent_link}" />
-      <child link="${device_namespace}_orbbec_astra_link" />
+      <child link="${component_name}_orbbec_astra_link" />
     </joint>
-    <link name="${device_namespace}_orbbec_astra_link">
+    <link name="${component_name}_orbbec_astra_link">
       <!-- <visual>
         <origin xyz="0.0 0.0 0.0" rpy="0.0 0.0 0.0" />
@@ -79,36 +79,36 @@
       </inertial>
     </link>
-    <joint name="${parent_link.rstrip('_link')}_to_${device_namespace}_color_joint" type="fixed">
+    <joint name="${parent_link.rstrip('_link')}_to_${component_name}_color_joint" type="fixed">
       <origin xyz="-0.002 0.0125 0.03325" rpy="-0.003 0.0 -0.003" />
-      <parent link="${device_namespace}_link" />
-      <child link="${device_namespace}_color_frame" />
+      <parent link="${component_name}_link" />
+      <child link="${component_name}_color_frame" />
     </joint>
-    <link name="${device_namespace}_depth_frame" />
-    <joint name="${parent_link.rstrip('_link')}_to_${device_namespace}_depth_joint" type="fixed">
+    <link name="${component_name}_depth_frame" />
+    <joint name="${parent_link.rstrip('_link')}_to_${component_name}_depth_joint" type="fixed">
       <origin xyz="0.0 0.0 0.03325" rpy="0.0 0.0 0.0" />
-      <parent link="${device_namespace}_link" />
-      <child link="${device_namespace}_depth_frame" />
+      <parent link="${component_name}_link" />
+      <child link="${component_name}_depth_frame" />
     </joint>
-    <link name="${device_namespace}_color_frame" />
-    <joint name="${device_namespace}_color_to_${device_namespace}_color_optical_joint" type="fixed">
+    <link name="${component_name}_color_frame" />
+    <joint name="${component_name}_color_to_${component_name}_color_optical_joint" type="fixed">
       <origin xyz="0.0 0.0 0.0" rpy="${-pi/2} 0.0 ${-pi/2}" />
-      <parent link="${device_namespace}_color_frame" />
-      <child link="${device_namespace}_color_optical_frame" />
+      <parent link="${component_name}_color_frame" />
+      <child link="${component_name}_color_optical_frame" />
     </joint>
-    <link name="${device_namespace}_depth_optical_frame" />
-    <joint name="${device_namespace}_depth_to_${device_namespace}_depth_optical_joint" type="fixed">
+    <link name="${component_name}_depth_optical_frame" />
+    <joint name="${component_name}_depth_to_${component_name}_depth_optical_joint" type="fixed">
       <origin xyz="0.0 0.0 0.0" rpy="${-pi/2} 0.0 ${-pi/2}" />
-      <parent link="${device_namespace}_depth_frame" />
-      <child link="${device_namespace}_depth_optical_frame" />
+      <parent link="${component_name}_depth_frame" />
+      <child link="${component_name}_depth_optical_frame" />
     </joint>
-    <link name="${device_namespace}_color_optical_frame" />
+    <link name="${component_name}_color_optical_frame" />
     <!-- GAZEBO -->
     <!-- https://github.com/orbbec/OrbbecSDK_ROS2#all-available-topics -->
     <xacro:include filename="$(find husarion_components_description)/urdf/gz_sensor.urdf.xacro" ns="gz_sensor" />
     <xacro:gz_sensor.camera
-      reference="${device_namespace}_link"
-      name="${ns}${device_namespace}_orbbec_astra_color"
-      topic="${ns}${device_namespace}/color/image_raw"
-      frame_id="${ns}${device_namespace}_color_optical_frame"
+      reference="${component_name}_link"
+      name="${ns}${component_name}_orbbec_astra_color"
+      topic="${ns}${component_name}/color/image_raw"
+      frame_id="${ns}${component_name}_color_optical_frame"
       frequency="30"
       width="640"
@@ -116,8 +116,8 @@
       fov="${60.0/180.0*pi}" />
     <xacro:gz_sensor.depth_camera
-      reference="${device_namespace}_link"
-      name="${ns}${device_namespace}_orbbec_astra_depth"
-      topic="${ns}${device_namespace}/depth/image_raw"
-      frame_id="${ns}${device_namespace}_depth_optical_frame"
+      reference="${component_name}_link"
+      name="${ns}${component_name}_orbbec_astra_depth"
+      topic="${ns}${component_name}/depth/image_raw"
+      frame_id="${ns}${component_name}_depth_optical_frame"
       frequency="30"
       width="640"

File: urdf/ouster.urdf.xacro (robot description, xacro)
@@ -19,5 +19,5 @@
                        model:=os1_32
                        robot_namespace:=''
-                       device_namespace:=''">
+                       component_name:=''">
     <xacro:if value="${model == 'os0_32'}">
       <xacro:property name="vfov" value="${radians(90.0)}" scope="parent" />
@@ -57,6 +57,6 @@
     </xacro:if>
     <xacro:property name="ns" value="${robot_namespace + '/' if robot_namespace != '' else ''}" />
-    <xacro:property name="prefix" value="${device_namespace + '_' if device_namespace != '' else ''}" />
-    <xacro:property name="device_ns" value="${device_namespace + '/' if device_namespace != '' else ''}" />
+    <xacro:property name="prefix" value="${component_name + '_' if component_name != '' else ''}" />
+    <xacro:property name="device_ns" value="${component_name + '/' if component_name != '' else ''}" />
     <joint name="${parent_link.rstrip('_link')}_to_${prefix}ouster_${model}_joint" type="fixed">
       <origin xyz="${xyz}" rpy="${rpy}" />
