Commit message: device_namespace -> component_name

File: urdf/robotiq.urdf.xacro (robot description, xacro)
@@ -18,10 +18,10 @@
                        rpy:='0.0 0.0 0.0'
                        robotiq_type:=2f_85
-                       device_namespace:=''">
+                       component_name:=''">
     <xacro:include
       filename="$(find robotiq_description)/urdf/robotiq_${robotiq_type}_macro.urdf.xacro"
       ns="gripper" />
-    <xacro:property name="prefix" value="${device_namespace + '_' if device_namespace != '' else ''}" />
-    <xacro:gripper.robotiq_gripper name="${device_namespace}robotiq_${robotiq_type}"
+    <xacro:property name="prefix" value="${component_name + '_' if component_name != '' else ''}" />
+    <xacro:gripper.robotiq_gripper name="${component_name}robotiq_${robotiq_type}"
       prefix="${prefix}"
       parent="${parent_link}"

File: urdf/slamtec_rplidar.urdf.xacro (robot description, xacro)
@@ -18,9 +18,9 @@
                        rpy:='0.0 0.0 0.0'
                        robot_namespace:=''
-                       device_namespace:=''
+                       component_name:=''
                        model:=s3">
     <xacro:property name="ns" value="${robot_namespace + '/' if robot_namespace != '' else ''}" />
-    <xacro:property name="prefix" value="${device_namespace + '_' if device_namespace != '' else ''}" />
-    <xacro:property name="device_ns" value="${device_namespace + '/' if device_namespace != '' else ''}" />
+    <xacro:property name="prefix" value="${component_name + '_' if component_name != '' else ''}" />
+    <xacro:property name="device_ns" value="${component_name + '/' if component_name != '' else ''}" />
     <xacro:if value="${model == 's3'}">
       <!-- Spec: https://www.slamtec.ai/wp-content/uploads/2023/11/SLAMTEC_rplidar_datasheet_S3_v1.0_en.pdf -->

File: urdf/stereolabs_zed.urdf.xacro (robot description, xacro)
@@ -22,5 +22,5 @@
                        model:=zed
                        robot_namespace:=''
-                       device_namespace:=zed">
+                       component_name:=zed">
     <xacro:property name="ns" value="${robot_namespace + '/' if robot_namespace != '' else ''}" />
     <xacro:if value="${model == 'zed'}">
@@ -160,12 +160,12 @@
     </xacro:if>
     <!-- Camera mounting point (the threaded screw hole in the bottom) -->
-    <link name="${device_namespace}_camera_link" />
-    <joint name="${device_namespace}_base_joint" type="fixed">
+    <link name="${component_name}_camera_link" />
+    <joint name="${component_name}_base_joint" type="fixed">
       <parent link="${parent_link}" />
-      <child link="${device_namespace}_camera_link" />
+      <child link="${component_name}_camera_link" />
       <origin xyz="${xyz}" rpy="${rpy}" />
     </joint>
     <!-- Camera Center -->
-    <link name="${device_namespace}_camera_center">
+    <link name="${component_name}_camera_center">
       <xacro:unless value="${model == 'virtual'}">
         <visual>
@@ -188,12 +188,12 @@
       </xacro:unless>
     </link>
-    <joint name="${device_namespace}_camera_center_joint" type="fixed">
-      <parent link="${device_namespace}_camera_link"/>
-      <child link="${device_namespace}_camera_center"/>
+    <joint name="${component_name}_camera_center_joint" type="fixed">
+      <parent link="${component_name}_camera_link"/>
+      <child link="${component_name}_camera_center"/>
       <origin xyz="0 0 ${height/2}" rpy="0 ${bottom_slope} 0" />
     </joint>
     <xacro:unless value="${mono}">
       <!-- Left Camera -->
-      <link name="${device_namespace}_left_camera_frame">
+      <link name="${component_name}_left_camera_frame">
         <xacro:if value="${model == 'virtual'}">
           <visual>
@@ -214,17 +214,17 @@
         </xacro:if>
       </link>
-      <joint name="${device_namespace}_left_camera_joint" type="fixed">
-        <parent link="${device_namespace}_camera_center"/>
-        <child link="${device_namespace}_left_camera_frame"/>
+      <joint name="${component_name}_left_camera_joint" type="fixed">
+        <parent link="${component_name}_camera_center"/>
+        <child link="${component_name}_left_camera_frame"/>
         <origin xyz="${optical_offset_x} ${baseline/2} 0" rpy="0 0 0" />
       </joint>
-      <link name="${device_namespace}_left_camera_optical_frame"/>
-      <joint name="${device_namespace}_left_camera_optical_joint" type="fixed">
+      <link name="${component_name}_left_camera_optical_frame"/>
+      <joint name="${component_name}_left_camera_optical_joint" type="fixed">
         <origin xyz="0 0 0" rpy="-${M_PI/2} 0.0 -${M_PI/2}"/>
-        <parent link="${device_namespace}_left_camera_frame"/>
-        <child link="${device_namespace}_left_camera_optical_frame"/>
+        <parent link="${component_name}_left_camera_frame"/>
+        <child link="${component_name}_left_camera_optical_frame"/>
       </joint>
       <!-- Right Camera -->
-      <link name="${device_namespace}_right_camera_frame">
+      <link name="${component_name}_right_camera_frame">
         <xacro:if value="${model == 'virtual'}">
           <visual>
@@ -245,39 +245,39 @@
         </xacro:if>
       </link>
-      <joint name="${device_namespace}_right_camera_joint" type="fixed">
-        <parent link="${device_namespace}_camera_center"/>
-        <child link="${device_namespace}_right_camera_frame"/>
+      <joint name="${component_name}_right_camera_joint" type="fixed">
+        <parent link="${component_name}_camera_center"/>
+        <child link="${component_name}_right_camera_frame"/>
         <origin xyz="${optical_offset_x} -${baseline/2} 0" rpy="0 0 0" />
       </joint>
-      <link name="${device_namespace}_right_camera_optical_frame"/>
-      <joint name="${device_namespace}_right_camera_optical_joint" type="fixed">
+      <link name="${component_name}_right_camera_optical_frame"/>
+      <joint name="${component_name}_right_camera_optical_joint" type="fixed">
         <origin xyz="0 0 0" rpy="-${M_PI/2} 0.0 -${M_PI/2}"/>
-        <parent link="${device_namespace}_right_camera_frame"/>
-        <child link="${device_namespace}_right_camera_optical_frame"/>
+        <parent link="${component_name}_right_camera_frame"/>
+        <child link="${component_name}_right_camera_optical_frame"/>
       </joint>
       <!-- ZED2 Sensors -->
       <xacro:if value="${model == 'zed2'}">
-        <link name="${device_namespace}_mag_link" />
-        <joint name="${device_namespace}_mag_joint" type="fixed">
-          <parent link="${device_namespace}_camera_center"/>
-          <child link="${device_namespace}_mag_link"/>
+        <link name="${component_name}_mag_link" />
+        <joint name="${component_name}_mag_joint" type="fixed">
+          <parent link="${component_name}_camera_center"/>
+          <child link="${component_name}_mag_link"/>
           <origin xyz="0 0 0" rpy="0 0 0" />
         </joint>
-        <link name="${device_namespace}_baro_link" />
-        <joint name="${device_namespace}_baro_joint" type="fixed">
-          <parent link="${device_namespace}_camera_center"/>
-          <child link="${device_namespace}_baro_link"/>
+        <link name="${component_name}_baro_link" />
+        <joint name="${component_name}_baro_joint" type="fixed">
+          <parent link="${component_name}_camera_center"/>
+          <child link="${component_name}_baro_link"/>
           <origin xyz="0 0 0" rpy="0 0 0" />
         </joint>
-        <link name="${device_namespace}_temp_left_link" />
-        <joint name="${device_namespace}_temp_left_joint" type="fixed">
-          <parent link="${device_namespace}_left_camera_frame"/>
-          <child link="${device_namespace}_temp_left_link"/>
+        <link name="${component_name}_temp_left_link" />
+        <joint name="${component_name}_temp_left_joint" type="fixed">
+          <parent link="${component_name}_left_camera_frame"/>
+          <child link="${component_name}_temp_left_link"/>
           <origin xyz="0 0 0" rpy="0 0 0" />
         </joint>
-        <link name="${device_namespace}_temp_right_link" />
-        <joint name="${device_namespace}_temp_right_joint" type="fixed">
-          <parent link="${device_namespace}_right_camera_frame"/>
-          <child link="${device_namespace}_temp_right_link"/>
+        <link name="${component_name}_temp_right_link" />
+        <joint name="${component_name}_temp_right_joint" type="fixed">
+          <parent link="${component_name}_right_camera_frame"/>
+          <child link="${component_name}_temp_right_link"/>
           <origin xyz="0 0 0" rpy="0 0 0" />
         </joint>
@@ -286,15 +286,15 @@
     <xacro:if value="${mono}">
       <!-- Camera -->
-      <link name="${device_namespace}_camera_frame" />
-      <joint name="${device_namespace}_camera_joint" type="fixed">
-        <parent link="${device_namespace}_camera_center"/>
-        <child link="${device_namespace}_camera_frame"/>
+      <link name="${component_name}_camera_frame" />
+      <joint name="${component_name}_camera_joint" type="fixed">
+        <parent link="${component_name}_camera_center"/>
+        <child link="${component_name}_camera_frame"/>
         <origin xyz="${optical_offset_x} 0 0" rpy="0 0 0" />
       </joint>
-      <link name="${device_namespace}_camera_optical_frame"/>
-      <joint name="${device_namespace}_camera_optical_joint" type="fixed">
+      <link name="${component_name}_camera_optical_frame"/>
+      <joint name="${component_name}_camera_optical_joint" type="fixed">
         <origin xyz="0 0 0" rpy="-${M_PI/2} 0.0 -${M_PI/2}"/>
-        <parent link="${device_namespace}_camera_frame"/>
-        <child link="${device_namespace}_camera_optical_frame"/>
+        <parent link="${component_name}_camera_frame"/>
+        <child link="${component_name}_camera_optical_frame"/>
       </joint>
     </xacro:if>
@@ -302,8 +302,8 @@
     <xacro:include filename="$(find husarion_components_description)/urdf/gz_sensor.urdf.xacro" ns="gz_sensor" />
     <xacro:gz_sensor.camera
-      reference="${device_namespace}_camera_center"
-      name="${ns}${device_namespace}_stereolabs_zed_color"
-      topic="${ns}${device_namespace}/zed_node/rgb/image_rect_color"
-      frame_id="${ns}${device_namespace}_camera_center"
+      reference="${component_name}_camera_center"
+      name="${ns}${component_name}_stereolabs_zed_color"
+      topic="${ns}${component_name}/zed_node/rgb/image_rect_color"
+      frame_id="${ns}${component_name}_camera_center"
       frequency="30"
       width="1280"
@@ -311,8 +311,8 @@
       fov="${110.0/180.0*pi}" />
     <xacro:gz_sensor.depth_camera
-      reference="${device_namespace}_camera_center"
-      name="${ns}${device_namespace}_stereolabs_zed_depth"
-      topic="${ns}${device_namespace}/zed_node/depth"
-      frame_id="${ns}${device_namespace}_camera_center"
+      reference="${component_name}_camera_center"
+      name="${ns}${component_name}_stereolabs_zed_depth"
+      topic="${ns}${component_name}/zed_node/depth"
+      frame_id="${ns}${component_name}_camera_center"
       frequency="30"
       width="1280"

File: urdf/teltonika_003R-00253.urdf.xacro (robot description, xacro)
@@ -18,8 +18,8 @@
                        rpy:='0.0 0.0 0.0'
                        robot_namespace:=''
-                       device_namespace:=gps">
+                       component_name:=gps">
     <xacro:property name="ns" value="${robot_namespace + '/' if robot_namespace != '' else ''}" />
-    <xacro:property name="prefix" value="${device_namespace + '_' if device_namespace != '' else ''}" />
-    <xacro:property name="device_ns" value="${device_namespace + '/' if device_namespace != '' else ''}" />
+    <xacro:property name="prefix" value="${component_name + '_' if component_name != '' else ''}" />
+    <xacro:property name="device_ns" value="${component_name + '/' if component_name != '' else ''}" />
     <joint name="${parent_link.rstrip('_link')}_to_${prefix}teltonika_mounting_joint"
       type="fixed">

File: urdf/ur.urdf.xacro (robot description, xacro)
@@ -42,8 +42,8 @@
                        xyz:='0.0 0.0 0.0'
                        rpy:='0.0 0.0 0.0'
-                       device_namespace:=''
+                       component_name:=''
                        ur_type:=ur3e">
     <xacro:include filename="$(find ur_description)/urdf/ur_macro.xacro" ns="ur_manipulator" />
-    <xacro:property name="prefix" value="${device_namespace + '_' if device_namespace != '' else ''}" />
+    <xacro:property name="prefix" value="${component_name + '_' if component_name != '' else ''}" />
     <xacro:property name="joint_limit_params"
       value="$(find ur_description)/config/${ur_type}/joint_limits.yaml" scope="parent" />

File: urdf/velodyne_puck.urdf.xacro (robot description, xacro)
@@ -18,8 +18,8 @@
                        rpy:='0.0 0.0 0.0'
                        robot_namespace:=''
-                       device_namespace:=''">
+                       component_name:=''">
     <xacro:property name="ns" value="${robot_namespace + '/' if robot_namespace != '' else ''}" />
-    <xacro:property name="prefix" value="${device_namespace + '_' if device_namespace != '' else ''}" />
-    <xacro:property name="device_ns" value="${device_namespace + '/' if device_namespace != '' else ''}" />
+    <xacro:property name="prefix" value="${component_name + '_' if component_name != '' else ''}" />
+    <xacro:property name="device_ns" value="${component_name + '/' if component_name != '' else ''}" />
     <joint name="${parent_link.rstrip('_link')}_to_${prefix}velodyne_puck_joint" type="fixed">
       <origin xyz="${xyz}" rpy="${rpy}" />

File: urdf/wibotic_receiver.urdf.xacro (robot description, xacro)
@@ -18,7 +18,7 @@
                        rpy:='0.0 0.0 0.0'
                        robot_namespace:=''
-                       device_namespace:=''">
+                       component_name:=''">
     <xacro:property name="ns" value="${robot_namespace + '/' if robot_namespace != '' else ''}" />
-    <xacro:property name="prefix" value="${device_namespace + '_' if device_namespace != '' else ''}" />
+    <xacro:property name="prefix" value="${component_name + '_' if component_name != '' else ''}" />
     <joint name="${parent_link.rstrip('_link')}_to_${prefix}wibotic_receiver_joint" type="fixed">
       <origin xyz="${xyz}" rpy="${rpy}" />

File: urdf/wibotic_station.urdf.xacro (robot description, xacro)
@@ -13,5 +13,5 @@
 -->
 <robot xmlns:xacro="http://www.ros.org/wiki/xacro" name="wibotic_station">
-  <xacro:arg name="device_namespace" default="" />
+  <xacro:arg name="component_name" default="" />
   <xacro:arg name="apriltag_image_path" default="" />
   <xacro:arg name="apriltag_size" default="0.07" />
@@ -20,6 +20,6 @@
                        xyz:='0.0 0.0 0.0'
                        rpy:='0.0 0.0 0.0'
-                       device_namespace:='station'">
-    <xacro:property name="prefix" value="${device_namespace + '_' if device_namespace != '' else ''}" />
+                       component_name:='station'">
+    <xacro:property name="prefix" value="${component_name + '_' if component_name != '' else ''}" />
     <joint name="${parent_link.rstrip('_link')}_to_${prefix}wibotic_station_joint" type="fixed">
       <origin xyz="${xyz}" rpy="${rpy}" />
@@ -70,6 +70,6 @@
   </xacro:macro>
   <xacro:macro name="create_apriltag"
-    params="name size:=$(arg apriltag_size) device_namespace:=''">
-    <xacro:property name="prefix" value="${device_namespace + '_' if device_namespace != '' else ''}" />
+    params="name size:=$(arg apriltag_size) component_name:=''">
+    <xacro:property name="prefix" value="${component_name + '_' if component_name != '' else ''}" />
     <link name="${prefix}${name}_link">
       <visual>
@@ -128,7 +128,7 @@
     <xacro:property name="apriltag_size_prop" value="$(arg apriltag_size)" />
     <xacro:wibotic_station
-      device_namespace="$(arg device_namespace)" parent_link="${prefix}${name}_image_link"  xyz="0.0 0.0 0.5"
+      component_name="$(arg component_name)" parent_link="${prefix}${name}_image_link"  xyz="0.0 0.0 0.5"
       rpy="${pi} 0 0 " />
   </xacro:macro>
-  <xacro:create_apriltag name="apriltag" device_namespace="$(arg device_namespace)" size="$(arg apriltag_size)" />
+  <xacro:create_apriltag name="apriltag" component_name="$(arg component_name)" size="$(arg apriltag_size)" />
 </robot>

Commit message: main urdf: ns -> robot_namespace_value

File: urdf/components.urdf.xacro (robot description, xacro)
@@ -32,5 +32,5 @@
       <xacro:property name="component" value="${config['components'][index]}" scope="parent" />
       <xacro:property name="type" value="${component['type']}" scope="parent" />
-      <xacro:property name="ns" value="${robot_namespace}" scope="parent" />
+      <xacro:property name="robot_namespace_value" value="${robot_namespace}" scope="parent" />
       <xacro:property name="dev_models_dict"
         value="${dict ([
@@ -68,5 +68,5 @@
             xyz="${xyz}"
             rpy="${rpy}"
-            robot_namespace="${ns}"
+            robot_namespace="${robot_namespace_value}"
             component_name="${component_name}"
           />
@@ -80,5 +80,5 @@
             xyz="${xyz}"
             rpy="${rpy}"
-            robot_namespace="${ns}"
+            robot_namespace="${robot_namespace_value}"
             component_name="${component_name}"
           />
@@ -92,5 +92,5 @@
             xyz="${xyz}"
             rpy="${rpy}"
-            robot_namespace="${ns}"
+            robot_namespace="${robot_namespace_value}"
             component_name="${component_name}"
             use_nominal_extrinsics="${use_sim}"
@@ -112,5 +112,5 @@
             xyz="${xyz}"
             rpy="${rpy}"
-            robot_namespace="${ns}"
+            robot_namespace="${robot_namespace_value}"
             component_name="${component_name}"
             model="${zed_models_dict[type]}"
@@ -130,5 +130,5 @@
             xyz="${xyz}"
             rpy="${rpy}"
-            robot_namespace="${ns}"
+            robot_namespace="${robot_namespace_value}"
             component_name="${component_name}"
             model="${luxonis_models_dict[type]}"
@@ -152,5 +152,5 @@
             xyz="${xyz}"
             rpy="${rpy}"
-            robot_namespace="${ns}"
+            robot_namespace="${robot_namespace_value}"
             component_name="${component_name}"
             model="${rplidar_models_dict[type]}"
@@ -175,5 +175,5 @@
             xyz="${xyz}"
             rpy="${rpy}"
-            robot_namespace="${ns}"
+            robot_namespace="${robot_namespace_value}"
             component_name="${component_name}"
             model="${ouster_models_dict[type]}"
@@ -189,5 +189,5 @@
             xyz="${xyz}"
             rpy="${rpy}"
-            robot_namespace="${ns}"
+            robot_namespace="${robot_namespace_value}"
             component_name="${component_name}"
           />
@@ -228,5 +228,5 @@
             xyz="${xyz}"
             rpy="${rpy}"
-            robot_namespace="${ns}"
+            robot_namespace="${robot_namespace_value}"
             component_name="${component_name}"
             kinova_type="gen3"
@@ -245,5 +245,5 @@
             xyz="${xyz}"
             rpy="${rpy}"
-            robot_namespace="${ns}"
+            robot_namespace="${robot_namespace_value}"
             component_name="${component_name}"
             kinova_type="gen3"
@@ -262,5 +262,5 @@
             xyz="${xyz}"
             rpy="${rpy}"
-            robot_namespace="${ns}"
+            robot_namespace="${robot_namespace_value}"
             component_name="${component_name}"
             kinova_type="gen3"
@@ -279,5 +279,5 @@
             xyz="${xyz}"
             rpy="${rpy}"
-            robot_namespace="${ns}"
+            robot_namespace="${robot_namespace_value}"
             kinova_type="gen3"
             dof="7"
@@ -306,5 +306,5 @@
             xyz="${xyz}"
             rpy="${rpy}"
-            robot_namespace="${ns}"
+            robot_namespace="${robot_namespace_value}"
             component_name="${component_name}"
           />
