Commit message: main urdf: remove robot_namespace_value

File: urdf/components.urdf.xacro (robot description, xacro)
@@ -32,5 +32,4 @@
       <xacro:property name="component" value="${config['components'][index]}" scope="parent" />
       <xacro:property name="type" value="${component['type']}" scope="parent" />
-      <xacro:property name="robot_namespace_value" value="${robot_namespace}" scope="parent" />
       <xacro:property name="dev_models_dict"
         value="${dict ([
@@ -68,5 +67,5 @@
             xyz="${xyz}"
             rpy="${rpy}"
-            robot_namespace="${robot_namespace_value}"
+            robot_namespace="${robot_namespace}"
             component_name="${component_name}"
           />
@@ -80,5 +79,5 @@
             xyz="${xyz}"
             rpy="${rpy}"
-            robot_namespace="${robot_namespace_value}"
+            robot_namespace="${robot_namespace}"
             component_name="${component_name}"
           />
@@ -92,5 +91,5 @@
             xyz="${xyz}"
             rpy="${rpy}"
-            robot_namespace="${robot_namespace_value}"
+            robot_namespace="${robot_namespace}"
             component_name="${component_name}"
             use_nominal_extrinsics="${use_sim}"
@@ -112,5 +111,5 @@
             xyz="${xyz}"
             rpy="${rpy}"
-            robot_namespace="${robot_namespace_value}"
+            robot_namespace="${robot_namespace}"
             component_name="${component_name}"
             model="${zed_models_dict[type]}"
@@ -130,5 +129,5 @@
             xyz="${xyz}"
             rpy="${rpy}"
-            robot_namespace="${robot_namespace_value}"
+            robot_namespace="${robot_namespace}"
             component_name="${component_name}"
             model="${luxonis_models_dict[type]}"
@@ -152,5 +151,5 @@
             xyz="${xyz}"
             rpy="${rpy}"
-            robot_namespace="${robot_namespace_value}"
+            robot_namespace="${robot_namespace}"
             component_name="${component_name}"
             model="${rplidar_models_dict[type]}"
@@ -175,5 +174,5 @@
             xyz="${xyz}"
             rpy="${rpy}"
-            robot_namespace="${robot_namespace_value}"
+            robot_namespace="${robot_namespace}"
             component_name="${component_name}"
             model="${ouster_models_dict[type]}"
@@ -189,5 +188,5 @@
             xyz="${xyz}"
             rpy="${rpy}"
-            robot_namespace="${robot_namespace_value}"
+            robot_namespace="${robot_namespace}"
             component_name="${component_name}"
           />
@@ -228,5 +227,5 @@
             xyz="${xyz}"
             rpy="${rpy}"
-            robot_namespace="${robot_namespace_value}"
+            robot_namespace="${robot_namespace}"
             component_name="${component_name}"
             kinova_type="gen3"
@@ -245,5 +244,5 @@
             xyz="${xyz}"
             rpy="${rpy}"
-            robot_namespace="${robot_namespace_value}"
+            robot_namespace="${robot_namespace}"
             component_name="${component_name}"
             kinova_type="gen3"
@@ -262,5 +261,5 @@
             xyz="${xyz}"
             rpy="${rpy}"
-            robot_namespace="${robot_namespace_value}"
+            robot_namespace="${robot_namespace}"
             component_name="${component_name}"
             kinova_type="gen3"
@@ -279,5 +278,5 @@
             xyz="${xyz}"
             rpy="${rpy}"
-            robot_namespace="${robot_namespace_value}"
+            robot_namespace="${robot_namespace}"
             kinova_type="gen3"
             dof="7"
@@ -306,5 +305,5 @@
             xyz="${xyz}"
             rpy="${rpy}"
-            robot_namespace="${robot_namespace_value}"
+            robot_namespace="${robot_namespace}"
             component_name="${component_name}"
           />

Commit message: Add tf_prefix arg and fix depthai reference frame for camera

File: urdf/components.urdf.xacro (robot description, xacro)
@@ -14,18 +14,20 @@
 <robot xmlns:xacro="http://wiki.ros.org/xacro">
   <xacro:macro name="create_components"
-    params="components_config_path namespace:='' use_sim:=False">
+              params="components_config_path
+                      namespace:=''
+                      use_sim:=False
+                      use_tf_prefix:=True">
     <xacro:unless value="${components_config_path == ''}">
-        <xacro:property
-          name="components_config"
-          value="${xacro.load_yaml(components_config_path)}" />
+      <xacro:property name="components_config" value="${xacro.load_yaml(components_config_path)}" />
       <xacro:load_componenet
         config="${components_config}"
         counter="${len(components_config['components'])}"
         robot_namespace="${namespace}"
-        use_sim="${use_sim}" />
+        use_sim="${use_sim}"
+        use_tf_prefix="${use_tf_prefix}" />
     </xacro:unless>
   </xacro:macro>
   <xacro:macro name="load_componenet"
-    params="config counter robot_namespace use_sim:=False">
+    params="config counter robot_namespace use_sim:=False use_tf_prefix:=True">
     <xacro:if value="${counter}">
       <xacro:property name="index" value="${counter - 1}" scope="parent" />
@@ -69,4 +71,5 @@
             robot_namespace="${robot_namespace}"
             component_name="${component_name}"
+            use_tf_prefix="${use_tf_prefix}"
           />
         </xacro:if>
@@ -81,4 +84,5 @@
             robot_namespace="${robot_namespace}"
             component_name="${component_name}"
+            use_tf_prefix="${use_tf_prefix}"
           />
         </xacro:if>
@@ -94,4 +98,5 @@
             component_name="${component_name}"
             use_nominal_extrinsics="${use_sim}"
+            use_tf_prefix="${use_tf_prefix}"
           />
         </xacro:if>
@@ -114,4 +119,5 @@
             component_name="${component_name}"
             model="${zed_models_dict[type]}"
+            use_tf_prefix="${use_tf_prefix}"
           />
         </xacro:if>
@@ -132,4 +138,5 @@
             component_name="${component_name}"
             model="${luxonis_models_dict[type]}"
+            use_tf_prefix="${use_tf_prefix}"
           />
         </xacro:if>
@@ -154,4 +161,5 @@
             component_name="${component_name}"
             model="${rplidar_models_dict[type]}"
+            use_tf_prefix="${use_tf_prefix}"
           />
         </xacro:if>
@@ -177,4 +185,5 @@
             component_name="${component_name}"
             model="${ouster_models_dict[type]}"
+            use_tf_prefix="${use_tf_prefix}"
           />
         </xacro:if>
@@ -190,4 +199,5 @@
             robot_namespace="${robot_namespace}"
             component_name="${component_name}"
+            use_tf_prefix="${use_tf_prefix}"
           />
         </xacro:if>
@@ -203,4 +213,5 @@
             component_name="${component_name}"
             ur_type="ur3e"
+            use_tf_prefix="${use_tf_prefix}"
           />
         </xacro:if>
@@ -216,4 +227,5 @@
             component_name="${component_name}"
             ur_type="ur5e"
+            use_tf_prefix="${use_tf_prefix}"
           />
         </xacro:if>
@@ -233,4 +245,5 @@
             gripper="robotiq_2f_85"
             vision="false"
+            use_tf_prefix="${use_tf_prefix}"
           />
         </xacro:if>
@@ -250,4 +263,5 @@
             gripper="robotiq_2f_85"
             vision="true"
+            use_tf_prefix="${use_tf_prefix}"
           />
         </xacro:if>
@@ -267,4 +281,5 @@
             gripper="robotiq_2f_85"
             vision="false"
+            use_tf_prefix="${use_tf_prefix}"
           />
         </xacro:if>
@@ -284,4 +299,5 @@
             vision="true"
             component_name="${component_name}"
+            use_tf_prefix="${use_tf_prefix}"
           />
         </xacro:if>
@@ -295,4 +311,5 @@
             component_name="${component_name}"
             robotiq_type="2f_85"
+            use_tf_prefix="${use_tf_prefix}"
           />
         </xacro:if>
@@ -307,4 +324,5 @@
             robot_namespace="${robot_namespace}"
             component_name="${component_name}"
+            use_tf_prefix="${use_tf_prefix}"
           />
         </xacro:if>
@@ -316,4 +334,5 @@
           robot_namespace="${robot_namespace}"
           use_sim="${use_sim}"
+          use_tf_prefix="${use_tf_prefix}"
         />
       </xacro:if>

File: urdf/intel_realsense_d435.urdf.xacro (robot description, xacro)
@@ -20,9 +20,11 @@
                        use_nominal_extrinsics:=false
                        robot_namespace:=''
-                       component_name:=''">
+                       component_name:=''
+                       use_tf_prefix:=True">
     <xacro:if value="${component_name == ''}">
       <xacro:property name="component_name" value="camera" />
     </xacro:if>
     <xacro:property name="robot_namespace_slash" value="${robot_namespace + '/' if robot_namespace != '' else ''}" />
+    <xacro:property name="tf_prefix" value="${robot_namespace_slash if use_tf_prefix in ['True', True] else ''}" />
     <xacro:property name="component_name_underscore" value="${component_name + '_' if component_name != '' else ''}" />
     <xacro:property name="component_name_slash" value="${component_name + '/' if component_name != '' else ''}" />
@@ -144,5 +146,5 @@
       name="${robot_namespace_slash}${component_name_underscore}intel_realsense_d435_color"
       topic="${robot_namespace_slash}${component_name_slash}color/image_raw"
-      frame_id="${robot_namespace_slash}${component_name_underscore}color_optical_frame"
+      frame_id="${tf_prefix}${component_name_underscore}color_optical_frame"
       frequency="30"
       width="1280"
@@ -153,5 +155,5 @@
       name="${robot_namespace_slash}${component_name_underscore}intel_realsense_d435_depth"
       topic="${robot_namespace_slash}${component_name_slash}depth/image_rect_raw"
-      frame_id="${robot_namespace_slash}${component_name_underscore}depth_optical_frame"
+      frame_id="${tf_prefix}${component_name_underscore}depth_optical_frame"
       frequency="30"
       width="1280"

File: urdf/kinova.urdf.xacro (robot description, xacro)
@@ -47,9 +47,11 @@
                        vision:=false
                        robot_namespace:=''
-                       component_name:=''">
+                       component_name:=''
+                       use_tf_prefix:=True">
     <xacro:if value="${component_name == ''}">
       <xacro:property name="component_name" value="kinova" />
     </xacro:if>
     <xacro:property name="robot_namespace_slash" value="${robot_namespace + '/' if robot_namespace != '' else ''}" />
+    <xacro:property name="tf_prefix" value="${robot_namespace_slash if use_tf_prefix in ['True', True] else ''}" />
     <xacro:property name="component_name_underscore" value="${component_name + '_' if component_name != '' else ''}" />
     <xacro:property name="component_name_slash" value="${component_name + '/' if component_name != '' else ''}" />
@@ -181,5 +183,5 @@
             <optical_frame_id>${component_name_underscore}color_optical_frame</optical_frame_id>
           </camera>
-          <gz_frame_id>${robot_namespace_slash}${component_name_underscore}camera_color_frame</gz_frame_id>
+          <gz_frame_id>${tf_prefix}${component_name_underscore}camera_color_frame</gz_frame_id>
           <always_on>1</always_on>
           <update_rate>${camera_fps}</update_rate>

File: urdf/luxonis_depthai.urdf.xacro (robot description, xacro)
@@ -20,9 +20,11 @@
                        component_name:=''
                        model:='OAK-D-PRO'
-                       use_sim:=False">
+                       use_sim:=False
+                       use_tf_prefix:=True">
     <xacro:if value="${component_name == ''}">
       <xacro:property name="component_name" value="oak" />
     </xacro:if>
     <xacro:property name="robot_namespace_slash" value="${robot_namespace + '/' if robot_namespace != '' else ''}" />
+    <xacro:property name="tf_prefix" value="${robot_namespace_slash if use_tf_prefix in ['True', True] else ''}" />
     <xacro:property name="component_name_underscore" value="${component_name + '_' if component_name != '' else ''}" />
     <xacro:property name="component_name_slash" value="${component_name + '/' if component_name != '' else ''}" />
@@ -31,5 +33,5 @@
     <xacro:include filename="$(find depthai_descriptions)/urdf/include/depthai_macro.urdf.xacro" />
     <xacro:depthai_camera camera_name="${component_name}" parent="${parent_link}"
-      base_frame="${robot_namespace_slash}${component_name_underscore_nonempty}link" camera_model="${model}"
+      base_frame="${component_name_underscore_nonempty}link" camera_model="${model}"
       cam_pos_x="${xyz.split()[0]}" cam_pos_y="${xyz.split()[1]}" cam_pos_z="${xyz.split()[2]}"
       cam_roll="${rpy.split()[0]}" cam_pitch="${rpy.split()[1]}" cam_yaw="${rpy.split()[2]}"
@@ -41,5 +43,5 @@
       name="${robot_namespace_slash}${component_name_underscore}color"
       topic="${robot_namespace_slash}${component_name_slash}rgb/color"
-      frame_id="${robot_namespace_slash}${component_name_underscore}rgb_camera_frame"
+      frame_id="${tf_prefix}${component_name_underscore}rgb_camera_frame"
       frequency="30"
       width="1280"
@@ -50,5 +52,5 @@
       name="${robot_namespace_slash}${component_name_underscore}depth"
       topic="${robot_namespace_slash}${component_name_slash}stereo/depth"
-      frame_id="${robot_namespace_slash}${component_name_underscore}rgb_camera_frame"
+      frame_id="${tf_prefix}${component_name_underscore}rgb_camera_frame"
       frequency="30"
       width="1280"

File: urdf/orbbec_astra.urdf.xacro (robot description, xacro)
@@ -18,9 +18,11 @@
                        rpy:='0.0 0.0 0.0'
                        robot_namespace:=''
-                       component_name:=''">
+                       component_name:=''
+                       use_tf_prefix:=True">
     <xacro:if value="${component_name == ''}">
       <xacro:property name="component_name" value="camera" />
     </xacro:if>
     <xacro:property name="robot_namespace_slash" value="${robot_namespace + '/' if robot_namespace != '' else ''}" />
+    <xacro:property name="tf_prefix" value="${robot_namespace_slash if use_tf_prefix in ['True', True] else ''}" />
     <xacro:property name="component_name_underscore" value="${component_name + '_' if component_name != '' else ''}" />
     <xacro:property name="component_name_slash" value="${component_name + '/' if component_name != '' else ''}" />
@@ -115,5 +117,5 @@
       name="${robot_namespace_slash}${component_name_underscore}camera_color"
       topic="${robot_namespace_slash}${component_name_slash}color/image_raw"
-      frame_id="${robot_namespace_slash}${component_name_underscore}color_optical_frame"
+      frame_id="${tf_prefix}${component_name_underscore}color_optical_frame"
       frequency="30"
       width="640"
@@ -124,5 +126,5 @@
       name="${robot_namespace_slash}${component_name_underscore}camera_depth"
       topic="${robot_namespace_slash}${component_name_slash}depth/image_raw"
-      frame_id="${robot_namespace_slash}${component_name_underscore}depth_optical_frame"
+      frame_id="${tf_prefix}${component_name_underscore}depth_optical_frame"
       frequency="30"
       width="640"

File: urdf/ouster.urdf.xacro (robot description, xacro)
@@ -19,5 +19,6 @@
                        model:=os1_32
                        robot_namespace:=''
-                       component_name:=''">
+                       component_name:=''
+                       use_tf_prefix:=True">
     <!-- <xacro:if value="${component_name == ''}">
       <xacro:property name="component_name" value="ouster" />
@@ -25,4 +26,5 @@
     <!-- ^ removed for compatibility with hw driver -->
     <xacro:property name="robot_namespace_slash" value="${robot_namespace + '/' if robot_namespace != '' else ''}" />
+    <xacro:property name="tf_prefix" value="${robot_namespace_slash if use_tf_prefix in ['True', True] else ''}" />
     <xacro:property name="component_name_underscore" value="${component_name + '_' if component_name != '' else ''}" />
     <xacro:property name="component_name_slash" value="${component_name + '/' if component_name != '' else ''}" />
@@ -130,5 +132,5 @@
         <update_rate>20.0</update_rate>
         <topic>${robot_namespace_slash}${component_name_slash}ouster/points</topic>
-        <gz_frame_id>${robot_namespace_slash}${component_name_underscore}os_lidar</gz_frame_id>
+        <gz_frame_id>${tf_prefix}${component_name_underscore}os_lidar</gz_frame_id>
         <always_on>true</always_on>
       </sensor>

File: urdf/slamtec_rplidar.urdf.xacro (robot description, xacro)
@@ -19,5 +19,6 @@
                        robot_namespace:=''
                        component_name:=''
-                       model:=s3">
+                       model:=s3
+                       use_tf_prefix:=True">
     <!-- <xacro:if value="${component_name == ''}">
       <xacro:property name="component_name" value="rplidar" />
@@ -25,4 +26,5 @@
     <!-- ^ removed for compatibility with hw driver -->
     <xacro:property name="robot_namespace_slash" value="${robot_namespace + '/' if robot_namespace != '' else ''}" />
+    <xacro:property name="tf_prefix" value="${robot_namespace_slash if use_tf_prefix in ['True', True] else ''}" />
     <xacro:property name="component_name_underscore" value="${component_name + '_' if component_name != '' else ''}" />
     <xacro:property name="component_name_slash" value="${component_name + '/' if component_name != '' else ''}" />
@@ -240,5 +242,5 @@
         <visualize>false</visualize>
         <topic>${robot_namespace_slash}${component_name_slash}scan</topic>
-        <gz_frame_id>${robot_namespace_slash}${component_name_underscore}laser</gz_frame_id>
+        <gz_frame_id>${tf_prefix}${component_name_underscore}laser</gz_frame_id>
         <ray>
           <scan>

File: urdf/stereolabs_zed.urdf.xacro (robot description, xacro)
@@ -22,9 +22,11 @@
                        model:=zed
                        robot_namespace:=''
-                       component_name:=''">
+                       component_name:=''
+                       use_tf_prefix:=True">
     <xacro:if value="${component_name == ''}">
       <xacro:property name="component_name" value="zed" />
     </xacro:if>
     <xacro:property name="robot_namespace_slash" value="${robot_namespace + '/' if robot_namespace != '' else ''}" />
+    <xacro:property name="tf_prefix" value="${robot_namespace_slash if use_tf_prefix in ['True', True] else ''}" />
     <xacro:property name="component_name_underscore" value="${component_name + '_' if component_name != '' else ''}" />
     <xacro:property name="component_name_slash" value="${component_name + '/' if component_name != '' else ''}" />
@@ -310,5 +312,5 @@
       name="${robot_namespace_slash}${component_name_underscore}camera_color"
       topic="${robot_namespace_slash}${component_name_slash}zed_node/rgb/image_rect_color"
-      frame_id="${robot_namespace_slash}${component_name_underscore}camera_center"
+      frame_id="${tf_prefix}${component_name_underscore}camera_center"
       frequency="30"
       width="1280"
@@ -319,5 +321,5 @@
       name="${robot_namespace_slash}${component_name_underscore}camera_depth"
       topic="${robot_namespace_slash}${component_name_slash}zed_node/depth"
-      frame_id="${robot_namespace_slash}${component_name_underscore}camera_center"
+      frame_id="${tf_prefix}${component_name_underscore}camera_center"
       frequency="30"
       width="1280"

File: urdf/teltonika_003R-00253.urdf.xacro (robot description, xacro)
@@ -18,9 +18,11 @@
                        rpy:='0.0 0.0 0.0'
                        robot_namespace:=''
-                       component_name:=''">
+                       component_name:=''
+                       use_tf_prefix:=True">
     <xacro:if value="${component_name == ''}">
       <xacro:property name="component_name" value="gps" />
     </xacro:if>
     <xacro:property name="robot_namespace_slash" value="${robot_namespace + '/' if robot_namespace != '' else ''}" />
+    <xacro:property name="tf_prefix" value="${robot_namespace_slash if use_tf_prefix in ['True', True] else ''}" />
     <xacro:property name="component_name_underscore" value="${component_name + '_' if component_name != '' else ''}" />
     <xacro:property name="component_name_slash" value="${component_name + '/' if component_name != '' else ''}" />
@@ -67,5 +69,5 @@
         <update_rate>1</update_rate>
         <topic>${robot_namespace_slash}${component_name_slash}fix</topic>
-        <gz_frame_id>${robot_namespace_slash}${component_name_underscore}antenna</gz_frame_id>
+        <gz_frame_id>${tf_prefix}${component_name_underscore}antenna</gz_frame_id>
       </sensor>
     </gazebo>

File: urdf/velodyne_puck.urdf.xacro (robot description, xacro)
@@ -18,5 +18,6 @@
                        rpy:='0.0 0.0 0.0'
                        robot_namespace:=''
-                       component_name:=''">
+                       component_name:=''
+                       use_tf_prefix:=True">
     <!-- <xacro:if value="${component_name == ''}">
       <xacro:property name="component_name" value="velodyne" />
@@ -24,4 +25,5 @@
     <!-- ^ removed for compatibility with hw driver -->
     <xacro:property name="robot_namespace_slash" value="${robot_namespace + '/' if robot_namespace != '' else ''}" />
+    <xacro:property name="tf_prefix" value="${robot_namespace_slash if use_tf_prefix in ['True', True] else ''}" />
     <xacro:property name="component_name_underscore" value="${component_name + '_' if component_name != '' else ''}" />
     <xacro:property name="component_name_slash" value="${component_name + '/' if component_name != '' else ''}" />
@@ -104,5 +106,5 @@
         </ray>
         <topic>${robot_namespace_slash}${component_name_slash}velodyne_points</topic>
-        <gz_frame_id>${robot_namespace_slash}${component_name_underscore}velodyne</gz_frame_id>
+        <gz_frame_id>${tf_prefix}${component_name_underscore}velodyne</gz_frame_id>
         <always_on>true</always_on>
       </sensor>
