Commit message: Add tf_prefix arg and fix depthai reference frame for camera (#14)

File: urdf/components.urdf.xacro (robot description, xacro)
@@ -14,18 +14,20 @@
 <robot xmlns:xacro="http://wiki.ros.org/xacro">
   <xacro:macro name="create_components"
-    params="components_config_path namespace:='' use_sim:=False">
+              params="components_config_path
+                      namespace:=''
+                      use_sim:=False
+                      use_tf_prefix:=True">
     <xacro:unless value="${components_config_path == ''}">
-        <xacro:property
-          name="components_config"
-          value="${xacro.load_yaml(components_config_path)}" />
+      <xacro:property name="components_config" value="${xacro.load_yaml(components_config_path)}" />
       <xacro:load_componenet
         config="${components_config}"
         counter="${len(components_config['components'])}"
         robot_namespace="${namespace}"
-        use_sim="${use_sim}" />
+        use_sim="${use_sim}"
+        use_tf_prefix="${use_tf_prefix}" />
     </xacro:unless>
   </xacro:macro>
   <xacro:macro name="load_componenet"
-    params="config counter robot_namespace use_sim:=False">
+    params="config counter robot_namespace use_sim:=False use_tf_prefix:=True">
     <xacro:if value="${counter}">
       <xacro:property name="index" value="${counter - 1}" scope="parent" />
@@ -69,4 +71,5 @@
             robot_namespace="${robot_namespace}"
             component_name="${component_name}"
+            use_tf_prefix="${use_tf_prefix}"
           />
         </xacro:if>
@@ -81,4 +84,5 @@
             robot_namespace="${robot_namespace}"
             component_name="${component_name}"
+            use_tf_prefix="${use_tf_prefix}"
           />
         </xacro:if>
@@ -94,4 +98,5 @@
             component_name="${component_name}"
             use_nominal_extrinsics="${use_sim}"
+            use_tf_prefix="${use_tf_prefix}"
           />
         </xacro:if>
@@ -114,4 +119,5 @@
             component_name="${component_name}"
             model="${zed_models_dict[type]}"
+            use_tf_prefix="${use_tf_prefix}"
           />
         </xacro:if>
@@ -132,4 +138,5 @@
             component_name="${component_name}"
             model="${luxonis_models_dict[type]}"
+            use_tf_prefix="${use_tf_prefix}"
           />
         </xacro:if>
@@ -154,4 +161,5 @@
             component_name="${component_name}"
             model="${rplidar_models_dict[type]}"
+            use_tf_prefix="${use_tf_prefix}"
           />
         </xacro:if>
@@ -177,4 +185,5 @@
             component_name="${component_name}"
             model="${ouster_models_dict[type]}"
+            use_tf_prefix="${use_tf_prefix}"
           />
         </xacro:if>
@@ -190,4 +199,5 @@
             robot_namespace="${robot_namespace}"
             component_name="${component_name}"
+            use_tf_prefix="${use_tf_prefix}"
           />
         </xacro:if>
@@ -233,4 +243,5 @@
             gripper="robotiq_2f_85"
             vision="false"
+            use_tf_prefix="${use_tf_prefix}"
           />
         </xacro:if>
@@ -250,4 +261,5 @@
             gripper="robotiq_2f_85"
             vision="true"
+            use_tf_prefix="${use_tf_prefix}"
           />
         </xacro:if>
@@ -267,4 +279,5 @@
             gripper="robotiq_2f_85"
             vision="false"
+            use_tf_prefix="${use_tf_prefix}"
           />
         </xacro:if>
@@ -284,4 +297,5 @@
             vision="true"
             component_name="${component_name}"
+            use_tf_prefix="${use_tf_prefix}"
           />
         </xacro:if>
@@ -316,4 +330,5 @@
           robot_namespace="${robot_namespace}"
           use_sim="${use_sim}"
+          use_tf_prefix="${use_tf_prefix}"
         />
       </xacro:if>

Commit message: Added reling component
Signed-off-by: Jakub Delicat <jakub.delicat@husarion.com>

File: urdf/components.urdf.xacro (robot description, xacro)
@@ -71,4 +71,18 @@
           />
         </xacro:if>
+        <xacro:if value="${type == 'REL'}">
+          <xacro:include
+            filename="$(find husarion_components_description)/urdf/reling.urdf.xacro"
+            ns="relings" />
+         <xacro:property name="length" value="${component['length'] if 'length' in component else '1.0'}" scope="parent" />
+          <xacro:relings.reling
+            parent_link="${parent_link}"
+            length="${length}"
+            xyz="${xyz}"
+            rpy="${rpy}"
+            robot_namespace="${robot_namespace}"
+            component_name="${component_name}"
+          />
+        </xacro:if>
         <xacro:if value="${type == 'CAM01'}">
           <xacro:include

Commit message: Add reling component (#15)

File: urdf/components.urdf.xacro (robot description, xacro)
@@ -74,4 +74,18 @@
           />
         </xacro:if>
+        <xacro:if value="${type == 'REL'}">
+          <xacro:include
+            filename="$(find husarion_components_description)/urdf/reling.urdf.xacro"
+            ns="relings" />
+         <xacro:property name="length" value="${component['length'] if 'length' in component else '1.0'}" scope="parent" />
+          <xacro:relings.reling
+            parent_link="${parent_link}"
+            length="${length}"
+            xyz="${xyz}"
+            rpy="${rpy}"
+            robot_namespace="${robot_namespace}"
+            component_name="${component_name}"
+          />
+        </xacro:if>
         <xacro:if value="${type == 'CAM01'}">
           <xacro:include

Commit message: add multiple elements to rails

File: urdf/components.urdf.xacro (robot description, xacro)
@@ -20,5 +20,5 @@
     <xacro:unless value="${components_config_path == ''}">
       <xacro:property name="components_config" value="${xacro.load_yaml(components_config_path)}" />
-      <xacro:load_componenet
+      <xacro:load_component
         config="${components_config}"
         counter="${len(components_config['components'])}"
@@ -28,5 +28,5 @@
     </xacro:unless>
   </xacro:macro>
-  <xacro:macro name="load_componenet"
+  <xacro:macro name="load_component"
     params="config counter robot_namespace use_sim:=False use_tf_prefix:=True">
     <xacro:if value="${counter}">
@@ -81,9 +81,9 @@
           <xacro:relings.reling
             parent_link="${parent_link}"
-            length="${length}"
-            xyz="${xyz}"
-            rpy="${rpy}"
-            robot_namespace="${robot_namespace}"
-            component_name="${component_name}"
+            xyz="${xyz}"
+            rpy="${rpy}"
+            robot_namespace="${robot_namespace}"
+            component_name="${component_name}"
+            elements="${component['elements']}"
           />
         </xacro:if>
@@ -339,5 +339,5 @@
       </xacro:unless>
       <xacro:if value="${index}">
-        <xacro:load_componenet
+        <xacro:load_component
           counter="${index}"
           config="${config}"

File: urdf/reling.urdf.xacro (robot description, xacro)
@@ -15,9 +15,9 @@
   <xacro:macro name="reling"
                params="parent_link
-                       length:='1.0'
                        xyz:='0.0 0.0 0.0'
                        rpy:='0.0 0.0 0.0'
                        robot_namespace:=''
-                       component_name:=''">
+                       component_name:=''
+                       elements">
     <xacro:if value="${component_name == ''}">
       <xacro:property name="component_name" value="reling" />
@@ -31,17 +31,27 @@
     </joint>
     <link name="${component_name_underscore}mount_link">
+      <xacro:load_element elements="${elements}" counter="${len(elements)}" />
+    </link>
+  </xacro:macro>
+  <xacro:macro name="load_element" params="elements counter">
+    <xacro:if value="${counter}">
+      <xacro:property name="index" value="${counter - 1}" scope="parent" />
+      <xacro:property name="component" value="${elements[index]}" scope="parent" />
       <visual>
-        <origin xyz="0.0 0.0 0.0" rpy="0.0 0.0 0.0" />
+        <origin xyz="${component['xyz']}" rpy="${component['rpy']}" />
         <geometry>
-          <mesh filename="package://husarion_components_description/meshes/reling.dae" scale="${length} 1.0 1.0"/>
+          <mesh filename="package://husarion_components_description/meshes/reling.dae" scale="${component['length']} 1.0 1.0"/>
         </geometry>
       </visual>
       <collision>
-         <origin xyz="0.0 0.0 0.0" rpy="0.0 ${pi/2.0} 0.0" />
+         <origin xyz="${component['xyz']}" rpy="${component['rpy']}" />
         <geometry>
-          <box size="0.0202 0.0202 ${length}" />
+          <box size="0.0202 0.0202 ${component['length']}" />
         </geometry>
       </collision>
-    </link>
+      <xacro:if value="${index}">
+        <xacro:load_element elements="${elements}" counter="${index}" />
+      </xacro:if>
+    </xacro:if>
   </xacro:macro>
 </robot>

Commit message: rename reling to rack

File: urdf/components.urdf.xacro (robot description, xacro)
@@ -74,10 +74,10 @@
           />
         </xacro:if>
-        <xacro:if value="${type == 'REL'}">
-          <xacro:include
-            filename="$(find husarion_components_description)/urdf/reling.urdf.xacro"
-            ns="relings" />
+        <xacro:if value="${type == 'RCK'}">
+          <xacro:include
+            filename="$(find husarion_components_description)/urdf/rack.urdf.xacro"
+            ns="rack" />
          <xacro:property name="length" value="${component['length'] if 'length' in component else '1.0'}" scope="parent" />
-          <xacro:relings.reling
+          <xacro:rack.rack
             parent_link="${parent_link}"
             xyz="${xyz}"

File: urdf/rack.urdf.xacro (robot description, xacro)
@@ -13,5 +13,5 @@
 -->
 <robot xmlns:xacro="http://www.ros.org/wiki/xacro">
-  <xacro:macro name="reling"
+  <xacro:macro name="rack"
                params="parent_link
                        xyz:='0.0 0.0 0.0'
@@ -21,5 +21,5 @@
                        elements">
     <xacro:if value="${component_name == ''}">
-      <xacro:property name="component_name" value="reling" />
+      <xacro:property name="component_name" value="rack" />
     </xacro:if>
     <xacro:property name="robot_namespace_slash" value="${robot_namespace + '/' if robot_namespace != '' else ''}" />
@@ -41,5 +41,5 @@
         <origin xyz="${component['xyz']}" rpy="${component['rpy']}" />
         <geometry>
-          <mesh filename="package://husarion_components_description/meshes/reling.dae" scale="${component['length']} 1.0 1.0"/>
+          <mesh filename="package://husarion_components_description/meshes/v_slot_profile.dae" scale="${component['length']} 1.0 1.0"/>
         </geometry>
       </visual>

Commit message: Rails elements (#17)
* add multiple elements to rails

* fix collision

* test different runner

* test container

* try core and manual install

* init rosdep

* simplify and install coveragepy

* clean up

* rename reling to rack

File: urdf/components.urdf.xacro (robot description, xacro)
@@ -20,5 +20,5 @@
     <xacro:unless value="${components_config_path == ''}">
       <xacro:property name="components_config" value="${xacro.load_yaml(components_config_path)}" />
-      <xacro:load_componenet
+      <xacro:load_component
         config="${components_config}"
         counter="${len(components_config['components'])}"
@@ -28,5 +28,5 @@
     </xacro:unless>
   </xacro:macro>
-  <xacro:macro name="load_componenet"
+  <xacro:macro name="load_component"
     params="config counter robot_namespace use_sim:=False use_tf_prefix:=True">
     <xacro:if value="${counter}">
@@ -74,16 +74,16 @@
           />
         </xacro:if>
-        <xacro:if value="${type == 'REL'}">
-          <xacro:include
-            filename="$(find husarion_components_description)/urdf/reling.urdf.xacro"
-            ns="relings" />
+        <xacro:if value="${type == 'RCK'}">
+          <xacro:include
+            filename="$(find husarion_components_description)/urdf/rack.urdf.xacro"
+            ns="rack" />
          <xacro:property name="length" value="${component['length'] if 'length' in component else '1.0'}" scope="parent" />
-          <xacro:relings.reling
-            parent_link="${parent_link}"
-            length="${length}"
-            xyz="${xyz}"
-            rpy="${rpy}"
-            robot_namespace="${robot_namespace}"
-            component_name="${component_name}"
+          <xacro:rack.rack
+            parent_link="${parent_link}"
+            xyz="${xyz}"
+            rpy="${rpy}"
+            robot_namespace="${robot_namespace}"
+            component_name="${component_name}"
+            elements="${component['elements']}"
           />
         </xacro:if>
@@ -339,5 +339,5 @@
       </xacro:unless>
       <xacro:if value="${index}">
-        <xacro:load_componenet
+        <xacro:load_component
           counter="${index}"
           config="${config}"

File: urdf/rack.urdf.xacro (robot description, xacro)
@@ -13,13 +13,13 @@
 -->
 <robot xmlns:xacro="http://www.ros.org/wiki/xacro">
-  <xacro:macro name="reling"
+  <xacro:macro name="rack"
                params="parent_link
-                       length:='1.0'
                        xyz:='0.0 0.0 0.0'
                        rpy:='0.0 0.0 0.0'
                        robot_namespace:=''
-                       component_name:=''">
+                       component_name:=''
+                       elements">
     <xacro:if value="${component_name == ''}">
-      <xacro:property name="component_name" value="reling" />
+      <xacro:property name="component_name" value="rack" />
     </xacro:if>
     <xacro:property name="robot_namespace_slash" value="${robot_namespace + '/' if robot_namespace != '' else ''}" />
@@ -31,17 +31,27 @@
     </joint>
     <link name="${component_name_underscore}mount_link">
+      <xacro:load_element elements="${elements}" counter="${len(elements)}" />
+    </link>
+  </xacro:macro>
+  <xacro:macro name="load_element" params="elements counter">
+    <xacro:if value="${counter}">
+      <xacro:property name="index" value="${counter - 1}" scope="parent" />
+      <xacro:property name="component" value="${elements[index]}" scope="parent" />
       <visual>
-        <origin xyz="0.0 0.0 0.0" rpy="0.0 0.0 0.0" />
+        <origin xyz="${component['xyz']}" rpy="${component['rpy']}" />
         <geometry>
-          <mesh filename="package://husarion_components_description/meshes/reling.dae" scale="${length} 1.0 1.0"/>
+          <mesh filename="package://husarion_components_description/meshes/v_slot_profile.dae" scale="${component['length']} 1.0 1.0"/>
         </geometry>
       </visual>
       <collision>
-         <origin xyz="0.0 0.0 0.0" rpy="0.0 ${pi/2.0} 0.0" />
+         <origin xyz="${component['xyz']}" rpy="${component['rpy']}" />
         <geometry>
-          <box size="0.0202 0.0202 ${length}" />
+          <box size="${component['length']} 0.0202 0.0202" />
         </geometry>
       </collision>
-    </link>
+      <xacro:if value="${index}">
+        <xacro:load_element elements="${elements}" counter="${index}" />
+      </xacro:if>
+    </xacro:if>
   </xacro:macro>
 </robot>

Commit message: Let components.yaml slide DEV joint xyz on the mount plate
The DEV05 pillar, DEV07 small gate, and DEV09 large gate bolt onto the
v-slot grid on top of the mount plate and the customer can shift them
forwards/backwards in practice. The URDF was hardcoding one position per
DEV, so the rendered configuration didn't match what was actually built.

This commit lets components.yaml override the dev macro's default xyz:

  - components:
      - type: DEV07
        xyz: 0.10 0 0.143    # 10 cm forward of default

dev.urdf.xacro grows an optional xyz_override macro parameter; when
non-empty it replaces the model's default xyz on the joint origin.
components.urdf.xacro reads the optional xyz field from each DEV-type
component entry and passes it through. Existing components.yaml files
without an xyz field continue to use the original defaults.

File: urdf/components.urdf.xacro (robot description, xacro)
@@ -111,6 +111,10 @@
           ns="dev"
         />
+        <!-- Optional xyz override: lets components.yaml slide DEV05/07/09
+             along the mount plate. Empty string means "use macro default". -->
+        <xacro:property name="dev_xyz" value="${component['xyz'] if 'xyz' in component else ''}" scope="parent" />
         <xacro:dev.dev
           model="${dev_models_dict[type]}"
+          xyz_override="${dev_xyz}"
         />
       </xacro:if>

File: urdf/dev.urdf.xacro (robot description, xacro)
@@ -39,5 +39,5 @@
   -->
   <xacro:macro name="dev"
-               params="model:=dev01">
+               params="model:=dev01 xyz_override:=''">
     <xacro:if value="${model == 'dev01'}">
       <xacro:property name="parent_link" value="body_link" scope="parent" />
@@ -132,4 +132,9 @@
       <xacro:property name="collision_box_xyz"  value="0 0 -0.125"      scope="parent" />
     </xacro:if>
+    <!-- xyz_override (optional) replaces the model's default mount xyz.
+         Lets components.yaml slide DEV05/07/09 along the mount plate. -->
+    <xacro:if value="${xyz_override != ''}">
+      <xacro:property name="xyz" value="${xyz_override}" scope="parent" />
+    </xacro:if>
     <joint name="${model}_joint" type="fixed">
       <origin xyz="${xyz}" rpy="${rpy}" />

Commit message: Add custom component type for user URDF/mesh

File: urdf/components.urdf.xacro (robot description, xacro)
@@ -337,4 +337,27 @@
           />
         </xacro:if>
+        <!-- User-supplied URDF/xacro. `file` is resolved against `package` when -->
+        <!-- present ($(find package)/file), otherwise taken as an absolute path. -->
+        <!-- The included file must define a macro with the standard component -->
+        <!-- signature; its name defaults to `custom_component` and is overridable -->
+        <!-- via `macro_name`. -->
+        <xacro:if value="${type == 'custom'}">
+          <xacro:property name="macro_name"
+            value="${component['macro_name'] if 'macro_name' in component else 'custom_component'}" scope="parent" />
+          <xacro:if value="${'package' in component}">
+            <xacro:include filename="$(find ${component['package']})/${component['file']}" ns="custom" />
+          </xacro:if>
+          <xacro:unless value="${'package' in component}">
+            <xacro:include filename="${component['file']}" ns="custom" />
+          </xacro:unless>
+          <xacro:call macro="custom.${macro_name}"
+            parent_link="${parent_link}"
+            xyz="${xyz}"
+            rpy="${rpy}"
+            robot_namespace="${robot_namespace}"
+            component_name="${component_name}"
+            use_tf_prefix="${use_tf_prefix}"
+          />
+        </xacro:if>
       </xacro:unless>
       <xacro:if value="${index}">
